File: kicad/Ryujin/Ryujin.kicad_sch (KiCad schematic)
At the start: 15 parts, among them J3 BAT, J4 SDI12, Q1 IRLML6244, U1 TXS0101DBV, U2 R-78E5.0-0.5, U3 W25Q32JVSS

Commit message: The Road to Calydon
Parts:
- added C4, C5: 0.1uF, Capacitor_SMD:C_0603_1608Metric, symbol Device:C
- C3: MPN 0.1uF 0201 -> 0.1uF 0603
- R1, R3: MPN 47k 0201 -> 47k 0603
- R2: MPN 100 0201 -> 100 0603
- R4: value 953k -> 1.2M; MPN 953k 0201 -> 1.2M 0603
- R5: value 348k -> 330k; MPN 348k 0201 -> 330k 0603
Connections:
- net at A1.3V3 (3.3V), R1.2, U1.1 (V_{CCA})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: now also U3.3 (IO2), U3.7 (IO3), C5.1
- net at A1.GND, C1.2, C2.2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: now also J3.1 (Pin_1), J4.1 (Pin_1), U3.1 (~{CS}), C4.2, C5.2; no longer J3.2 (Pin_2), Q1.2 (S)
- net at U1.4 (B): now also J4.3 (Pin_3); no longer J4.1 (Pin_1)
- net at J4.2 (Pin_2): now also Q1.2 (S); no longer Q1.3 (D)
- net at C1.1, R4.1, U2.1 (IN): now also J3.2 (Pin_2), Q1.3 (D); no longer J3.1 (Pin_1), J4.3 (Pin_3)
- net at A1.5V, U1.6 (V_{CCB}): now also C4.1

Commit message: The Festival of Dionysus
Parts:
- C3: MPN 0.1uF 0603 -> 0.1uF 16V 0603
- C4, C5: MPN 0.1uF 0603 -> 0.1uF 6.3V 0603
Other:
- note added: "2024-12-15"
Changed lines of the file:
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@@
+		)
+	)
+	(text "2024-12-15"
+		(exclude_from_sim no)
+		(at 213.868 193.548 0)
+		(effects
+			(font
+				(size 1.27 1.27)
+			)
 		)
 	)
@@
 			)
 		)
-		(property "MPN" "0.1uF 0603"
+		(property "MPN" "0.1uF 6.3V 0603"
 			(at 114.3 100.33 90)
 			(effects
@@
 			)
 		)
-		(property "MPN" "0.1uF 0603"
+		(property "MPN" "0.1uF 16V 0603"
 			(at 52.07 116.84 90)
 			(effects
@@
 			)
 		)
-		(property "MPN" "0.1uF 0603"
+		(property "MPN" "0.1uF 6.3V 0603"
 			(at 110.49 93.98 90)
 			(effects

Commit message: Ares
Parts:
- C3: MPN 0.1uF 16V 0603 -> 0.1uF 0603 16V
- C4: MPN 0.1uF 6.3V 0603 -> 0.1uF 0603 6V
- C5: MPN 0.1uF 6.3V 0603 -> 0.1uF 0603 4V
Other:
- moved on the sheet: A1, U3

Commit message: Pride Comes Before a Brawl
Parts:
- A1: footprint PCM_arduino-library:Arduino_MKR_FOX_1200_Socket -> Custom:Arduino_MKR_NB_1500_Socket
- C3: MPN 0.1uF 0603 16V -> 0.1uF 16V 0603
- C4: MPN 0.1uF 0603 6V -> 0.1uF 6.3V 0603
- C5: MPN 0.1uF 0603 4V -> 0.1uF 6.3V 0603
- R4: value 1.2M -> 330k; MPN 1.2M 0603 -> 330k 0603
- R5: value 330k -> 1.2M; MPN 330k 0603 -> 1.2M 0603
- renumbered J3 to J1, J4 to J2
Connections:
- net 3V3: now reaches A1.3V3 (3.3V), C5.1, R1.2, U1.1 (V_{CCA}), U3.3 (IO2), U3.7 (IO3), U3.8 (VCC)
- net GND: now reaches A1.GND, C1.2, C2.2, C5.2, J1.1 (Pin_1), J2.1 (Pin_1), R3.1, U1.2 (GND), U2.2 (GND), U3.1 (~{CS}), U3.4 (GND)
- net GND: now also C3.2, C4.1, R4.2; no longer C3.1, C4.2, R5.1
- net at Q1.1 (G), R3.2: now also R2.1; no longer R2.2
- net BAT+: now reaches Q1.2 (S)
- net BAT+: now also C1.1, J1.2 (Pin_2), R5.1, U2.1 (IN); no longer J2.2 (Pin_2)
- net BUS: now reaches J2.3 (Pin_3), U1.4 (B)
- net at A1.D1: no longer R2.1
- net A1: now reaches A1.A1, R5.2
- net A1: now also C3.1, R4.1; no longer C3.2, R4.2
- net 5V: now reaches A1.5V, U1.6 (V_{CCB})
- net 5V: now also C4.2; no longer C4.1
- net VIN: now reaches A1.VIN, C2.1, U2.3 (OUT)
- net at A1.D0: no longer U1.3 (A)
- net D2: now reaches A1.D2
- net D2: now also U1.3 (A)
- net D3: now reaches A1.D3
- net D3: now also R2.2
- new net SDI+: J2.2 (Pin_2), Q1.3 (D)
Other:
- moved on the sheet: A1, C1, C2, J1, J2, U1, U2, U3

Commit message: The Road to Calydon
Parts:
- added C6: 0.1uF, Capacitor_SMD:C_0603_1608Metric, symbol Device:C
- added R6, R7: 10k, Resistor_SMD:R_0603_1608Metric, symbol Device:R
- added U4: SHTC3, Sensor_Humidity:Sensirion_DFN-4-1EP_2x2mm_P1mm_EP0.7x1.6mm, symbol Sensor_Humidity:SHTC3
- C3: MPN 0.1uF 16V 0603 -> 0.1uF 6.3V 0603
Connections:
- net 3V3: now also C6.1, R6.2, R7.2, U4.1 (VDD)
- net BAT+: now also Q1.3 (D); no longer Q1.2 (S)
- net GND: now also C6.2, U4.4 (VSS)
- net SDI+: now also Q1.2 (S); no longer Q1.3 (D)
- net SDA: now reaches A1.D11 (D11/SDA)
- net SDA: now also R7.1, U4.3 (SDA)
- net SCL: now reaches A1.D12 (D12/SCL)
- net SCL: now also R6.1, U4.2 (SCL)
Other:
- note added: "DC DC CONVERTER 5V 3W"
- note added: "HUMIDITY/TEMPERATURE"
- note added: "MOSFET"
- note added: "SPI MEMORY"
- note added: "VOLTAGE DIVIDER 15V3 -> 3V3"
- note added: "VOLTAGE LEVEL-TRANSLATOR"

Commit message: Gladiator
Parts:
- removed A1: Arduino_MKR_NB_1500_Socket, Custom:Arduino_MKR_NB_1500_Socket, symbol PCM_arduino-library:Arduino_MKR_NB_1500_Socket
- added J3, J4: Conn_01x14_Socket, Custom:65342372, symbol Connector:Conn_01x14_Socket
Connections:
- net 3V3: now also J4.3 (Pin_3)
- net 5V: now also J4.1 (Pin_1)
- net A1: now also J3.3 (Pin_3)
- net D2: now also J3.11 (Pin_11)
- net D3: now also J3.12 (Pin_12)
- net GND: now also J4.4 (Pin_4)
- net SCL: now also J4.8 (Pin_8)
- net SDA: now also J4.9 (Pin_9)
- net VIN: now also J4.2 (Pin_2)
- net CIPO: now reaches U3.2 (DO(IO1))
- net CIPO: now also J4.10 (Pin_10)
- net COPI: now reaches U3.5 (DI(IO0))
- net COPI: now also J4.12 (Pin_12)
- net SCK: now reaches U3.6 (CLK)
- net SCK: now also J4.11 (Pin_11)

Commit message: The Festival of Dionysus
Connections:
- net D1: now reaches J3.10 (D1)
- net D1: now also U1.3 (A)
- net D0: now reaches J3.9 (D0)
- net D0: now also R2.2
- net D2: no longer names the net of J3.11 (~D2)
- net D2: no longer U1.3 (A)
- net D3: no longer names the net of J3.12 (~D3)
- net D3: no longer R2.2
Other:
- note added: "Arduino MKR NB 1500"
- moved on the sheet: U3

Commit message: The March to Freedom
Connections:
- net BAT+: now also J1.1 (Pin_1); no longer J1.2 (Pin_2)
- net BUS: now also J2.1 (Pin_1); no longer J2.3 (Pin_3)
- net GND: now also J1.2 (Pin_2), J2.3 (Pin_3); no longer J1.1 (Pin_1), J2.1 (Pin_1), U3.1 (~{CS})
- net D7: now reaches J4.13 (~D7)
- net D7: now also U3.1 (~{CS})
Changed lines of the file:
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@@
+	(wire
+		(pts
+			(xy 274.32 52.07) (xy 270.51 52.07)
+		)
+		(stroke
+			(width 0)
+			(type default)
+		)
+	)
 	(wire
 		(pts
@@
 	)
 	(rectangle
-		(start 246.38 19.05)
-		(end 267.97 57.15)
+		(start 247.65 20.32)
+		(end 266.7 55.88)
 		(stroke
 			(width 0)
@@
 		)
 	)
-	(label "GND"
+	(label "BAT+"
+		(at 33.02 35.56 0)
+		(fields_autoplaced yes)
+		(effects
+			(font
+				(size 1.27 1.27)
+			)
+			(justify left bottom)
+		)
+	)
+	(label "D7"
 		(at 181.61 81.28 0)
 		(fields_autoplaced yes)
@@
 		)
 	)
-	(label "GND"
-		(at 33.02 20.32 0)
-		(fields_autoplaced yes)
-		(effects
-			(font
-				(size 1.27 1.27)
-			)
-			(justify left bottom)
-		)
-	)
 	(label "SCL"
 		(at 38.1 158.75 0)
@@
 		)
 	)
-	(label "GND"
-		(at 33.02 35.56 0)
-		(fields_autoplaced yes)
-		(effects
-			(font
-				(size 1.27 1.27)
-			)
-			(justify left bottom)
-		)
-	)
 	(label "COPI"
 		(at 274.32 49.53 180)
@@
 		)
 	)
+	(label "GND"
+		(at 33.02 38.1 0)
+		(fields_autoplaced yes)
+		(effects
+			(font
+				(size 1.27 1.27)
+			)
+			(justify left bottom)
+		)
+	)
 	(label "5V"
 		(at 274.32 21.59 180)
@@
 		)
 	)
+	(label "BUS"
+		(at 33.02 20.32 0)
+		(fields_autoplaced yes)
+		(effects
+			(font
+				(size 1.27 1.27)
+			)
+			(justify left bottom)
+		)
+	)
+	(label "GND"
+		(at 33.02 25.4 0)
+		(fields_autoplaced yes)
+		(effects
+			(font
+				(size 1.27 1.27)
+			)
+			(justify left bottom)
+		)
+	)
 	(label "BAT+"
 		(at 25.4 83.82 0)
@@
 		)
 	)
-	(label "BUS"
-		(at 33.02 25.4 0)
-		(fields_autoplaced yes)
-		(effects
-			(font
-				(size 1.27 1.27)
-			)
-			(justify left bottom)
-		)
-	)
 	(label "CIPO"
 		(at 181.61 88.9 0)
@@
 		)
 	)
-	(label "BAT+"
-		(at 33.02 38.1 0)
-		(fields_autoplaced yes)
-		(effects
-			(font
-				(size 1.27 1.27)
-			)
-			(justify left bottom)
+	(label "D7"
+		(at 274.32 52.07 180)
+		(fields_autoplaced yes)
+		(effects
+			(font
+				(size 1.27 1.27)
+			)
+			(justify right bottom)
 		)
 	)
@@
 			)
 		)
-		(property "Datasheet" "~"
+		(property "Datasheet" "../../docs/1711039_07_en_03.pdf"
 			(at 17.78 22.86 0)
 			(effects
@@
 			)
 		)
-		(property "Datasheet" "http://www.winbond.com/resource-files/w25q32jv%20revg%2003272018%20plus.pdf"
+		(property "Datasheet" "../../docs/w25q32jv revg 03272018 plus.pdf"
 			(at 195.58 88.9 0)
 			(effects
@@
 			)
 		)
-		(property "Datasheet" "https://www.sensirion.com/fileadmin/user_upload/customers/sensirion/Dokumente/0_Datasheets/Humidity/Sensirion_Humidity_Sensors_SHTC3_Datasheet.pdf"
+		(property "Datasheet" "../../docs/Datasheet_SHTC3.pdf"
 			(at 52.07 149.86 0)
 			(effects
@@
 			)
 		)
-		(property "Datasheet" "https://www.recom-power.com/pdf/Innoline/R-78Exx-0.5.pdf"
+		(property "Datasheet" "../../docs/R-78E-0.5.pdf"
 			(at 127 34.29 0)
 			(effects
@@
 			)
 		)
-		(property "Datasheet" "~"
+		(property "Datasheet" "../../docs/1711026_07_en_04.pdf"
 			(at 17.78 35.56 0)
 			(effects
@@
 			)
 		)
-		(property "Datasheet" "~"
+		(property "Datasheet" "../../docs/ds_1307819_ampmodu_0911.pdf"
 			(at 248.92 36.83 0)
 			(effects
@@
 			)
 		)
-		(property "Datasheet" "https://www.ti.com/lit/ds/symlink/txs0101.pdf"
+		(property "Datasheet" "../../docs/txs0101.pdf"
 			(at 91.44 81.28 0)
 			(effects
@@
 			)
 		)
-		(property "Datasheet" "https://www.infineon.com/dgdl/Infineon-IRLML6244-DataSheet-v01_01-EN.pdf?fileId=5546d462533600a4015356686fed261f"
+		(property "Datasheet" "../../docs/Infineon-IRLML6244-DataSheet-v01_01-EN.pdf"
 			(at 132.08 129.54 0)
 			(effects
