File: kicad/Ryujin/Ryujin.kicad_sch (KiCad schematic)
At the start: 22 parts, among them J1 Screw_Terminal_01x06, J2 Conn_02x02_Odd_Even, J3 Conn_01x14_Socket, J4 Conn_01x14_Socket, Q1 IRLML6244, U1 74LVC1G17, U2 74AHCT1G14, U3 TMUX1119DBVR, U4 SHTC3, U5 W25Q32JVSS, U6 R-78E5.0-0.5

Commit message: Render Unto Caesar
Parts:
- added R1: 47k, Resistor_SMD:R_0603_1608Metric, symbol Device:R
Connections:
- net D1: now also R1.2
- net GND: now also R1.1
Changed lines of the file:
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@@
 	)
 	(junction
+		(at 142.24 95.25)
+		(diameter 0)
+		(color 0 0 0 0)
+	)
+	(junction
 		(at 173.99 30.48)
 		(diameter 0)
@@
 	)
 	(junction
+		(at 142.24 104.14)
+		(diameter 0)
+		(color 0 0 0 0)
+	)
+	(junction
 		(at 204.47 76.2)
 		(diameter 0)
@@
 	(wire
 		(pts
-			(xy 137.16 104.14) (xy 149.86 104.14)
+			(xy 137.16 104.14) (xy 142.24 104.14)
 		)
 		(stroke
@@
 	(wire
 		(pts
+			(xy 142.24 104.14) (xy 149.86 104.14)
+		)
+		(stroke
+			(width 0)
+			(type default)
+		)
+	)
+	(wire
+		(pts
 			(xy 97.79 38.1) (xy 116.84 38.1)
 		)
@@
 	(wire
 		(pts
+			(xy 142.24 95.25) (xy 142.24 96.52)
+		)
+		(stroke
+			(width 0)
+			(type default)
+		)
+	)
+	(wire
+		(pts
 			(xy 204.47 66.04) (xy 207.01 66.04)
 		)
@@
 	(wire
 		(pts
-			(xy 113.03 30.48) (xy 116.84 30.48)
+			(xy 137.16 127) (xy 137.16 130.81)
 		)
 		(stroke
@@
 	(wire
 		(pts
-			(xy 262.89 45.72) (xy 259.08 45.72)
+			(xy 113.03 30.48) (xy 116.84 30.48)
 		)
 		(stroke
@@
 	(wire
 		(pts
-			(xy 105.41 88.9) (xy 127 88.9)
+			(xy 262.89 45.72) (xy 259.08 45.72)
 		)
 		(stroke
@@
 	(wire
 		(pts
-			(xy 242.57 90.17) (xy 246.38 90.17)
+			(xy 105.41 88.9) (xy 127 88.9)
 		)
 		(stroke
@@
 	(wire
 		(pts
-			(xy 30.48 44.45) (xy 30.48 49.53)
+			(xy 242.57 90.17) (xy 246.38 90.17)
 		)
 		(stroke
@@
 	(wire
 		(pts
-			(xy 214.63 76.2) (xy 214.63 71.12)
+			(xy 30.48 44.45) (xy 30.48 49.53)
 		)
 		(stroke
@@
 	(wire
 		(pts
-			(xy 173.99 30.48) (xy 184.15 30.48)
+			(xy 214.63 76.2) (xy 214.63 71.12)
 		)
 		(stroke
@@
 	(wire
 		(pts
-			(xy 137.16 127) (xy 137.16 130.81)
+			(xy 173.99 30.48) (xy 184.15 30.48)
 		)
 		(stroke
@@
 	(wire
 		(pts
+			(xy 142.24 95.25) (xy 149.86 95.25)
+		)
+		(stroke
+			(width 0)
+			(type default)
+		)
+	)
+	(wire
+		(pts
 			(xy 30.48 44.45) (xy 34.29 44.45)
 		)
@@
 	(wire
 		(pts
-			(xy 146.05 99.06) (xy 149.86 99.06)
+			(xy 139.7 95.25) (xy 142.24 95.25)
 		)
 		(stroke
@@
 	(wire
 		(pts
-			(xy 142.24 101.6) (xy 149.86 101.6)
+			(xy 146.05 101.6) (xy 149.86 101.6)
 		)
 		(stroke
@@
 	(wire
 		(pts
+			(xy 149.86 95.25) (xy 149.86 99.06)
+		)
+		(stroke
+			(width 0)
+			(type default)
+		)
+	)
+	(wire
+		(pts
 			(xy 246.38 85.09) (xy 242.57 85.09)
 		)
@@
 		)
 	)
+	(label "D1"
+		(at 139.7 95.25 0)
+		(effects
+			(font
+				(size 1.27 1.27)
+			)
+			(justify left bottom)
+		)
+	)
 	(label "CIPO"
 		(at 262.89 48.26 180)
@@
 		)
 	)
-	(label "D1"
-		(at 146.05 99.06 0)
-		(effects
-			(font
-				(size 1.27 1.27)
-			)
-			(justify left bottom)
-		)
-	)
 	(label "COPI"
 		(at 262.89 53.34 180)
@@
 	)
 	(symbol
+		(lib_id "Device:R")
+		(at 142.24 100.33 180)
+		(unit 1)
+		(exclude_from_sim no)
+		(in_bom yes)
+		(on_board yes)
+		(dnp no)
+		(property "Reference" "R1"
+			(at 139.7 100.33 90)
+			(effects
+				(font
+					(size 1.27 1.27)
+				)
+			)
+		)
+		(property "Value" "47k"
+			(at 142.24 100.33 90)
+			(effects
+				(font
+					(size 1.27 1.27)
+				)
+			)
+		)
+		(property "Footprint" "Resistor_SMD:R_0603_1608Metric"
+			(at 144.018 100.33 90)
+			(effects
+				(font
+					(size 1.27 1.27)
+				)
+				(hide yes)
+			)
+		)
+		(property "Datasheet" "~"
+			(at 142.24 100.33 0)
+			(effects
+				(font
+					(size 1.27 1.27)
+				)
+				(hide yes)
+			)
+		)
+		(property "Description" "Resistor"
+			(at 142.24 100.33 0)
+			(effects
+				(font
+					(size 1.27 1.27)
+				)
+				(hide yes)
+			)
+		)
+		(property "MPN" "10k 0603"
+			(at 142.24 100.33 0)
+			(effects
+				(font
+					(size 1.27 1.27)
+				)
+				(hide yes)
+			)
+		)
+		(pin "2"
+		)
+		(pin "1"
+		)
+		(instances
+			(project "Ryujin"
+				(path "/a03941d3-2006-4bae-a82d-663063c77238"
+					(reference "R1")
+					(unit 1)
+				)
+			)
+		)
+	)
+	(symbol
 		(lib_id "Memory_Flash:W25Q32JVSS")
 		(at 256.54 90.17 0)
@@
 		(on_board yes)
 		(dnp no)
-		(fields_autoplaced yes)
 		(property "Reference" "R6"
-			(at 186.69 139.6999 0)
+			(at 186.69 142.494 90)
 			(effects
 				(font
@@
 		)
 		(property "Value" "10k"
-			(at 186.69 142.2399 0)
+			(at 184.15 142.494 90)
 			(effects
 				(font
@@
 		(on_board yes)
 		(dnp no)
-		(fields_autoplaced yes)
 		(property "Reference" "R3"
-			(at 207.01 69.8499 0)
+			(at 201.93 72.898 90)
 			(effects
 				(font
@@
 		)
 		(property "Value" "47k"
-			(at 207.01 72.3899 0)
+			(at 204.47 72.898 90)
 			(effects
 				(font
@@
 		(on_board yes)
 		(dnp no)
-		(fields_autoplaced yes)
 		(property "Reference" "R4"
-			(at 119.38 33.0199 0)
+			(at 119.38 36.576 90)
 			(effects
 				(font
@@
 		)
 		(property "Value" "330k"
-			(at 119.38 35.5599 0)
+			(at 116.84 36.576 90)
 			(effects
 				(font
@@
 		(on_board yes)
 		(dnp no)
-		(fields_autoplaced yes)
 		(property "Reference" "R7"
-			(at 172.72 142.2399 0)
+			(at 172.72 145.288 90)
 			(effects
 				(font
@@
 		)
 		(property "Value" "10k"
-			(at 172.72 144.7799 0)
+			(at 170.18 145.288 90)
 			(effects
 				(font
@@
 	(symbol
 		(lib_id "power:+5V")
-		(at 142.24 101.6 0)
+		(at 146.05 101.6 0)
 		(unit 1)
 		(exclude_from_sim no)
@@
 		(fields_autoplaced yes)
 		(property "Reference" "#PWR06"
-			(at 142.24 105.41 0)
+			(at 146.05 105.41 0)
 			(effects
 				(font
@@
 		)
 		(property "Value" "+5V"
-			(at 142.24 96.52 0)
+			(at 146.05 96.52 0)
 			(effects
 				(font
@@
 		)
 		(property "Footprint" ""
-			(at 142.24 101.6 0)
+			(at 146.05 101.6 0)
 			(effects
 				(font
@@
 		)
 		(property "Datasheet" ""
-			(at 142.24 101.6 0)
+			(at 146.05 101.6 0)
 			(effects
 				(font
@@
 		)
 		(property "Description" "Power symbol creates a global label with name \"+5V\""
-			(at 142.24 101.6 0)
+			(at 146.05 101.6 0)
 			(effects
 				(font
@@
 		(on_board yes)
 		(dnp no)
-		(fields_autoplaced yes)
 		(property "Reference" "R2"
-			(at 198.12 59.69 90)
+			(at 198.12 63.5 90)
 			(effects
 				(font
@@
 		)
 		(property "Value" "100"
-			(at 198.12 62.23 90)
+			(at 198.12 66.04 90)
 			(effects
 				(font
@@
 		(dnp no)
 		(property "Reference" "R5"
-			(at 109.22 24.13 90)
+			(at 109.22 27.94 90)
 			(effects
 				(font
@@
 		)
 		(property "Value" "1.2M"
-			(at 109.22 26.67 90)
+			(at 109.22 30.48 90)
 			(effects
 				(font

Commit message: Norse by Norsevest
Parts:
- removed J1: Screw_Terminal_01x06, ThirdParty:SMKDSN-1-5-6-5-08_3D, symbol Connector:Screw_Terminal_01x06
- added J1: 1704376, footprints:FFKDSA1_508_3, symbol PhoenixContact:1704376
- added J6: 1789210, footprints:FFKDSA1_508_2, symbol PhoenixContact:1789210
- J3, J4: footprint Custom:65342372 -> footprints:65342372
- R1: value 47k -> 3k3; MPN 10k 0603 -> 3.3k 0603
- R3: value 47k -> 33k; MPN 47k 0603 -> 33k 0603
Connections:
- net +12V: now also J1.B2, J6.2 (1.2)
- net -12V: now also J1.B1
- net GND: now also J6.4 (2.2)
- net LINE: now also J1.B3
- no-connect marks 15 -> 19

Commit message: For Those of You Just Joining Us
Parts:
- removed J1: 1704376, footprints:FFKDSA1_508_3, symbol PhoenixContact:1704376
- removed J6: 1789210, footprints:FFKDSA1_508_2, symbol PhoenixContact:1789210
- added J1: 1869211, footprints:SMKDSN_508_2, symbol PhoenixContact:1869211
- added J5: 1869224, footprints:SMKDSN_508_3, symbol PhoenixContact:1869224
Connections:
- net +12V: now also J1.1, J5.2
- net -12V: now also J5.3
- net GND: now also J1.2
- net LINE: now also J5.1
- no-connect marks 19 -> 14

Commit message: Let There Be Light
Parts:
- removed J1: 1869211, footprints:SMKDSN_508_2, symbol PhoenixContact:1869211
- removed J5: 1869224, footprints:SMKDSN_508_3, symbol PhoenixContact:1869224
- added J1: SMKDSN_6_508, footprints:SMKDSN_508_6, symbol PhoenixContact:SMKDSN_6_508
Connections:
- net +12V: now also J1.3, J1.5
- net -12V: now also J1.2
- net GND: now also J1.6
- net LINE: now also J1.1

Commit message: Sky High
Parts:
- added J5: Conn_01x03_Pin, Connector_Molex:Molex_KK-254_AE-6410-03A_1x03_P2.54mm_Vertical, symbol Connector:Conn_01x03_Pin
Changed lines of the file:
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@@
+	)
+	(symbol
+		(lib_id "Connector:Conn_01x03_Pin")
+		(at 36.83 45.72 0)
+		(unit 1)
+		(exclude_from_sim no)
+		(in_bom yes)
+		(on_board yes)
+		(dnp no)
+		(fields_autoplaced yes)
+		(property "Reference" "J5"
+			(at 37.465 38.1 0)
+			(effects
+				(font
+					(size 1.27 1.27)
+				)
+			)
+		)
+		(property "Value" "Conn_01x03_Pin"
+			(at 37.465 40.64 0)
+			(effects
+				(font
+					(size 1.27 1.27)
+				)
+			)
+		)
+		(property "Footprint" "Connector_Molex:Molex_KK-254_AE-6410-03A_1x03_P2.54mm_Vertical"
+			(at 36.83 45.72 0)
+			(effects
+				(font
+					(size 1.27 1.27)
+				)
+				(hide yes)
+			)
+		)
+		(property "Datasheet" "~"
+			(at 36.83 45.72 0)
+			(effects
+				(font
+					(size 1.27 1.27)
+				)
+				(hide yes)
+			)
+		)
+		(property "Description" "Generic connector, single row, 01x03, script generated"
+			(at 36.83 45.72 0)
+			(effects
+				(font
+					(size 1.27 1.27)
+				)
+				(hide yes)
+			)
+		)
+		(pin "2"
+		)
+		(pin "1"
+		)
+		(pin "3"
+		)
+		(instances
+			(project ""
+				(path "/a03941d3-2006-4bae-a82d-663063c77238"
+					(reference "J5")
+					(unit 1)
+				)
+			)
+		)
 	)
 	(symbol

Commit message: Stranger and Stranger
Parts:
- removed J1: SMKDSN_6_508, footprints:SMKDSN_508_6, symbol PhoenixContact:SMKDSN_6_508
- J5: footprint Connector_Molex:Molex_KK-254_AE-6410-03A_1x03_P2.54mm_Vertical -> footprints:GROVE-HW4-2.0; MPN (none) -> 1125S-4P
Connections:
- net +12V: now also J5.2 (Pin_2)
- net -12V: now also J5.3 (Pin_3)
- net LINE: now also J5.1 (Pin_1)
Other:
- moved on the sheet: J5

Commit message: ...and Fancy Free
Parts:
- J5: MPN 1125S-4P -> 110990030
Changed lines of the file:
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@@
 (kicad_sch
-	(version 20231120)
+	(version 20250114)
 	(generator "eeschema")
-	(generator_version "8.0")
+	(generator_version "9.0")
 	(paper "A4")
 	(title_block
@@
 		(company "Julius-Maximilians-Universität Würzburg")
 	)
+	(rectangle
+		(start 236.22 24.13)
+		(end 255.27 59.69)
+		(stroke
+			(width 0)
+			(type default)
+			(color 132 0 0 1)
+		)
+		(fill
+			(type color)
+			(color 255 255 194 1)
+		)
+	)
+	(text "HUMIDITY/TEMPERATURE"
+		(exclude_from_sim no)
+		(at 179.324 129.794 0)
+		(effects
+			(font
+				(size 1.27 1.27)
+			)
+			(justify left)
+		)
+	)
+	(text "VOLTAGE LEVEL-TRANSLATOR"
+		(exclude_from_sim no)
+		(at 138.176 65.532 0)
+		(effects
+			(font
+				(size 1.27 1.27)
+			)
+			(justify left)
+		)
+	)
+	(text "VOLTAGE DIVIDER 15V3 -> 3V3"
+		(exclude_from_sim no)
+		(at 101.346 21.082 0)
+		(effects
+			(font
+				(size 1.27 1.27)
+			)
+			(justify left)
+		)
+	)
+	(text "SPI MEMORY"
+		(exclude_from_sim no)
+		(at 262.128 73.66 0)
+		(effects
+			(font
+				(size 1.27 1.27)
+			)
+			(justify left)
+		)
+	)
+	(text "Arduino MKR NB 1500"
+		(exclude_from_sim no)
+		(at 245.872 21.59 0)
+		(effects
+			(font
+				(size 1.27 1.27)
+			)
+		)
+	)
+	(text "DC DC CONVERTER 5V 3W"
+		(exclude_from_sim no)
+		(at 178.562 18.542 0)
+		(effects
+			(font
+				(size 1.27 1.27)
+			)
+			(justify left)
+		)
+	)
+	(text "MOSFET"
+		(exclude_from_sim no)
+		(at 200.406 52.832 0)
+		(effects
+			(font
+				(size 1.27 1.27)
+			)
+			(justify left)
+		)
+	)
 	(junction
 		(at 137.16 104.14)
@@
 		)
 	)
-	(rectangle
-		(start 236.22 24.13)
-		(end 255.27 59.69)
-		(stroke
-			(width 0)
-			(type default)
-			(color 132 0 0 1)
-		)
-		(fill
-			(type color)
-			(color 255 255 194 1)
-		)
-	)
-	(text "HUMIDITY/TEMPERATURE"
-		(exclude_from_sim no)
-		(at 179.324 129.794 0)
-		(effects
-			(font
-				(size 1.27 1.27)
-			)
-			(justify left)
-		)
-	)
-	(text "VOLTAGE LEVEL-TRANSLATOR"
-		(exclude_from_sim no)
-		(at 138.176 65.532 0)
-		(effects
-			(font
-				(size 1.27 1.27)
-			)
-			(justify left)
-		)
-	)
-	(text "VOLTAGE DIVIDER 15V3 -> 3V3"
-		(exclude_from_sim no)
-		(at 101.346 21.082 0)
-		(effects
-			(font
-				(size 1.27 1.27)
-			)
-			(justify left)
-		)
-	)
-	(text "SPI MEMORY"
-		(exclude_from_sim no)
-		(at 262.128 73.66 0)
-		(effects
-			(font
-				(size 1.27 1.27)
-			)
-			(justify left)
-		)
-	)
-	(text "Arduino MKR NB 1500"
-		(exclude_from_sim no)
-		(at 245.872 21.59 0)
-		(effects
-			(font
-				(size 1.27 1.27)
-			)
-		)
-	)
-	(text "DC DC CONVERTER 5V 3W"
-		(exclude_from_sim no)
-		(at 178.562 18.542 0)
-		(effects
-			(font
-				(size 1.27 1.27)
-			)
-			(justify left)
-		)
-	)
-	(text "MOSFET"
-		(exclude_from_sim no)
-		(at 200.406 52.832 0)
-		(effects
-			(font
-				(size 1.27 1.27)
-			)
-			(justify left)
-		)
-	)
 	(label "SCK"
 		(at 262.89 50.8 180)
@@
 			)
 		)
-		(property "MPN" "1125S-4P"
+		(property "MPN" "110990030"
 			(at 33.02 52.07 0)
 			(effects
@@
 		)
 	)
+	(embedded_fonts no)
 )

Commit message: Love on the Rocks
Parts:
- removed J5: Conn_01x03_Pin, footprints:GROVE-HW4-2.0, symbol Connector:Conn_01x03_Pin
- added J1: Screw_Terminal_01x02, TerminalBlock_Phoenix:TerminalBlock_Phoenix_MKDS-1,5-2-5.08_1x02_P5.08mm_Horizontal, symbol Connector:Screw_Terminal_01x02
- added J5: Conn_01x04_Pin, footprints:GROVE-HW4-2.0, symbol Connector:Conn_01x04_Pin
Connections:
- net +12V: now also J1.2 (Pin_2), J5.2 (Pin_2)
- net -12V: now also J5.3 (Pin_3)
- net GND: now also J1.1 (Pin_1)
- net LINE: now also J5.1 (Pin_1)
- no-connect marks 14 -> 15
