File: kicad/Ryujin/Ryujin.kicad_sch (KiCad schematic)
At the start: 34 parts, among them J1 Conn_01x02_Socket, J10 Conn_01x04_Pin, J11 Conn_01x04_Pin, J12 Conn_01x04_Pin, J2 1822972, J3 Conn_01x14_Socket, J4 Conn_01x14_Socket, J5 1822972, J6 Conn_01x04_Pin, J7 Conn_01x04_Pin, J8 Conn_01x04_Pin, J9 Conn_01x04_Pin, Q1 IRLML5203, Q2 IRLML6244, U1 74LVC1G17, U2 74AHCT1G14, U3 TMUX1119DBVR, U4 SHTC3, U5 W25Q32JVSS, U7 R-78E5.0-1.0

Commit message: Is There a Doctor in the House?
Connections:
- no-connect marks 18 -> 19
Other:
- sheet Battery Charger ports: added CE; removed none
Changed lines of the file:
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@@
 	)
 	(no_connect
+		(at 21.59 21.59)
+	)
+	(no_connect
 		(at 259.08 38.1)
 	)
@@
 	(wire
 		(pts
-			(xy 21.59 36.83) (xy 21.59 24.13)
+			(xy 21.59 36.83) (xy 21.59 26.67)
 		)
 		(stroke
@@
 	(wire
 		(pts
+			(xy 21.59 21.59) (xy 25.4 21.59)
+		)
+		(stroke
+			(width 0)
+			(type default)
+		)
+	)
+	(wire
+		(pts
 			(xy 62.23 30.48) (xy 55.88 30.48)
 		)
@@
 	(wire
 		(pts
-			(xy 21.59 24.13) (xy 25.4 24.13)
+			(xy 21.59 26.67) (xy 25.4 26.67)
 		)
 		(stroke
@@
 		)
 		(pin "TS" output
-			(at 25.4 24.13 180)
+			(at 25.4 26.67 180)
+			(effects
+				(font
+					(size 1.27 1.27)
+				)
+				(justify left)
+			)
+		)
+		(pin "CE" input
+			(at 25.4 21.59 180)
 			(effects
 				(font

Commit message: Orphan of War
Parts:
- added D8: D1, footprints:PDS104013, symbol Device:D_AAK
Connections:
- net +12V: now also D8.1 (A), D8.2 (A); no longer C1.1, U7.1 (IN)
- net D5: now reaches J3.14 (~D5)
- new net: C1.1, D8.3 (K), U7.1 (IN)
- no-connect marks 19 -> 17
Other:
- moved on the sheet: C1, C2, U7

Commit message: A Tale of Two Muses
Parts:
- removed D8: D1, footprints:PDS104013, symbol Device:D_AAK
- added D8: D2, Package_TO_SOT_SMD:SOT-23, symbol Diode:BAT54W
Connections:
- net +12V: now also D8.1 (A)
- net at C1.1, U7.1 (IN): now also D8.3 (K)
Changed lines of the file:
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@@
 	)
 	(junction
-		(at 129.54 30.48)
-		(diameter 0)
-		(color 0 0 0 0)
-	)
-	(junction
 		(at 224.79 138.43)
 		(diameter 0)
@@
 	(wire
 		(pts
-			(xy 129.54 30.48) (xy 129.54 33.02)
-		)
-		(stroke
-			(width 0)
-			(type default)
-		)
-	)
-	(wire
-		(pts
 			(xy 50.8 29.21) (xy 50.8 26.67)
 		)
@@
 	(wire
 		(pts
-			(xy 120.65 30.48) (xy 129.54 30.48)
+			(xy 120.65 30.48) (xy 130.81 30.48)
 		)
 		(stroke
@@
 	)
 	(symbol
-		(lib_id "Device:D_AAK")
-		(at 134.62 30.48 180)
-		(unit 1)
-		(exclude_from_sim no)
-		(in_bom yes)
-		(on_board yes)
-		(dnp no)
-		(fields_autoplaced yes)
-		(property "Reference" "D8"
-			(at 133.4135 24.13 0)
-			(effects
-				(font
-					(size 1.27 1.27)
-				)
-				(hide yes)
-			)
-		)
-		(property "Value" "D1"
-			(at 133.4135 26.67 0)
-			(effects
-				(font
-					(size 1.27 1.27)
-				)
-			)
-		)
-		(property "Footprint" "footprints:PDS104013"
-			(at 134.62 30.48 0)
-			(effects
-				(font
-					(size 1.27 1.27)
-				)
-				(hide yes)
-			)
-		)
-		(property "Datasheet" "../../docs/PDS1040.pdf"
-			(at 134.62 30.48 0)
-			(effects
-				(font
-					(size 1.27 1.27)
-				)
-				(hide yes)
-			)
-		)
-		(property "Description" "Diode, anode on pins 1 and 2"
-			(at 134.62 30.48 0)
-			(effects
-				(font
-					(size 1.27 1.27)
-				)
-				(hide yes)
-			)
-		)
-		(property "MPN" "PDS1040-13"
-			(at 134.62 30.48 0)
-			(effects
-				(font
-					(size 1.27 1.27)
-				)
-				(hide yes)
-			)
-		)
-		(pin "3"
-		)
-		(pin "2"
-		)
-		(pin "1"
-		)
-		(instances
-			(project "Ryujin"
-				(path "/a03941d3-2006-4bae-a82d-663063c77238"
-					(reference "D8")
-					(unit 1)
-				)
-			)
-		)
-	)
-	(symbol
 		(lib_id "power:GND")
 		(at 177.8 92.71 0)
@@
 					(unit 1)
 				)
+			)
+		)
+	)
+	(symbol
+		(lib_id "Diode:BAT54W")
+		(at 134.62 30.48 180)
+		(unit 1)
+		(exclude_from_sim no)
+		(in_bom yes)
+		(on_board yes)
+		(dnp no)
+		(fields_autoplaced yes)
+		(property "Reference" "D8"
+			(at 136.2076 33.02 90)
+			(effects
+				(font
+					(size 1.27 1.27)
+				)
+				(justify left)
+				(hide yes)
+			)
+		)
+		(property "Value" "D2"
+			(at 134.9375 26.67 0)
+			(effects
+				(font
+					(size 1.27 1.27)
+				)
+			)
+		)
+		(property "Footprint" "Package_TO_SOT_SMD:SOT-23"
+			(at 134.62 26.035 0)
+			(effects
+				(font
+					(size 1.27 1.27)
+				)
+				(hide yes)
+			)
+		)
+		(property "Datasheet" "https://assets.nexperia.com/documents/data-sheet/BAT54W_SER.pdf"
+			(at 134.62 30.48 0)
+			(effects
+				(font
+					(size 1.27 1.27)
+				)
+				(hide yes)
+			)
+		)
+		(property "Description" "Schottky barrier diode"
+			(at 134.62 30.48 0)
+			(effects
+				(font
+					(size 1.27 1.27)
+				)
+				(hide yes)
+			)
+		)
+		(property "MPN" " BAT54"
+			(at 134.62 30.48 90)
+			(effects
+				(font
+					(size 1.27 1.27)
+				)
+				(hide yes)
+			)
+		)
+		(pin "1"
+		)
+		(pin "2"
+		)
+		(pin "3"
+		)
+		(instances
+			(project "Ryujin"
+				(path "/a03941d3-2006-4bae-a82d-663063c77238"
+					(reference "D8")
+					(unit 1)
+				)

Commit message: Past Imperfect
Parts:
- removed D8: D2, Package_TO_SOT_SMD:SOT-23, symbol Diode:BAT54W
- added D1: SS34, Diode_SMD:D_SMA, symbol Diode:SS34
Connections:
- net +12V: now also D1.2 (A)
- net at C1.1, U7.1 (IN): now also D1.1 (K)
Changed lines of the file:
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@@
-	)
-	(symbol
-		(lib_id "Diode:BAT54W")
-		(at 134.62 30.48 180)
-		(unit 1)
-		(exclude_from_sim no)
-		(in_bom yes)
-		(on_board yes)
-		(dnp no)
-		(fields_autoplaced yes)
-		(property "Reference" "D8"
-			(at 136.2076 33.02 90)
-			(effects
-				(font
-					(size 1.27 1.27)
-				)
-				(justify left)
-				(hide yes)
-			)
-		)
-		(property "Value" "D2"
-			(at 134.9375 26.67 0)
-			(effects
-				(font
-					(size 1.27 1.27)
-				)
-			)
-		)
-		(property "Footprint" "Package_TO_SOT_SMD:SOT-23"
-			(at 134.62 26.035 0)
-			(effects
-				(font
-					(size 1.27 1.27)
-				)
-				(hide yes)
-			)
-		)
-		(property "Datasheet" "https://assets.nexperia.com/documents/data-sheet/BAT54W_SER.pdf"
-			(at 134.62 30.48 0)
-			(effects
-				(font
-					(size 1.27 1.27)
-				)
-				(hide yes)
-			)
-		)
-		(property "Description" "Schottky barrier diode"
-			(at 134.62 30.48 0)
-			(effects
-				(font
-					(size 1.27 1.27)
-				)
-				(hide yes)
-			)
-		)
-		(property "MPN" " BAT54"
-			(at 134.62 30.48 90)
-			(effects
-				(font
-					(size 1.27 1.27)
-				)
-				(hide yes)
-			)
-		)
-		(pin "1"
-		)
-		(pin "2"
-		)
-		(pin "3"
-		)
-		(instances
-			(project "Ryujin"
-				(path "/a03941d3-2006-4bae-a82d-663063c77238"
-					(reference "D8")
-					(unit 1)
-				)
-			)
-		)
 	)
 	(symbol
@@
 					(unit 1)
 				)
+			)
+		)
+	)
+	(symbol
+		(lib_id "Diode:SS34")
+		(at 134.62 30.48 180)
+		(unit 1)
+		(exclude_from_sim no)
+		(in_bom yes)
+		(on_board yes)
+		(dnp no)
+		(fields_autoplaced yes)
+		(property "Reference" "D1"
+			(at 134.9375 24.13 0)
+			(effects
+				(font
+					(size 1.27 1.27)
+				)
+			)
+		)
+		(property "Value" "SS34"
+			(at 134.9375 26.67 0)
+			(effects
+				(font
+					(size 1.27 1.27)
+				)
+			)
+		)
+		(property "Footprint" "Diode_SMD:D_SMA"
+			(at 134.62 26.035 0)
+			(effects
+				(font
+					(size 1.27 1.27)
+				)
+				(hide yes)
+			)
+		)
+		(property "Datasheet" "https://www.vishay.com/docs/88751/ss32.pdf"
+			(at 134.62 30.48 0)
+			(effects
+				(font
+					(size 1.27 1.27)
+				)
+				(hide yes)
+			)
+		)
+		(property "Description" "40V 3A Schottky Diode, SMA"
+			(at 134.62 30.48 0)
+			(effects
+				(font
+					(size 1.27 1.27)
+				)
+				(hide yes)
+			)
+		)
+		(pin "2"
+		)
+		(pin "1"
+		)
+		(instances
+			(project ""
+				(path "/a03941d3-2006-4bae-a82d-663063c77238"
+					(reference "D1")
+					(unit 1)
+				)

Commit message: The Convert
Parts:
- removed U5: W25Q32JVSS, Package_SO:SOIC-8_5.23x5.23mm_P1.27mm, symbol Memory_Flash:W25Q32JVSS
- added U5: W25Q128JVS, Package_SO:SOIC-8_5.3x5.3mm_P1.27mm, symbol Memory_Flash:W25Q128JVS
Connections:
- net +3.3V: now also U5.3 (~{WP}/IO_{2}), U5.7 (~{HOLD}/~{RESET}/IO_{3}), U5.8 (VCC)
- net CIPO: now also U5.2 (DO/IO_{1})
- net COPI: now also U5.5 (DI/IO_{0})
- net D7: now also U5.1 (~{CS})
- net GND: now also U5.4 (GND)
- net SCK: now also U5.6 (CLK)
Changed lines of the file:
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@@
-	)
-	(symbol
-		(lib_id "Memory_Flash:W25Q32JVSS")
-		(at 43.18 152.4 0)
-		(unit 1)
-		(exclude_from_sim no)
-		(in_bom yes)
-		(on_board yes)
-		(dnp no)
-		(fields_autoplaced yes)
-		(property "Reference" "U5"
-			(at 52.07 151.1299 0)
-			(effects
-				(font
-					(size 1.27 1.27)
-				)
-				(justify left)
-			)
-		)
-		(property "Value" "W25Q32JVSS"
-			(at 52.07 153.6699 0)
-			(effects
-				(font
-					(size 1.27 1.27)
-				)
-				(justify left)
-			)
-		)
-		(property "Footprint" "Package_SO:SOIC-8_5.23x5.23mm_P1.27mm"
-			(at 43.18 152.4 0)
-			(effects
-				(font
-					(size 1.27 1.27)
-				)
-				(hide yes)
-			)
-		)
-		(property "Datasheet" "../../docs/w25q32jv revg 03272018 plus.pdf"
-			(at 43.18 152.4 0)
-			(effects
-				(font
-					(size 1.27 1.27)
-				)
-				(hide yes)
-			)
-		)
-		(property "Description" "32Mb Serial Flash Memory, Standard/Dual/Quad SPI, SOIC-8"
-			(at 43.18 152.4 0)
-			(effects
-				(font
-					(size 1.27 1.27)
-				)
-				(hide yes)
-			)
-		)
-		(property "MPN" "W25Q32JVSSIQ TR"
-			(at 43.18 152.4 0)
-			(effects
-				(font
-					(size 1.27 1.27)
-				)
-				(hide yes)
-			)
-		)
-		(pin "4"
-		)
-		(pin "3"
-		)
-		(pin "7"
-		)
-		(pin "8"
-		)
-		(pin "5"
-		)
-		(pin "2"
-		)
-		(pin "6"
-		)
-		(pin "1"
-		)
-		(instances
-			(project ""
-				(path "/a03941d3-2006-4bae-a82d-663063c77238"
-					(reference "U5")
-					(unit 1)
-				)
-			)
-		)
 	)
 	(symbol
@@
 					(unit 1)
 				)
+			)
+		)
+	)
+	(symbol
+		(lib_id "Memory_Flash:W25Q128JVS")
+		(at 43.18 152.4 0)
+		(unit 1)
+		(exclude_from_sim no)
+		(in_bom yes)
+		(on_board yes)
+		(dnp no)
+		(fields_autoplaced yes)
+		(property "Reference" "U5"
+			(at 54.61 151.1299 0)
+			(effects
+				(font
+					(size 1.27 1.27)
+				)
+				(justify left)
+			)
+		)
+		(property "Value" "W25Q128JVS"
+			(at 54.61 153.6699 0)
+			(effects
+				(font
+					(size 1.27 1.27)
+				)
+				(justify left)
+			)
+		)
+		(property "Footprint" "Package_SO:SOIC-8_5.3x5.3mm_P1.27mm"
+			(at 43.18 129.54 0)
+			(effects
+				(font
+					(size 1.27 1.27)
+				)
+				(hide yes)
+			)
+		)
+		(property "Datasheet" "https://www.winbond.com/resource-files/w25q128jv_dtr%20revc%2003272018%20plus.pdf"
+			(at 43.18 127 0)
+			(effects
+				(font
+					(size 1.27 1.27)
+				)
+				(hide yes)
+			)
+		)
+		(property "Description" "128Mbit / 16MiB Serial Flash Memory, Standard/Dual/Quad SPI, 2.7-3.6V, SOIC-8"
+			(at 43.18 124.46 0)
+			(effects
+				(font
+					(size 1.27 1.27)
+				)
+				(hide yes)
+			)
+		)
+		(property "MPN" "W25Q128JVSIQ TR"
+			(at 43.18 152.4 0)
+			(effects
+				(font
+					(size 1.27 1.27)
+				)
+				(hide yes)
+			)
+		)
+		(pin "3"
+		)
+		(pin "2"
+		)
+		(pin "5"
+		)
+		(pin "7"
+		)
+		(pin "6"
+		)
+		(pin "1"
+		)
+		(pin "8"
+		)
+		(pin "4"
+		)
+		(instances
+			(project ""
+				(path "/a03941d3-2006-4bae-a82d-663063c77238"
+					(reference "U5")
+					(unit 1)
+				)

Commit message: God Fearing Child
Parts:
- removed D1: SS34, Diode_SMD:D_SMA, symbol Diode:SS34
- added D1: D_Zener, Diode_SMD:D_0805_2012Metric, symbol Device:D_Zener
- added Q5: IRLML5203, Package_TO_SOT_SMD:SOT-23, symbol Transistor_FET:IRLML5203
- added R11: 127k, Resistor_SMD:R_0603_1608Metric, symbol Device:R
Connections:
- net +12V: now also Q5.2 (S), R11.2
- net GND: now also D1.2 (A)
- net at C1.1, U7.1 (IN): now also Q5.3 (D)
- new net: D1.1 (K), Q5.1 (G), R11.1

Commit message: Eternal Bonds
Parts:
- added Q6: IRLML5203, Package_TO_SOT_SMD:SOT-23, symbol Transistor_FET:IRLML5203
Connections:
- net +12V: now also Q6.2 (S), Q6.3 (D)
- net at D1.1 (K), Q5.1 (G), R11.1: now also Q6.1 (G)
Other:
- moved on the sheet: R11
Changed lines of the file:
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@@
 	)
 	(junction
+		(at 105.41 30.48)
+		(diameter 0)
+		(color 0 0 0 0)
+	)
+	(junction
 		(at 248.92 114.3)
 		(diameter 0)
@@
 	)
 	(junction
+		(at 113.03 30.48)
+		(diameter 0)
+		(color 0 0 0 0)
+	)
+	(junction
+		(at 123.19 30.48)
+		(diameter 0)
+		(color 0 0 0 0)
+	)
+	(junction
 		(at 256.54 156.21)
 		(diameter 0)
@@
 	)
 	(junction
-		(at 121.92 30.48)
+		(at 118.11 39.37)
 		(diameter 0)
 		(color 0 0 0 0)
@@
 	(wire
 		(pts
-			(xy 121.92 39.37) (xy 121.92 30.48)
-		)
-		(stroke
-			(width 0)
-			(type default)
-		)
-	)
-	(wire
-		(pts
-			(xy 123.19 39.37) (xy 121.92 39.37)
-		)
-		(stroke
-			(width 0)
-			(type default)
-		)
-	)
-	(wire
-		(pts
 			(xy 170.18 30.48) (xy 175.26 30.48)
 		)
@@
 	(wire
 		(pts
-			(xy 121.92 30.48) (xy 128.27 30.48)
-		)
-		(stroke
-			(width 0)
-			(type default)
-		)
-	)
-	(wire
-		(pts
 			(xy 50.8 29.21) (xy 50.8 26.67)
 		)
@@
 	(wire
 		(pts
+			(xy 123.19 30.48) (xy 128.27 30.48)
+		)
+		(stroke
+			(width 0)
+			(type default)
+		)
+	)
+	(wire
+		(pts
 			(xy 133.35 46.99) (xy 144.78 46.99)
 		)
@@
 	(wire
 		(pts
+			(xy 118.11 38.1) (xy 118.11 39.37)
+		)
+		(stroke
+			(width 0)
+			(type default)
+		)
+	)
+	(wire
+		(pts
 			(xy 127.9829 139.7) (xy 147.0329 139.7)
 		)
@@
 	(wire
 		(pts
+			(xy 113.03 30.48) (xy 123.19 30.48)
+		)
+		(stroke
+			(width 0)
+			(type default)
+		)
+	)
+	(wire
+		(pts
 			(xy 62.23 30.48) (xy 55.88 30.48)
 		)
@@
 	(wire
 		(pts
-			(xy 118.11 30.48) (xy 121.92 30.48)
+			(xy 271.78 138.43) (xy 256.54 138.43)
 		)
 		(stroke
@@
 	(wire
 		(pts
-			(xy 271.78 138.43) (xy 256.54 138.43)
+			(xy 105.41 30.48) (xy 113.03 30.48)
 		)
 		(stroke
@@
 	(wire
 		(pts
+			(xy 102.87 30.48) (xy 105.41 30.48)
+		)
+		(stroke
+			(width 0)
+			(type default)
+		)
+	)
+	(wire
+		(pts
 			(xy 44.45 64.77) (xy 66.04 64.77)
 		)
@@
 	(wire
 		(pts
+			(xy 118.11 39.37) (xy 133.35 39.37)
+		)
+		(stroke
+			(width 0)
+			(type default)
+		)
+	)
+	(wire
+		(pts
 			(xy 21.59 26.67) (xy 25.4 26.67)
 		)
@@
 	(wire
 		(pts
-			(xy 130.81 39.37) (xy 133.35 39.37)
+			(xy 113.03 39.37) (xy 118.11 39.37)
 		)
 		(stroke
@@
 	(wire
 		(pts
+			(xy 105.41 30.48) (xy 105.41 39.37)
+		)
+		(stroke
+			(width 0)
+			(type default)
+		)
+	)
+	(wire
+		(pts
 			(xy 198.12 78.74) (xy 198.12 81.28)
 		)
@@
 	)
 	(symbol
+		(lib_id "Transistor_FET:IRLML5203")
+		(at 118.11 33.02 90)
+		(unit 1)
+		(exclude_from_sim no)
+		(in_bom yes)
+		(on_board yes)
+		(dnp no)
+		(property "Reference" "Q6"
+			(at 123.19 23.368 90)
+			(effects
+				(font
+					(size 1.27 1.27)
+				)
+				(justify left)
+			)
+		)
+		(property "Value" "IRLML5203"
+			(at 123.19 25.908 90)
+			(effects
+				(font
+					(size 1.27 1.27)
+				)
+				(justify left)
+			)
+		)
+		(property "Footprint" "Package_TO_SOT_SMD:SOT-23"
+			(at 120.015 27.94 0)
+			(effects
+				(font
+					(size 1.27 1.27)
+					(italic yes)
+				)
+				(justify left)
+				(hide yes)
+			)
+		)
+		(property "Datasheet" "../../docs/Infineon-IRLML5203-DataSheet-v01_01-EN.pdf"
+			(at 121.92 27.94 0)
+			(effects
+				(font
+					(size 1.27 1.27)
+				)
+				(justify left)
+				(hide yes)
+			)
+		)
+		(property "Description" "-3.0A Id, -30V Vds, 98mOhm Rds, P-Channel HEXFET Power MOSFET, SOT-23"
+			(at 118.11 33.02 0)
+			(effects
+				(font
+					(size 1.27 1.27)
+				)
+				(hide yes)
+			)
+		)
+		(property "MPN" "IRLML5203TRPBF"
+			(at 118.11 33.02 0)
+			(effects
+				(font
+					(size 1.27 1.27)
+				)
+				(hide yes)
+			)
+		)
+		(pin "1"
+		)
+		(pin "2"
+		)
+		(pin "3"
+		)
+		(instances
+			(project "Ryujin"
+				(path "/a03941d3-2006-4bae-a82d-663063c77238"
+					(reference "Q6")
+					(unit 1)
+				)
+			)
+		)
+	)
+	(symbol
 		(lib_id "Connector:Conn_01x04_Pin")
 		(at 122.9029 134.62 0)
@@
 	(symbol
 		(lib_id "power:+12V")
-		(at 118.11 30.48 0)
+		(at 102.87 30.48 0)
 		(unit 1)
 		(exclude_from_sim no)
@@
 		(fields_autoplaced yes)
 		(property "Reference" "#PWR08"
-			(at 118.11 34.29 0)
+			(at 102.87 34.29 0)
 			(effects
 				(font
@@
 		)
 		(property "Value" "+12V"
-			(at 118.11 25.4 0)
+			(at 102.87 25.4 0)
 			(effects
 				(font
@@
 		)
 		(property "Footprint" ""
-			(at 118.11 30.48 0)
+			(at 102.87 30.48 0)
 			(effects
 				(font
@@
 		)
 		(property "Datasheet" ""
-			(at 118.11 30.48 0)
+			(at 102.87 30.48 0)
 			(effects
 				(font
@@
 		)
 		(property "Description" "Power symbol creates a global label with name \"+12V\""
-			(at 118.11 30.48 0)
+			(at 102.87 30.48 0)
 			(effects
 				(font
@@
 	(symbol
 		(lib_id "Device:R")
-		(at 127 39.37 270)
+		(at 109.22 39.37 270)
 		(unit 1)
 		(exclude_from_sim no)
@@
 		(dnp no)
 		(property "Reference" "R11"
-			(at 128.778 36.83 90)
+			(at 110.998 36.83 90)
 			(effects
 				(font
@@
 		)
 		(property "Value" "127k"
-			(at 129.286 39.37 90)
+			(at 111.506 39.37 90)
 			(effects
 				(font
@@
 		)
 		(property "Footprint" "Resistor_SMD:R_0603_1608Metric"
-			(at 127 37.592 90)
+			(at 109.22 37.592 90)
 			(effects
 				(font
@@
 		)
 		(property "Datasheet" "~"
-			(at 127 39.37 0)
+			(at 109.22 39.37 0)
 			(effects
 				(font
@@
 		)
 		(property "Description" "Resistor"
-			(at 127 39.37 0)
+			(at 109.22 39.37 0)
 			(effects
 				(font
@@
 		)
 		(property "MPN" "127k 0603"
-			(at 127 39.37 0)
+			(at 109.22 39.37 0)
 			(effects
 				(font

Commit message: Warrior… Priestess… Tramp
Parts:
- removed D1: D_Zener, Diode_SMD:D_0805_2012Metric, symbol Device:D_Zener
- removed Q1, Q5, Q6: IRLML5203, Package_TO_SOT_SMD:SOT-23, symbol Transistor_FET:IRLML5203
- added Q5, Q6: IRLML6402, Package_TO_SOT_SMD:SOT-23, symbol Transistor_FET:IRLML6402
Connections:
- net +12V: now also C1.1, U7.1 (IN), Q5.2 (S); no longer J10.2 (Pin_2), J11.2 (Pin_2), J12.2 (Pin_2), J6.2 (Pin_2), J7.2 (Pin_2), J8.2 (Pin_2), J9.2 (Pin_2), R11.2, R5.1, R8.2
- net GND: now also R11.1
- net VBUS: now also Q6.3 (D)
- net at Q2.3 (D), R8.1: now also Q6.1 (G)
- new net: Q5.1 (G), R11.2
- new net VCC: J10.2 (Pin_2), J11.2 (Pin_2), J12.2 (Pin_2), J6.2 (Pin_2), J7.2 (Pin_2), J8.2 (Pin_2), J9.2 (Pin_2), Q5.3 (D), Q6.2 (S), R5.1, R8.2
