File: kicad/Ryujin/Ryujin.kicad_pcb (KiCad board)
At the start: 2 copper layers, 56 x 77 mm, 32 parts, among them J1 BAT, J2 SDI12, J3 Conn_01x14_Socket, J4 Conn_01x14_Socket, J5 USB_A, Q1 IRLML6244, U1 TXS0101DBV, U2 R-78E5.0-0.5, U3 W25Q32JVSS, U4 SHTC3, U5 CH340N

Commit message: Unchained Heart
Parts:
- removed C7: 0.1uF, Capacitor_SMD:C_0603_1608Metric
- removed FB2: FerriteBead, Inductor_SMD:L_0603_1608Metric
- moved FB1 2.00 mm to (251.5, 86.1)
Connections:
- J4 pad 5: /RTS -> unconnected-(J4-RESET-Pad5)
- J5 pad 1: Net-(J5-VBUS) -> /VIN
- U5 pad 4: Net-(U5-~{RTS}) -> unconnected-(U5-~{RTS}-Pad4)
Routing:
- net /RTS: track 34.6 -> 0.00 mm, vias 2 -> 0
- net Net-(J5-VBUS): track 15.6 -> 0.00 mm
- net /GND: track 143.9 -> 148.5 mm
- net /COPI: track 17.4 -> 21.3 mm
- net Net-(U5-~{RTS}): track 3.36 -> 0.00 mm
- net /BUS: track 36.1 -> 32.9 mm, vias 1 -> 0
- net /BAT+: track 91.5 -> 88.3 mm, vias 2 -> 1
- net /5V: track 37.2 -> 34.4 mm
- net /D0: track 46.5 -> 48.7 mm
- net /SCK: track 14.9 -> 16.9 mm
- net /VIN: track 40.5 -> 38.7 mm, vias 2 -> 1
- net /CIPO: track 9.80 -> 11.4 mm, vias 0 -> 1
- net /SDI+: track 13.3 -> 14.2 mm
- net Net-(J5-Shield): track 26.2 -> 25.3 mm
- net /3V3: track 84.9 -> 84.2 mm

Commit message: What's in a Name?
Other:
- board text removed: "2024-12-15"
- board text removed: "Ryujin"
Changed lines of the file:
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@@
 	(paper "A4")
 	(title_block
+		(title "Ryujin")
+		(date "2024-12-21")
+		(rev "17")
+		(company "Julius-Maximilians-Universität Würzburg")
 		(comment 4 "AISLER Project ID: ZJYYZNOG")
 	)
@@
 	)
 	(setup
+		(stackup
+			(layer "F.SilkS"
+				(type "Top Silk Screen")
+			)
+			(layer "F.Paste"
+				(type "Top Solder Paste")
+			)
+			(layer "F.Mask"
+				(type "Top Solder Mask")
+				(thickness 0.01)
+			)
+			(layer "F.Cu"
+				(type "copper")
+				(thickness 0.035)
+			)
+			(layer "dielectric 1"
+				(type "core")
+				(thickness 1.51)
+				(material "FR4")
+				(epsilon_r 4.5)
+				(loss_tangent 0.02)
+			)
+			(layer "B.Cu"
+				(type "copper")
+				(thickness 0.035)
+			)
+			(layer "B.Mask"
+				(type "Bottom Solder Mask")
+				(thickness 0.01)
+			)
+			(layer "B.Paste"
+				(type "Bottom Solder Paste")
+			)
+			(layer "B.SilkS"
+				(type "Bottom Silk Screen")
+			)
+			(copper_finish "None")
+			(dielectric_constraints no)
+		)
 		(pad_to_mask_clearance 0)
 		(allow_soldermask_bridges_in_footprints no)
@@
 			)
 			(justify left bottom)
-		)
-	)
-	(gr_text "Ryujin"
-		(at 187 190.5 0)
-		(layer "Cmts.User")
-		(effects
-			(font
-				(size 1.5 1.5)
-				(thickness 0.3)
-				(bold yes)
-			)
-			(justify left bottom)
-		)
-	)
-	(gr_text "2024-12-15"
-		(at 206.5 194 0)
-		(layer "Cmts.User")
-		(effects
-			(font
-				(size 1.5 1.5)
-				(thickness 0.3)
-				(bold yes)
-			)
-			(justify left bottom)

Commit message: The Vanishing Dead
Parts:
- removed FB1: FerriteBead, Inductor_SMD:L_0603_1608Metric
- removed U5: CH340N, Package_SO:SOP-8_3.9x4.9mm_P1.27mm
- J5: value USB_A -> Conn_02x03_Odd_Even; footprint Connector_USB:USB_A_Molex_105057_Vertical -> Connector_PinHeader_2.54mm:PinHeader_2x03_P2.54mm_Vertical
- moved J5 78.6 mm to (174.5, 46.7)
- moved U2 76.3 mm to (164.0, 61.0)
- moved A1 76.1 mm to (153.5, 28.5)
- moved C1 76.1 mm to (169.2, 61.4)
- moved C2 76.1 mm to (169.2, 55.4)
- moved C3 76.1 mm to (144.5, 34.5)
- moved C4 76.1 mm to (171.0, 67.0)
- moved C5 76.1 mm to (171.0, 74.0)
- moved C6 76.1 mm to (144.0, 62.5)
- moved H1 76.1 mm to (182.0, 22.0)
- moved H2 76.1 mm to (182.0, 93.0)
- moved H3 76.1 mm to (132.0, 93.0)
- moved H4 76.1 mm to (132.0, 22.0)
- moved J1 76.1 mm to (163.0, 84.5)
- moved J2 76.1 mm to (163.0, 40.5)
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Connections:
- J4 pad 5: unconnected-(J4-RESET-Pad5) -> /RTS
- J4 pad 6: /TX -> unconnected-(J4-D14/TX-Pad6)
- J4 pad 7: /RX -> unconnected-(J4-D13/RX-Pad7)
- J5 pad 1: /VIN -> /CIPO
- J5 pad 2: Net-(J5-D-) -> /5V
- J5 pad 3: Net-(J5-D+) -> /SCK
- J5 pad 4: /GND -> /COPI
- J5 pad 5: Net-(J5-Shield) -> /RTS
Routing:
- net /CIPO: track 11.4 -> 49.5 mm
- net /TX: track 32.7 -> 0.00 mm, vias 1 -> 0
- net /RX: track 29.7 -> 0.00 mm, vias 1 -> 0
- net /RTS: track 0.00 -> 27.9 mm, vias 0 -> 1
- net Net-(J5-Shield): track 25.3 -> 0.00 mm
- net /SCK: track 16.9 -> 41.5 mm
- net /COPI: track 21.3 -> 42.1 mm
- net /VIN: track 38.7 -> 19.9 mm
- net /3V3: track 84.2 -> 65.6 mm, vias 3 -> 1
- net Net-(J5-D-): track 17.1 -> 0.00 mm
- net Net-(J5-D+): track 13.3 -> 0.00 mm
- net /BUS: track 32.9 -> 44.0 mm, vias 0 -> 1
- net /5V: track 34.4 -> 44.0 mm, vias 1 -> 0
- net /GND: track 148.5 -> 139.5 mm, vias 2 -> 3
- net /BAT+: track 88.3 -> 92.5 mm, vias 1 -> 2
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
Commit message: The Gauntlet
Parts:
- moved J5 1.01 mm to (175.5, 47.0)
Routing:
- net /SCK: track 41.5 -> 51.4 mm, vias 1 -> 2
- net /GND: track 139.5 -> 147.2 mm, vias 3 -> 1
- net /RTS: track 27.9 -> 32.7 mm, vias 1 -> 0
- net /BUS: track 44.0 -> 46.8 mm
- net /D1: track 44.0 -> 41.9 mm
- net /BAT+: track 92.5 -> 90.7 mm
- net /D0: track 45.9 -> 47.5 mm
- net /3V3: track 65.6 -> 67.1 mm
- net /CIPO: track 49.5 -> 48.0 mm, vias 1 -> 2
- net /5V: track 44.0 -> 45.2 mm
- net /COPI: track 42.1 -> 42.9 mm

Commit message: Outcast
Parts:
- added J6: FTSH-105-01-L-D, Custom:SAMTEC_FTSH-105-01-L-D, F.Cu at (170.0, 48.5)
- J5: moved to B.Cu
- moved J5 34.2 mm to (142.0, 53.6), turned to 0 degrees
Connections:
- J5 pad 1: /CIPO -> unconnected-(J5-Pin_1-Pad1)
- J5 pad 2: /5V -> /SWDIO
- J5 pad 3: /SCK -> unconnected-(J5-Pin_3-Pad3)
- J5 pad 4: /COPI -> /SWCLK
- J5 pad 5: /RTS -> unconnected-(J5-Pin_5-Pad5)
- J5 pad 6: /GND -> unconnected-(J5-Pin_6-Pad6)
Routing:
- net /CIPO: track 48.0 -> 11.4 mm, vias 2 -> 1
- net /SCK: track 51.4 -> 16.9 mm, vias 2 -> 1
- net /SWCLK: track 0.00 -> 29.0 mm
- net /SWDIO: track 0.00 -> 28.1 mm
- net /COPI: track 42.9 -> 21.3 mm
- net /3V3: track 67.1 -> 84.8 mm
- net /BUS: track 46.8 -> 35.3 mm
- net /GND: track 147.2 -> 138.7 mm, vias 1 -> 2
- net /5V: track 45.2 -> 37.1 mm, vias 0 -> 1
- net /SCL: track 13.5 -> 18.9 mm
- net /RTS: track 32.7 -> 29.3 mm
- net /BAT+: track 90.7 -> 89.6 mm
- net /D0: track 47.5 -> 48.3 mm

Commit message: The Mother of All Monsters
Parts:
- moved J6 43.7 mm to (165.5, 92.0), turned to 180 degrees
Routing:
- net /SWCLK: track 29.0 -> 70.6 mm, vias 0 -> 1
- net /SWDIO: track 28.1 -> 68.2 mm, vias 0 -> 1
- net /GND: track 138.7 -> 151.4 mm, vias 2 -> 3
- net /RTS: track 29.3 -> 37.6 mm
- net /SCL: track 18.9 -> 13.5 mm
- net /D0: track 48.3 -> 46.6 mm
- net /SCK: track 16.9 -> 15.3 mm
- net /D7: track 9.16 -> 10.7 mm, vias 0 -> 1
- net /BAT+: track 89.6 -> 88.4 mm
- net /5V: track 37.1 -> 36.0 mm
- net /COPI: track 21.3 -> 20.5 mm

Commit message: Mother of All Monsters
Parts:
- J5: moved to F.Cu
- moved J5 2.58 mm to (144.5, 53.6), turned to 180 degrees
Routing:
- net /BAT+: track 88.4 -> 74.2 mm
- net /GND: track 151.4 -> 163.8 mm, vias 3 -> 2
- net /5V: track 36.0 -> 40.3 mm
- net /BUS: track 34.8 -> 39.0 mm
- net /3V3: track 84.8 -> 88.6 mm, vias 1 -> 3
- net /SWDIO: track 68.2 -> 66.2 mm
- net /SWCLK: track 70.6 -> 69.1 mm
- net /CIPO: track 11.3 -> 9.93 mm
- net /COPI: track 20.5 -> 19.4 mm
- net Net-(Q1-G): track 7.31 -> 8.19 mm
- net /D0: track 46.6 -> 47.3 mm
- net /SCK: track 15.3 -> 14.8 mm
- net /VIN: track 20.1 -> 20.4 mm, vias 1 -> 0

Commit message: The Other Side
Parts:
- removed C4, C5: 0.1uF, Capacitor_SMD:C_0603_1608Metric
- removed R1: 47k, Resistor_SMD:R_0603_1608Metric
- added U5: 74AHCT1G125, Package_TO_SOT_SMD:SOT-23-5, F.Cu at (171.9, 72.5)
- U1: value TXS0101DBV -> 74LVC1G17; footprint Package_TO_SOT_SMD:SOT-23-6 -> Package_TO_SOT_SMD:SOT-23-5
- moved J6 4.74 mm to (161.0, 93.5), turned to 0 degrees
- moved U1 2.72 mm to (171.9, 67.9), turned to 0 degrees
Connections:
- J2 pad 2: /SDI+ -> /BAT+
- J2 pad 3: /GND -> /SDI-
- Q1 pad 2: /SDI+ -> /GND
- Q1 pad 3: /BAT+ -> /SDI-
- U1 pad 1: /3V3 -> unconnected-(U1-NC-Pad1)
- U1 pad 2: /GND -> /BUS
- U1 pad 3: /D1 -> /GND
- U1 pad 4: /BUS -> /D1
- U1 pad 5: Net-(U1-OE) -> /3V3
Routing:
- net /GND: track 163.8 -> 0.00 mm, vias 2 -> 0
- net /3V3: track 88.6 -> 0.00 mm, vias 3 -> 0
- net /BAT+: track 74.2 -> 0.00 mm, vias 2 -> 0
- net /SWCLK: track 69.1 -> 0.00 mm, vias 1 -> 0
- net /SWDIO: track 66.2 -> 0.00 mm, vias 1 -> 0
- net /D0: track 47.3 -> 0.00 mm, vias 1 -> 0
- net /D1: track 42.3 -> 0.00 mm, vias 1 -> 0
- net /5V: track 40.3 -> 0.00 mm, vias 1 -> 0
- net /BUS: track 39.0 -> 0.00 mm, vias 1 -> 0
- net /RTS: track 37.6 -> 0.00 mm
- net /A1: track 24.3 -> 0.00 mm
- net /VIN: track 20.4 -> 0.00 mm
- net /COPI: track 19.4 -> 0.00 mm, vias 1 -> 0
- net /SCK: track 14.8 -> 0.00 mm, vias 1 -> 0
- net /SDI+: track 13.5 -> 0.00 mm
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