File: kicad/Ryujin/Ryujin.kicad_pcb (KiCad board)
At the start: 2 copper layers, 56 x 77 mm, 27 parts, among them J1 Screw_Terminal_01x06, J2 Conn_02x02_Odd_Even, J3 Conn_01x14_Socket, J4 Conn_01x14_Socket, Q1 IRLML6244, U1 74LVC1G17, U2 74AHCT1G14, U3 TMUX1119DBVR, U4 SHTC3, U5 W25Q32JVSS, U6 R-78E5.0-0.5

Commit message: Two Men and a Baby
Parts:
- added R1: 47k, Resistor_SMD:R_0603_1608Metric, F.Cu at (144.5, 43.0)
Routing:
- net /SCL: track 39.0 -> 47.5 mm
- net GND: track 145.8 -> 140.0 mm
- net +12V: track 75.5 -> 79.5 mm, vias 1 -> 2
- net /COPI: track 21.6 -> 17.7 mm, vias 0 -> 1
- net +5V: track 19.5 -> 22.2 mm
- net LINE: track 46.8 -> 48.6 mm
- net Net-(U3-S2): track 14.4 -> 12.8 mm
- net /SDA: track 39.1 -> 38.0 mm
- net Net-(Q1-G): track 7.77 -> 7.12 mm

Commit message: Norse by Norsevest
Parts:
- added J6: 1789210, footprints:FFKDSA1_508_2, F.Cu at (178.7, 78.2)
- J1: value Screw_Terminal_01x06 -> 1704376; footprint ThirdParty:SMKDSN-1-5-6-5-08_3D -> footprints:FFKDSA1_508_3
- J3, J4: footprint Custom:65342372 -> footprints:65342372
- R1: value 47k -> 3k3
- R3: value 47k -> 33k
- moved J1 19.9 mm to (178.6, 62.2)
- moved R3 17.2 mm to (174.1, 38.5)
- moved R2 17.2 mm to (177.7, 41.7)
- moved Q1 17.2 mm to (177.7, 38.5)
- moved C2 12.7 mm to (161.9, 48.6), turned to 0 degrees
- moved C1 8.61 mm to (161.9, 53.6), turned to 0 degrees
- moved U5 7.05 mm to (161.8, 76.4)
- moved J2 3.12 mm to (164.9, 28.4)
- moved U6 1.72 mm to (162.3, 41.8)
Routing:
- net /D0: track 41.7 -> 64.6 mm
- net GND: track 140.0 -> 149.9 mm, vias 2 -> 3
- net /SCL: track 47.5 -> 39.0 mm
- net /COPI: track 17.7 -> 11.0 mm
- net /SCK: track 15.6 -> 10.1 mm
- net LINE: track 48.6 -> 43.2 mm
- net -12V: track 23.8 -> 28.9 mm, vias 1 -> 0
- net /D2: track 67.4 -> 71.1 mm
- net /CIPO: track 9.23 -> 12.3 mm
- net /D7: track 8.73 -> 6.05 mm
- net VDD: track 25.3 -> 22.8 mm
- net +3.3V: track 68.4 -> 70.8 mm
- net +12V: track 79.5 -> 77.4 mm
- net /SDA: track 38.0 -> 39.1 mm
- net Net-(Q1-G): track 7.12 -> 7.77 mm
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
Commit message: For Those of You Just Joining Us
Parts:
- removed J6: 1789210, footprints:FFKDSA1_508_2
- added J5: 1869224, footprints:SMKDSN_508_3, F.Cu at (169.9, 55.5)
- J1: value 1704376 -> 1869211; footprint footprints:FFKDSA1_508_3 -> footprints:SMKDSN_508_2
- moved Q1 34.9 mm to (161.8, 69.6), turned to 0 degrees
- moved R3 32.3 mm to (165.4, 69.6), turned to 90 degrees
- moved R2 29.2 mm to (161.8, 66.3), turned to 0 degrees
- moved J1 14.2 mm to (175.0, 75.8), turned to 0 degrees
- moved U5 2.56 mm to (163.4, 78.4)
- moved C1 0.52 mm to (161.4, 53.8)
- moved C2 0.52 mm to (161.4, 48.8)
Routing:
- net GND: track 149.9 -> 0.00 mm, vias 3 -> 0
- net +12V: track 77.4 -> 0.00 mm, vias 2 -> 0
- net /D2: track 71.1 -> 0.00 mm, vias 1 -> 0
- net +3.3V: track 70.8 -> 0.00 mm
- net /D0: track 64.6 -> 0.00 mm, vias 1 -> 0
- net /RX: track 50.1 -> 0.00 mm
- net /TX: track 43.9 -> 0.00 mm
- net LINE: track 43.2 -> 0.00 mm, vias 1 -> 0
- net /SDA: track 39.1 -> 0.00 mm
- net /SCL: track 39.0 -> 0.00 mm
- net /D1: track 34.8 -> 0.00 mm
- net -12V: track 28.9 -> 0.00 mm
- net VDD: track 22.8 -> 0.00 mm
- net +5V: track 22.0 -> 0.00 mm, vias 1 -> 0
- net /CIPO: track 12.3 -> 0.00 mm
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
Commit message: Let There Be Light
Parts:
- removed J5: 1869224, footprints:SMKDSN_508_3
- J1: value 1869211 -> SMKDSN_6_508; footprint footprints:SMKDSN_508_2 -> footprints:SMKDSN_508_6
- moved J1 2.93 mm to (176.4, 78.4), turned to 90 degrees
Connections:
- J1 pad 1: +12V -> LINE
- J1 pad 2: GND -> -12V

Commit message: Sky High
Parts:
- added J5: Conn_01x03_Pin, Connector_Molex:Molex_KK-254_AE-6410-03A_1x03_P2.54mm_Vertical, F.Cu at (175.5, 40.8)

Commit message: Stranger and Stranger
Parts:
- removed J1: SMKDSN_6_508, footprints:SMKDSN_508_6
- added REF**: TerminalBlock_Phoenix_MKDS-1,5-2-5.08_1x02_P5.08mm_Horizont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, TerminalBlock_Phoenix:TerminalBlock_Phoenix_MKDS-1,5-2-5.08_1x02_P5.08mm_Horizontal, F.Cu at (167.4, 79.2)
- J5: footprint Connector_Molex:Molex_KK-254_AE-6410-03A_1x03_P2.54mm_Vertical -> footprints:GROVE-HW4-2.0
- moved Q1 19.2 mm to (166.8, 51.0)
- moved R2 19.2 mm to (166.8, 47.7)
- moved R3 19.2 mm to (170.3, 51.0)
- moved C2 19.0 mm to (163.4, 67.7), turned to -90 degrees
- moved U5 19.0 mm to (144.4, 78.2)
- moved U6 17.0 mm to (168.5, 57.6), turned to 180 degrees
- moved C1 15.6 mm to (168.5, 67.7), turned to 180 degrees
- moved J5 9.42 mm to (166.2, 42.2), turned to 180 degrees
Connections:
- J5 pad 1: unconnected-(J5-Pin_1-Pad1) -> LINE
- J5 pad 2: unconnected-(J5-Pin_2-Pad2) -> +12V
- J5 pad 3: unconnected-(J5-Pin_3-Pad3) -> -12V

Commit message: Just Passing Through
Parts:
- moved U6 2.44 mm to (168.5, 55.2)
- moved R3 1.87 mm to (170.4, 49.1)
- moved Q1 1.87 mm to (166.9, 49.1)
- moved R2 1.87 mm to (166.9, 45.9)
- moved J5 1.58 mm to (166.9, 40.8)
- moved C1 1.24 mm to (168.5, 66.5)
- moved C2 1.24 mm to (163.4, 66.5)
- moved U5 0.16 mm to (144.2, 78.2)
Routing:
- net GND: track 0.00 -> 167.4 mm, vias 0 -> 3
- net +3.3V: track 0.00 -> 80.2 mm, vias 0 -> 1
- net +12V: track 0.00 -> 71.4 mm, vias 0 -> 1
- net /D2: track 0.00 -> 70.4 mm, vias 0 -> 1
- net /RX: track 0.00 -> 51.5 mm
- net /D0: track 0.00 -> 51.3 mm, vias 0 -> 1
- net /TX: track 0.00 -> 50.0 mm, vias 0 -> 1
- net /SCL: track 0.00 -> 43.7 mm, vias 0 -> 2
- net /SDA: track 0.00 -> 38.0 mm
- net /D1: track 0.00 -> 34.3 mm
- net LINE: track 0.00 -> 32.2 mm, vias 0 -> 1
- net +5V: track 0.00 -> 22.5 mm, vias 0 -> 1
- net VDD: track 0.00 -> 20.7 mm
- net /CIPO: track 0.00 -> 18.1 mm, vias 0 -> 1
- net /D7: track 0.00 -> 15.9 mm, vias 0 -> 1
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
Commit message: Greece Is Burning
Parts:
- moved J5 2.54 mm to (166.9, 38.2), turned to 0 degrees
- moved U5 0.26 mm to (144.5, 78.2), turned to 180 degrees
Routing:
- net GND: track 167.4 -> 154.9 mm
- net /COPI: track 8.89 -> 18.8 mm, vias 0 -> 1
- net /D7: track 15.9 -> 7.42 mm, vias 1 -> 0
- net +12V: track 71.4 -> 79.7 mm
- net /TX: track 50.0 -> 42.5 mm, vias 1 -> 0
- net /CIPO: track 18.1 -> 11.3 mm, vias 1 -> 0
- net /SCK: track 10.6 -> 17.2 mm, vias 0 -> 1
- net LINE: track 32.2 -> 25.7 mm
- net +5V: track 22.5 -> 27.6 mm
- net /D0: track 51.3 -> 56.4 mm
- net /SCL: track 43.7 -> 39.9 mm, vias 2 -> 0
- net Net-(U3-S2): track 8.85 -> 10.9 mm, vias 2 -> 0
- net /D1: track 34.3 -> 36.0 mm
- net /RX: track 51.5 -> 50.1 mm
- net /SDA: track 38.0 -> 39.2 mm
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