File: kicad/Ryujin/Ryujin.kicad_pcb (KiCad board)
At the start: 2 copper layers, 173 x 72 mm, 59 parts, among them J1 Conn_01x02_Socket, J10 Conn_01x04_Pin, J11 Conn_01x04_Pin, J12 Conn_01x04_Pin, J2 1822972, J3 Conn_01x14_Socket, J4 Conn_01x14_Socket, J5 1822972, J6 Conn_01x04_Pin, J7 Conn_01x04_Pin, J8 Conn_01x04_Pin, J9 Conn_01x04_Pin, Q1 IRLML5203, Q2 IRLML6244, Q3 Si7288, U1 74LVC1G17, U2 74AHCT1G14, U3 TMUX1119DBVR, U4 SHTC3, U5 W25Q32JVSS, U6 BQ24650, U7 R-78E5.0-1.0

Commit message: Is There a Doctor in the House?
Other:
- outline, holes or cut-outs redrawn
Changed lines of the file:
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@@
 			(psa4output no)
 			(plot_black_and_white yes)
-			(plotinvisibletext no)
 			(sketchpadsonfab no)
 			(plotpadnumbers no)
@@
 		)
 	)
-	(gr_line
-		(start 14.75 93.3)
-		(end 14.75 31.3)
+	(gr_rect
+		(start 14.75 26.3)
+		(end 187.75 98.3)
 		(stroke
 			(width 0.05)
-			(type default)
-		)
-		(layer "Edge.Cuts")
-	)
-	(gr_line
-		(start 182.75 98.3)
-		(end 187.75 93.3)
-		(stroke
-			(width 0.05)
-			(type default)
-		)
-		(layer "Edge.Cuts")
-	)
-	(gr_line
-		(start 182.75 26.3)
-		(end 19.75 26.3)
-		(stroke
-			(width 0.05)
-			(type default)
-		)
-		(layer "Edge.Cuts")
-	)
-	(gr_line
-		(start 19.75 26.3)
-		(end 14.75 31.3)
-		(stroke
-			(width 0.05)
-			(type default)
-		)
-		(layer "Edge.Cuts")
-	)
-	(gr_line
-		(start 182.75 26.3)
-		(end 187.75 31.3)
-		(stroke
-			(width 0.05)
-			(type default)
-		)
-		(layer "Edge.Cuts")
-	)
-	(gr_line
-		(start 187.75 93.3)
-		(end 187.75 31.3)
-		(stroke
-			(width 0.05)
-			(type default)
-		)
-		(layer "Edge.Cuts")
-	)
-	(gr_line
-		(start 19.75 98.3)
-		(end 14.75 93.3)
-		(stroke
-			(width 0.05)
-			(type default)
-		)
-		(layer "Edge.Cuts")
-	)
-	(gr_line
-		(start 182.75 98.3)
-		(end 19.75 98.3)
-		(stroke
-			(width 0.05)
-			(type default)
+			(type solid)
 		)
+		(fill no)
 		(layer "Edge.Cuts")
 	)

Commit message: Orphan of War
Parts:
- added D8: D1, footprints:PDS104013, F.Cu at (90.8, 74.2)
- added Q4: 2N7002, Package_TO_SOT_SMD:SOT-23, F.Cu at (93.8, 80.3)
Connections:
- C1 pad 1: +12V -> Net-(D8-K)
- J3 pad 14: unconnected-(J3-~D5-Pad14) -> /D5
- U7 pad 1: +12V -> Net-(D8-K)
Routing:
- net /D5: track 0.00 -> 61.2 mm
- net Net-(Q4-D): track 8.14 -> 66.8 mm, vias 0 -> 2
- net Net-(D8-K): track 0.00 -> 15.3 mm
- net +12V: track 289.2 -> 295.0 mm
- net /Battery Charger/TS: track 82.1 -> 78.8 mm
- net /Battery Charger/VIN: track 44.7 -> 42.2 mm

Commit message: Remember Nothing
Parts:
- Q4: moved to B.Cu
- moved Q4 8.50 mm to (99.8, 74.2)
Routing:
- net Net-(Q4-D): track 66.8 -> 57.7 mm, vias 2 -> 1
- net /D5: track 61.2 -> 69.7 mm

Commit message: In Sickness and in Hell
Other:
- board size 173 x 72 mm -> 174 x 72 mm
Changed lines of the file:
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@@
 	)
 	(gr_rect
-		(start 14.75 26.3)
-		(end 187.75 98.3)
+		(start 14.25 26.3)
+		(end 188.25 98.3)
 		(stroke
 			(width 0.05)

Commit message: A Tale of Two Muses
Parts:
- removed Q4: 2N7002, Package_TO_SOT_SMD:SOT-23
- D8: value D1 -> D2; footprint footprints:PDS104013 -> Package_TO_SOT_SMD:SOT-23
- moved D8 1.13 mm to (89.8, 73.8)
Connections:
- D8 pad 2: +12V -> unconnected-(D8-NC-Pad2)
Routing:
- net /D5: track 69.7 -> 0.00 mm
- net Net-(U6-MPPSET): track 57.7 -> 8.29 mm, vias 1 -> 0
- net Net-(D8-K): track 15.3 -> 13.1 mm
- net +12V: track 295.0 -> 295.8 mm

Commit message: Past Imperfect
Parts:
- removed D8: D2, Package_TO_SOT_SMD:SOT-23
- added D1: SS34, Diode_SMD:D_SMA, B.Cu at (122.5, 74.8)
Routing:
- net Net-(D1-K): track 13.1 -> 45.1 mm
- net +12V: track 295.8 -> 266.4 mm

Commit message: Daughter of Pomira
Parts:
- moved D1 0.95 mm to (122.5, 73.8)
Routing:
- net +12V: track 266.4 -> 265.4 mm
Changed lines of the file:
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@@
 	(footprint "Diode_SMD:D_SMA"
 		(layer "B.Cu")
-		(at 122.46 74.79)
+		(at 122.46 73.84)
 		(descr "Diode SMA (DO-214AC)")
 		(tags "Diode SMA (DO-214AC)")
@@
 	)
 	(segment
+		(start 124.46 67.32)
+		(end 124.46 73.84)
+		(width 0.45)
+		(layer "B.Cu")
+		(net 3)
+	)
+	(segment
 		(start 162.084 75.2625)
 		(end 162.13 75.3073)
@@
 	)
 	(segment
-		(start 124.46 67.32)
-		(end 124.46 74.79)
-		(width 0.45)
-		(layer "B.Cu")
-		(net 3)
-	)
-	(segment
 		(start 99.46 52.32)
 		(end 99.46 37.32)
@@
 	)
 	(segment
-		(start 120.46 74.79)
-		(end 81.657 74.79)
-		(width 0.45)
-		(layer "B.Cu")
-		(net 60)
-	)
-	(segment
-		(start 81.657 74.79)
+		(start 120.46 73.84)
 		(end 80.707 73.84)
 		(width 0.45)

Commit message: The Convert
Parts:
- U5: value W25Q32JVSS -> W25Q128JVS; footprint Package_SO:SOIC-8_5.23x5.23mm_P1.27mm -> Package_SO:SOIC-8_5.3x5.3mm_P1.27mm
