File: kicad/Ryujin/Battery_Charger.kicad_sch (KiCad schematic)
At the start: 30 parts, among them Q3 IRLML6244, Q4 IRLML6244, Q5 IRLML6244, U6 BQ24650

Commit message: Destiny
Other:
- moved on the sheet: C15
Changed lines of the file:
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@@
 	)
 	(junction
+		(at 104.14 74.93)
+		(diameter 0)
+		(color 0 0 0 0)
+	)
+	(junction
 		(at 266.7 78.74)
 		(diameter 0)
@@
 	)
 	(junction
-		(at 109.22 74.93)
-		(diameter 0)
-		(color 0 0 0 0)
-	)
-	(junction
 		(at 59.69 48.26)
 		(diameter 0)
@@
 	(wire
 		(pts
-			(xy 109.22 74.93) (xy 113.03 74.93)
-		)
-		(stroke
-			(width 0)
-			(type default)
-		)
-	)
-	(wire
-		(pts
 			(xy 142.24 111.76) (xy 149.86 111.76)
 		)
@@
 	(wire
 		(pts
-			(xy 104.14 74.93) (xy 109.22 74.93)
+			(xy 261.62 95.25) (xy 261.62 97.79)
 		)
 		(stroke
@@
 	(wire
 		(pts
-			(xy 261.62 95.25) (xy 261.62 97.79)
+			(xy 154.94 80.01) (xy 161.29 80.01)
 		)
 		(stroke
@@
 	(wire
 		(pts
-			(xy 154.94 80.01) (xy 161.29 80.01)
+			(xy 199.39 78.74) (xy 201.93 78.74)
 		)
 		(stroke
@@
 	(wire
 		(pts
-			(xy 199.39 78.74) (xy 201.93 78.74)
+			(xy 107.95 95.25) (xy 107.95 129.54)
 		)
 		(stroke
@@
 	(wire
 		(pts
-			(xy 107.95 95.25) (xy 107.95 129.54)
+			(xy 104.14 74.93) (xy 113.03 74.93)
 		)
 		(stroke
@@
 	(wire
 		(pts
-			(xy 109.22 69.85) (xy 109.22 74.93)
+			(xy 104.14 69.85) (xy 104.14 74.93)
 		)
 		(stroke
@@
 	(symbol
 		(lib_id "Device:C")
-		(at 105.41 69.85 90)
+		(at 100.33 69.85 90)
 		(unit 1)
 		(exclude_from_sim no)
@@
 		(fields_autoplaced yes)
 		(property "Reference" "C15"
-			(at 105.41 62.23 90)
+			(at 100.33 62.23 90)
 			(effects
 				(font
@@
 		)
 		(property "Value" "C"
-			(at 105.41 64.77 90)
+			(at 100.33 64.77 90)
 			(effects
 				(font
@@
 		)
 		(property "Footprint" "Capacitor_SMD:C_0603_1608Metric"
-			(at 109.22 68.8848 0)
+			(at 104.14 68.8848 0)
 			(effects
 				(font
@@
 		)
 		(property "Datasheet" "~"
-			(at 105.41 69.85 0)
+			(at 100.33 69.85 0)
 			(effects
 				(font
@@
 		)
 		(property "Description" "Unpolarized capacitor"
-			(at 105.41 69.85 0)
+			(at 100.33 69.85 0)
 			(effects
 				(font
@@
 	(symbol
 		(lib_id "power:GND")
-		(at 101.6 69.85 270)
+		(at 96.52 69.85 270)
 		(unit 1)
 		(exclude_from_sim no)
@@
 		(fields_autoplaced yes)
 		(property "Reference" "#PWR046"
-			(at 95.25 69.85 0)
+			(at 90.17 69.85 0)
 			(effects
 				(font
@@
 		)
 		(property "Value" "GND"
-			(at 97.79 69.8499 90)
+			(at 92.71 69.8499 90)
 			(effects
 				(font
@@
 		)
 		(property "Footprint" ""
-			(at 101.6 69.85 0)
+			(at 96.52 69.85 0)
 			(effects
 				(font
@@
 		)
 		(property "Datasheet" ""
-			(at 101.6 69.85 0)
+			(at 96.52 69.85 0)
 			(effects
 				(font
@@
 		)
 		(property "Description" "Power symbol creates a global label with name \"GND\" , ground"
-			(at 101.6 69.85 0)
+			(at 96.52 69.85 0)
 			(effects
 				(font

Commit message: For Him the Bell Tolls
Parts:
- U6: MPN (none) -> BQ24650RVAR
Changed lines of the file:
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@@
 			)
 		)
-		(property "Datasheet" "https://www.ti.com/lit/ds/symlink/bq24650.pdf"
+		(property "Datasheet" "../../docs/bq24650.pdf"
 			(at 129.54 90.17 0)
 			(effects
@@
 			(effects
 				(font
+					(size 1.27 1.27)
+				)
+				(hide yes)
+			)
+		)
+		(property "MPN" "BQ24650RVAR"
+			(at 129.54 85.09 0)
+			(effects
+				(font

Commit message: The Execution
Parts:
- Q3, Q4, Q5: MPN (none) -> IRLML6244TRPBF
Changed lines of the file:
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@@
+			)
+		)
+		(property "MPN" "IRLML6244TRPBF"
+			(at 196.85 91.44 0)
+			(effects
+				(font
+					(size 1.27 1.27)
+				)
+				(hide yes)
 			)
 		)
@@
 			)
 		)
+		(property "MPN" "IRLML6244TRPBF"
+			(at 196.85 67.31 0)
+			(effects
+				(font
+					(size 1.27 1.27)
+				)
+				(hide yes)
+			)
+		)
 		(pin "1"
 		)
@@
 			(at 64.77 95.25 0)
 			(effects
+				(font
+					(size 1.27 1.27)
+				)
+				(hide yes)
+			)
+		)
+		(property "MPN" "IRLML6244TRPBF"
+			(at 64.77 95.25 0)
+			(effects

Commit message: Add files via upload
Parts:
- removed D5: D_Schottky, Diode_SMD:D_0603_1608Metric, symbol Device:D_Schottky
- removed Q3: IRLML6244, Package_TO_SOT_SMD:SOT-23, symbol Transistor_FET:IRLML6244
- removed R15: R, Resistor_SMD:R_0603_1608Metric, symbol Device:R
- added D6: BAT54W, Package_TO_SOT_SMD:SOT-323_SC-70, symbol Diode:BAT54W
- C10, C15, C8: value C -> 1uF; footprint Capacitor_SMD:C_0603_1608Metric -> Capacitor_SMD:C_0805_2012Metric; MPN (none) -> 1uF 10% 35V X7R 0805
- C11, C13: value C -> 0.1uF; footprint Capacitor_SMD:C_0603_1608Metric -> Capacitor_SMD:C_0805_2012Metric; MPN (none) -> 0.1uF 10% 35V X7R 0805
- C12, C9: value C -> 10uF; footprint Capacitor_SMD:C_0603_1608Metric -> Capacitor_SMD:C_1210_3225Metric; MPN (none) -> 10uF 20% 35V X7R 1210
- C7: value C -> 22uF; footprint Capacitor_SMD:C_0603_1608Metric -> Capacitor_SMD:C_1210_3225Metric; MPN (none) -> 22uF 10% 35V X7R 1210
- D2: value D -> PDS1040-13; MPN (none) -> PDS1040-13
- L1: footprint Inductor_SMD:L_0603_1608Metric -> Inductor_SMD:L_Vishay_IHLP-2525; MPN (none) -> IHLP2525CZER100MA1
- R1: value R -> 2; MPN (none) -> 2 0603 5% 1W
- R13: value R -> 10; footprint Resistor_SMD:R_0603_1608Metric -> Resistor_SMD:R_1206_3216Metric; MPN (none) -> 10 1206 0.5% 0.25W
- R14: value R -> 0.04; MPN (none) -> 0.04 1206 0.25W 0.5%
- R2: value R -> 301k; MPN (none) -> 301k 0603 0.5% 0.1W
- R3: value R -> 21k5; MPN (none) -> 21.5k 0603 0.5% 0.1W
Connections:
- net BAT+: now also C12.1, C13.1, R14.2, U6.9 (SRN)
- net at L1.1, Q4.2 (S), Q5.3 (D)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: now also C11.2; no longer C11.1
- net at L1.2, R14.1, U6.10 (SRP): now also C13.2; no longer C13.1
- net at C10.1, U6.12 (REGN): now also D6.1 (A)
- net at U6.16 (BTST): now also C11.1, D6.3 (K); no longer C11.2

Commit message: Blind Faith
Parts:
- removed D2: PDS1040-13, Diode_SMD:D_0603_1608Metric, symbol Device:D
- removed Q4, Q5: IRLML6244, Package_TO_SOT_SMD:SOT-23, symbol Transistor_FET:IRLML6244
- removed R17: R, Resistor_SMD:R_0603_1608Metric, symbol Device:R
- added D5: PDS1040-13, footprints:PDS104013, symbol Device:D_AAK
- added Q3: BSC014N04LS, footprints:INF-PG-TDSON-8-FL, symbol Infineon:BSC014N04LS
- added Q4: BSC014N04LSI, footprints:INF-PG-TDSON-8-FL, symbol Infineon:BSC014N04LSI
- added R15: 66k, Resistor_SMD:R_0603_1608Metric, symbol Device:R
- C14: value C -> 22pF; MPN (none) -> 22pF 10% 35V X7R 0603
- D3, D4: footprint LED_SMD:LED_0805_2012Metric -> LED_SMD:LED_0603_1608Metric; MPN (none) -> LTST-C190GKT
- D6: value BAT54W -> BAT54; footprint Package_TO_SOT_SMD:SOT-323_SC-70 -> Package_TO_SOT_SMD:SOT-23
- L1: value L -> 10uH
- R11, R12: value R -> 10k; MPN (none) -> 10k 0603 5% 0.1W
- R13: MPN 10 1206 0.5% 0.25W -> 10 1206 5% 0.25W
- R16: value R -> 330k; MPN (none) -> 330k 0603 0.5% 0.1W
- R18: value R -> 5k23; MPN (none) -> 5.23k 0603 5% 0.1W
- R19: value R -> 30k1; MPN (none) -> 30.1k 0603 5% 0.1W
- RSR1: renamed from R14; footprint Resistor_SMD:R_0603_1608Metric -> Resistor_SMD:R_1206_3216Metric; MPN 0.04 1206 0.25W 0.5% -> WSL1206R0400FEA
Connections:
- net BAT+: now also R16.1
- net GND: now also Q4.1 (SOURCE), Q4.2 (SOURCE), Q4.3 (SOURCE), R15.2; no longer R16.2
- net VIN: now also D5.1 (A), D5.2 (A)
- net at U6.13 (LODRV): now also Q4.4 (GATE)
- net at C11.2, L1.1, U6.14 (PH): now also Q3.1 (SOURCE), Q3.2 (SOURCE), Q3.3 (SOURCE), Q4.5 (DRAIN), Q4.6 (DRAIN), Q4.7 (DRAIN), Q4.8 (DRAIN)
- net at U6.15 (HIDRV): now also Q3.4 (GATE)
- net at C9.1, R13.1: now also D5.3 (K), Q3.5 (DRAIN), Q3.6 (DRAIN), Q3.7 (DRAIN), Q3.8 (DRAIN)
- net at C14.2, U6.8 (VFB): now also R16.2, R15.1; no longer R16.1

Commit message: Ulysses
Parts:
- removed C15: 1uF, Capacitor_SMD:C_0805_2012Metric, symbol Device:C
- removed Q3: BSC014N04LS, footprints:INF-PG-TDSON-8-FL, symbol Infineon:BSC014N04LS
- removed Q4: BSC014N04LSI, footprints:INF-PG-TDSON-8-FL, symbol Infineon:BSC014N04LSI
- removed R18: 5k23, Resistor_SMD:R_0603_1608Metric, symbol Device:R
- removed R19: 30k1, Resistor_SMD:R_0603_1608Metric, symbol Device:R
- added C16: C9, Capacitor_SMD:C_1210_3225Metric, symbol Device:C
- added Q3: Q1, Package_TO_SOT_SMD:LFPAK88, symbol Transistor_FET:SQJQ100E
- added Q4: Q2, Package_TO_SOT_SMD:LFPAK88, symbol Transistor_FET:SQJQ100E
- C10: value 1uF -> C4; MPN 1uF 10% 35V X7R 0805 -> 1uF 35V 0805
- C11: value 0.1uF -> C5; MPN 0.1uF 10% 35V X7R 0805 -> 0.1uF 35V 0805
- C12: value 10uF -> C8; MPN 10uF 20% 35V X7R 1210 -> 10uF 35V 1210
- C13: value 0.1uF -> C7; MPN 0.1uF 10% 35V X7R 0805 -> 0.1uF 35V 0805
- C14: value 22pF -> C10; MPN 22pF 10% 35V X7R 0603 -> 22pF 35V 0603
- C7: value 22uF -> C1; MPN 22uF 10% 35V X7R 1210 -> 2.2uF 35V 1210
- C8: value 1uF -> C2; MPN 1uF 10% 35V X7R 0805 -> 1uF 35V 0805
- C9: value 10uF -> C6; MPN 10uF 20% 35V X7R 1210 -> 10uF 35V 1210
- D5: value PDS1040-13 -> D1
- D6: value BAT54 -> D2
- L1: value 10uH -> L
- R1: value 2 -> R5; footprint Resistor_SMD:R_0603_1608Metric -> Resistor_SMD:R_0805_2012Metric; MPN 2 0603 5% 1W -> 2 0805
- R11: value 10k -> R7; footprint Resistor_SMD:R_0603_1608Metric -> Resistor_SMD:R_0402_1005Metric; MPN 10k 0603 5% 0.1W -> 10k 0402
- R12: value 10k -> R8; footprint Resistor_SMD:R_0603_1608Metric -> Resistor_SMD:R_0402_1005Metric; MPN 10k 0603 5% 0.1W -> 10k 0402
- R13: value 10 -> R6; MPN 10 1206 5% 0.25W -> 10 1206
- R15: value 66k -> R1; footprint Resistor_SMD:R_0603_1608Metric -> Resistor_SMD:R_0402_1005Metric; MPN 66k 0603 0.5% 0.1W -> 100k 0402
- R16: value 330k -> R2; footprint Resistor_SMD:R_0603_1608Metric -> Resistor_SMD:R_0402_1005Metric; MPN 330k 0603 0.5% 0.1W -> 499k 0402
- R2: value 301k -> R3; footprint Resistor_SMD:R_0603_1608Metric -> Resistor_SMD:R_0402_1005Metric; MPN 301k 0603 0.5% 0.1W -> 499k 0402
- R3: value 21k5 -> R4; footprint Resistor_SMD:R_0603_1608Metric -> Resistor_SMD:R_0402_1005Metric; MPN 21.5k 0603 0.5% 0.1W -> 36k 0402
- RSR1: value 0.04 -> RSR
Connections:
- net BAT+: now also C16.1
- net GND: now also U6.7 (TERM_EN), C16.2, Q4.2 (S), Q4.3 (S), Q4.4 (S)
- net at C11.2, L1.1, U6.14 (PH): now also Q3.2 (S), Q3.3 (S), Q3.4 (S), Q4.5 (D)
- net at U6.6 (VREF): no longer U6.7 (TERM_EN)
- net at C9.1, D5.3 (K), R13.1: now also Q3.5 (D)
- net at U6.15 (HIDRV): now also Q3.1 (G)
- net at U6.13 (LODRV): now also Q4.1 (G)
- net TERM: no longer names the net of U6.4 (TS)
- no-connect marks 0 -> 2

Commit message: The Price
Parts:
- C14: MPN 22pF 35V 0603 -> 22pF 50V 0603
- C16: footprint Capacitor_SMD:C_1210_3225Metric -> Capacitor_SMD:C_Elec_4x5.4; MPN 4.7uF 35V 1210 -> EEEFK1V4R7AR
- C7: MPN 2.2uF 35V 1210 -> 2.2uF 50V 1210
Other:
- moved on the sheet: U6

Commit message: Lost Mariner
Parts:
- added C15: C3, Capacitor_SMD:C_0805_2012Metric, symbol Device:C
- added R14: R9, Resistor_SMD:R_0402_1005Metric, symbol Device:R
- added R17: R10, Resistor_SMD:R_0402_1005Metric, symbol Device:R
Connections:
- net GND: now also C15.1, R17.2; no longer U6.7 (TERM_EN)
- net TS: now reaches U6.4 (TS)
- net TS: now also R14.2, R17.1
- net at U6.6 (VREF): now also U6.7 (TERM_EN), C15.2, R14.1
- no-connect marks 2 -> 0
