File: kicad/Ryujin/Battery_Charger.kicad_sch (KiCad schematic)
At the start: 29 parts, among them Q3 Q1, Q4 Q2, U6 BQ24650

Commit message: Fade Out
Parts:
- R1: MPN 2 0805 -> 2 0805 1W
- R13: MPN 10 1206 -> 10 1206 0.25W
- RSR1: MPN WSL1206R0400FEA -> WSL1206R0200DEA
Changed lines of the file:
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@@
 			)
 		)
-		(property "MPN" "2 0805"
+		(property "MPN" "2 0805 1W"
 			(at 46.99 58.42 0)
 			(effects
@@
 	)
 	(symbol
+		(lib_name "SQJQ100E_1")
 		(lib_id "Transistor_FET:SQJQ100E")
 		(at 184.15 67.31 0)
@@
 			)
 		)
-		(property "MPN" "10 1206"
+		(property "MPN" "10 1206 0.25W"
 			(at 116.84 54.61 0)
 			(effects
@@
 	)
 	(symbol
+		(lib_name "LED_1")
 		(lib_id "Device:LED")
 		(at 140.97 100.33 0)
@@
 			)
 		)
-		(property "MPN" "WSL1206R0400FEA"
+		(property "MPN" "WSL1206R0200DEA"
 			(at 212.09 78.74 90)
 			(effects

Commit message: The Furies
Parts:
- removed D3, D4: LED, LED_SMD:LED_0603_1608Metric, symbol Device:LED
- removed Q3: Q1, Package_TO_SOT_SMD:LFPAK88, symbol Transistor_FET:SQJQ100E
- removed Q4: Q2, Package_TO_SOT_SMD:LFPAK88, symbol Transistor_FET:SQJQ100E
- removed R11: R7, Resistor_SMD:R_0402_1005Metric, symbol Device:R
- removed R12: R8, Resistor_SMD:R_0402_1005Metric, symbol Device:R
- added Q5, Q6: IRF7403, Package_SO:SOIC-8_3.9x4.9mm_P1.27mm, symbol Transistor_FET:IRF7403
Connections:
- net GND: now also Q6.1 (S), Q6.2 (S), Q6.3 (S)
- net at C11.2, L1.1, U6.14 (PH): now also Q5.1 (S), Q5.2 (S), Q5.3 (S), Q6.5 (D), Q6.6 (D), Q6.7 (D), Q6.8 (D)
- net at C9.1, D5.3 (K), R13.1: now also Q5.5 (D), Q5.6 (D), Q5.7 (D), Q5.8 (D)
- net at U6.15 (HIDRV): now also Q5.4 (G)
- net at U6.13 (LODRV): now also Q6.4 (G)
- no-connect marks 0 -> 2

Commit message: My Best Girl's Wedding
Parts:
- Q5, Q6: MPN IRF7403TRPBF -> IRF7469TRPBF
Changed lines of the file:
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@@
+	(wire
+		(pts
+			(xy 186.69 107.95) (xy 186.69 96.52)
+		)
+		(stroke
+			(width 0)
+			(type default)
+		)
+	)
 	(wire
 		(pts
@@
 		)
 	)
+	(netclass_flag ""
+		(length 2.54)
+		(shape round)
+		(at 200.66 78.74 0)
+		(fields_autoplaced yes)
+		(effects
+			(font
+				(size 1.27 1.27)
+			)
+			(justify left bottom)
+		)
+		(property "Netclass" "PWR"
+			(at 201.3585 76.2 0)
+			(effects
+				(font
+					(size 1.27 1.27)
+				)
+				(justify left)
+			)
+		)
+		(property "Component Class" ""
+			(at 38.1 52.07 0)
+			(effects
+				(font
+					(size 1.27 1.27)
+					(italic yes)
+				)
+			)
+		)
+	)
+	(netclass_flag ""
+		(length 2.54)
+		(shape round)
+		(at 186.69 104.14 270)
+		(fields_autoplaced yes)
+		(effects
+			(font
+				(size 1.27 1.27)
+			)
+			(justify right bottom)
+		)
+		(property "Netclass" "PWR"
+			(at 189.23 103.4415 90)
+			(effects
+				(font
+					(size 1.27 1.27)
+				)
+				(justify left)
+			)
+		)
+		(property "Component Class" ""
+			(at 24.13 77.47 0)
+			(effects
+				(font
+					(size 1.27 1.27)
+					(italic yes)
+				)
+			)
+		)
+	)
+	(netclass_flag ""
+		(length 2.54)
+		(shape round)
+		(at 186.69 76.2 270)
+		(fields_autoplaced yes)
+		(effects
+			(font
+				(size 1.27 1.27)
+			)
+			(justify right bottom)
+		)
+		(property "Netclass" "PWR"
+			(at 189.23 75.5015 90)
+			(effects
+				(font
+					(size 1.27 1.27)
+				)
+				(justify left)
+			)
+		)
+		(property "Component Class" ""
+			(at 24.13 49.53 0)
+			(effects
+				(font
+					(size 1.27 1.27)
+					(italic yes)
+				)
+			)
+		)
+	)
+	(netclass_flag ""
+		(length 2.54)
+		(shape round)
+		(at 46.99 64.77 90)
+		(fields_autoplaced yes)
+		(effects
+			(font
+				(size 1.27 1.27)
+			)
+			(justify left bottom)
+		)
+		(property "Netclass" "PWR"
+			(at 44.45 64.0715 90)
+			(effects
+				(font
+					(size 1.27 1.27)
+				)
+				(justify left)
+			)
+		)
+		(property "Component Class" ""
+			(at -115.57 38.1 0)
+			(effects
+				(font
+					(size 1.27 1.27)
+					(italic yes)
+				)
+			)
+		)
+	)
+	(netclass_flag ""
+		(length 2.54)
+		(shape round)
+		(at 116.84 48.26 0)
+		(fields_autoplaced yes)
+		(effects
+			(font
+				(size 1.27 1.27)
+			)
+			(justify left bottom)
+		)
+		(property "Netclass" "PWR"
+			(at 117.5385 45.72 0)
+			(effects
+				(font
+					(size 1.27 1.27)
+				)
+				(justify left)
+			)
+		)
+		(property "Component Class" ""
+			(at -45.72 21.59 0)
+			(effects
+				(font
+					(size 1.27 1.27)
+					(italic yes)
+				)
+			)
+		)
+	)
 	(symbol
 		(lib_id "Device:C")
@@
 			)
 		)
-		(property "MPN" "IRF7403TRPBF"
+		(property "MPN" "IRF7469TRPBF"
 			(at 184.15 91.44 0)
 			(effects
@@
 	(symbol
 		(lib_id "power:GND")
-		(at 186.69 96.52 0)
+		(at 186.69 107.95 0)
 		(unit 1)
 		(exclude_from_sim no)
@@
 		(fields_autoplaced yes)
 		(property "Reference" "#PWR042"
-			(at 186.69 102.87 0)
+			(at 186.69 114.3 0)
 			(effects
 				(font
@@
 		)
 		(property "Value" "GND"
-			(at 186.69 101.6 0)
+			(at 186.69 113.03 0)
 			(effects
 				(font
@@
 		)
 		(property "Footprint" ""
-			(at 186.69 96.52 0)
+			(at 186.69 107.95 0)
 			(effects
 				(font
@@
 		)
 		(property "Datasheet" ""
-			(at 186.69 96.52 0)
+			(at 186.69 107.95 0)
 			(effects
 				(font
@@
 		)
 		(property "Description" "Power symbol creates a global label with name \"GND\" , ground"
-			(at 186.69 96.52 0)
+			(at 186.69 107.95 0)
 			(effects
 				(font
@@
 			)
 		)
-		(property "MPN" "IRF7403TRPBF"
+		(property "MPN" "IRF7469TRPBF"
 			(at 184.15 67.31 0)
 			(effects

Commit message: The Dirty Half Dozen
Parts:
- added R11: 0, Resistor_SMD:R_0805_2012Metric, symbol Device:R
Connections:
- net GND: now also R11.1; no longer C15.1, C8.1, R15.2, R17.2, R3.2, U6.11 (GND), U6.17 (GND)
- new net GNDA: C15.1, C8.1, R11.2, R15.2, R17.2, R3.2, U6.11 (GND), U6.17 (GND)

Commit message: The Deliverer
Parts:
- R11: footprint Resistor_SMD:R_0805_2012Metric -> Resistor_SMD:R_0402_1005Metric; MPN 0 0805 -> 0 0402
Changed lines of the file:
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@@
 			)
 		)
-		(property "Footprint" "Resistor_SMD:R_0805_2012Metric"
+		(property "Footprint" "Resistor_SMD:R_0402_1005Metric"
 			(at 110.49 109.982 90)
 			(effects
@@
 			)
 		)
-		(property "MPN" "0 0805"
+		(property "MPN" "0 0402"
 			(at 110.49 111.76 90)
 			(effects
