File: kicad/Ryujin/Battery_Charger.kicad_sch (KiCad schematic)
At the start: 26 parts, among them Q5 IRF7403, Q6 IRF7403, U6 BQ24650

Commit message: Forget Me Not
Parts:
- removed R11: 0, Resistor_SMD:R_0402_1005Metric, symbol Device:R
Connections:
- net GNDA is gone; now on net GND: C15.1, C8.1, R15.2, R17.2, R3.2, U6.11 (GND), U6.17 (GND)

Commit message: Full Circle
Parts:
- removed Q5, Q6: IRF7403, Package_SO:SOIC-8_3.9x4.9mm_P1.27mm, symbol Transistor_FET:IRF7403
- added Q3: Si7288, footprints:SI7288DPT1GE3, symbol Vishay:Si7288
Connections:
- net GND: now also Q3.3 (S)
- net at C11.2, L1.1, U6.14 (PH): now also Q3.1 (S), Q3.10 (D), Q3.12 (D), Q3.5 (D), Q3.6 (D)
- net at C9.1, D5.3 (K), R13.1: now also Q3.11 (D), Q3.7 (D), Q3.8 (D), Q3.9 (D)
- net at U6.13 (LODRV): now also Q3.4 (G)
- net at U6.15 (HIDRV): now also Q3.2 (G)
Other:
- company: (none) -> Julius-Maximilians-Universität Würzburg
- title: (none) -> Ryujin
Changed lines of the file:
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@@
 	(generator_version "9.0")
 	(paper "A4")
+	(title_block
+		(title "Ryujin")
+		(date "2025-03-24")
+		(rev "44")
+		(company "Julius-Maximilians-Universität Würzburg")
+	)
 	(junction
 		(at 148.59 69.85)
@@
 	)
 	(junction
+		(at 186.69 86.36)
+		(diameter 0)
+		(color 0 0 0 0)
+	)
+	(junction
 		(at 219.71 78.74)
 		(diameter 0)
@@
 	)
 	(junction
+		(at 186.69 62.23)
+		(diameter 0)
+		(color 0 0 0 0)
+	)
+	(junction
 		(at 205.74 93.98)
 		(diameter 0)
@@
 	(wire
 		(pts
+			(xy 186.69 86.36) (xy 189.23 86.36)
+		)
+		(stroke
+			(width 0)
+			(type default)
+		)
+	)
+	(wire
+		(pts
 			(xy 95.25 74.93) (xy 95.25 77.47)
 		)
@@
 	(wire
 		(pts
+			(xy 186.69 62.23) (xy 189.23 62.23)
+		)
+		(stroke
+			(width 0)
+			(type default)
+		)
+	)
+	(wire
+		(pts
 			(xy 254 78.74) (xy 254 87.63)
 		)
@@
 	)
 	(symbol
+		(lib_id "Vishay:Si7288")
+		(at 184.15 91.44 0)
+		(unit 2)
+		(exclude_from_sim no)
+		(in_bom yes)
+		(on_board yes)
+		(dnp no)
+		(fields_autoplaced yes)
+		(property "Reference" "Q3"
+			(at 190.5 90.1699 0)
+			(effects
+				(font
+					(size 1.27 1.27)
+				)
+				(justify left)
+			)
+		)
+		(property "Value" "Si7288"
+			(at 190.5 92.7099 0)
+			(effects
+				(font
+					(size 1.27 1.27)
+				)
+				(justify left)
+			)
+		)
+		(property "Footprint" "footprints:SI7288DPT1GE3"
+			(at 189.23 91.44 0)
+			(effects
+				(font
+					(size 1.27 1.27)
+				)
+				(hide yes)
+			)
+		)
+		(property "Datasheet" "https://www.vishay.com/docs/65366/si7288dp.pdf"
+			(at 189.23 91.44 0)
+			(effects
+				(font
+					(size 1.27 1.27)
+				)
+				(hide yes)
+			)
+		)
+		(property "Description" "Dual NMOS transistor, 12 pin package"
+			(at 184.15 91.44 0)
+			(effects
+				(font
+					(size 1.27 1.27)
+				)
+				(hide yes)
+			)
+		)
+		(pin "7"
+		)
+		(pin "6"
+		)
+		(pin "3"
+		)
+		(pin "8"
+		)
+		(pin "4"
+		)
+		(pin "9"
+		)
+		(pin "10"
+		)
+		(pin "12"
+		)
+		(pin "5"
+		)
+		(pin "1"
+		)
+		(pin "2"
+		)
+		(pin "11"
+		)
+		(instances
+			(project ""
+				(path "/a03941d3-2006-4bae-a82d-663063c77238/5d8fcbd7-e8f6-4322-b7f5-743508fec2cc"
+					(reference "Q3")
+					(unit 2)
+				)
+			)
+		)
+	)
+	(symbol
 		(lib_id "power:GND")
 		(at 46.99 77.47 0)
@@
 	)
 	(symbol
+		(lib_id "Vishay:Si7288")
+		(at 184.15 67.31 0)
+		(unit 1)
+		(exclude_from_sim no)
+		(in_bom yes)
+		(on_board yes)
+		(dnp no)
+		(fields_autoplaced yes)
+		(property "Reference" "Q3"
+			(at 190.5 66.0399 0)
+			(effects
+				(font
+					(size 1.27 1.27)
+				)
+				(justify left)
+			)
+		)
+		(property "Value" "Si7288"
+			(at 190.5 68.5799 0)
+			(effects
+				(font
+					(size 1.27 1.27)
+				)
+				(justify left)
+			)
+		)
+		(property "Footprint" "footprints:SI7288DPT1GE3"
+			(at 189.23 67.31 0)
+			(effects
+				(font
+					(size 1.27 1.27)
+				)
+				(hide yes)
+			)
+		)
+		(property "Datasheet" "https://www.vishay.com/docs/65366/si7288dp.pdf"
+			(at 189.23 67.31 0)
+			(effects
+				(font
+					(size 1.27 1.27)
+				)
+				(hide yes)
+			)
+		)
+		(property "Description" "Dual NMOS transistor, 12 pin package"
+			(at 184.15 67.31 0)
+			(effects
+				(font
+					(size 1.27 1.27)
+				)
+				(hide yes)
+			)
+		)
+		(pin "9"
+		)
+		(pin "8"
+		)
+		(pin "4"
+		)
+		(pin "1"
+		)
+		(pin "11"
+		)
+		(pin "3"
+		)
+		(pin "10"
+		)
+		(pin "2"
+		)
+		(pin "12"
+		)
+		(pin "7"
+		)
+		(pin "5"
+		)
+		(pin "6"
+		)
+		(instances
+			(project ""
+				(path "/a03941d3-2006-4bae-a82d-663063c77238/5d8fcbd7-e8f6-4322-b7f5-743508fec2cc"
+					(reference "Q3")
+					(unit 1)
+				)
+			)
+		)
+	)
+	(symbol
 		(lib_id "power:GND")
 		(at 240.03 86.36 0)
@@
 	)
 	(symbol
-		(lib_id "Transistor_FET:IRF7403")
-		(at 184.15 91.44 0)
-		(unit 1)
-		(exclude_from_sim no)
-		(in_bom yes)
-		(on_board yes)
-		(dnp no)
-		(fields_autoplaced yes)
-		(property "Reference" "Q6"
-			(at 190.5 90.1699 0)
-			(effects
-				(font
-					(size 1.27 1.27)
-				)
-				(justify left)
-			)
-		)
-		(property "Value" "IRF7403"
-			(at 190.5 92.7099 0)
-			(effects
-				(font
-					(size 1.27 1.27)
-				)
-				(justify left)
-			)
-		)
-		(property "Footprint" "Package_SO:SOIC-8_3.9x4.9mm_P1.27mm"
-			(at 189.23 93.345 0)
-			(effects
-				(font
-					(size 1.27 1.27)
-					(italic yes)
-				)
-				(justify left)
-				(hide yes)
-			)
-		)
-		(property "Datasheet" "https://www.infineon.com/dgdl/irf7403pbf.pdf?fileId=5546d462533600a4015355fa23541b9c"
-			(at 189.23 95.25 0)
-			(effects
-				(font
-					(size 1.27 1.27)
-				)
-				(justify left)
-				(hide yes)
-			)
-		)
-		(property "Description" "9.7A Id, 30V Vds, N-Channel HEXFET Power MOSFET, SO-8"
-			(at 184.15 91.44 0)
-			(effects
-				(font
-					(size 1.27 1.27)
-				)
-				(hide yes)
-			)
-		)
-		(property "MPN" "IRF7469TRPBF"
-			(at 184.15 91.44 0)
-			(effects
-				(font
-					(size 1.27 1.27)
-				)
-				(hide yes)
-			)
-		)
-		(pin "1"
-		)
-		(pin "7"
-		)
-		(pin "4"
-		)
-		(pin "3"
-		)
-		(pin "6"
-		)
-		(pin "2"
-		)
-		(pin "8"
-		)
-		(pin "5"
-		)
-		(instances
-			(project "Ryujin"
-				(path "/a03941d3-2006-4bae-a82d-663063c77238/5d8fcbd7-e8f6-4322-b7f5-743508fec2cc"
-					(reference "Q6")
-					(unit 1)
-				)
-			)
-		)
-	)
-	(symbol
 		(lib_id "power:GND")
 		(at 85.09 74.93 270)
@@
 					(unit 1)
 				)
-			)
-		)
-	)
-	(symbol
-		(lib_id "Transistor_FET:IRF7403")
-		(at 184.15 67.31 0)
-		(unit 1)
-		(exclude_from_sim no)
-		(in_bom yes)
-		(on_board yes)
-		(dnp no)
-		(fields_autoplaced yes)
-		(property "Reference" "Q5"
-			(at 190.5 66.0399 0)
-			(effects
-				(font
-					(size 1.27 1.27)
-				)
-				(justify left)
-			)
-		)
-		(property "Value" "IRF7403"
-			(at 190.5 68.5799 0)
-			(effects
-				(font
-					(size 1.27 1.27)
-				)
-				(justify left)
-			)
-		)
-		(property "Footprint" "Package_SO:SOIC-8_3.9x4.9mm_P1.27mm"
-			(at 189.23 69.215 0)
-			(effects
-				(font
-					(size 1.27 1.27)
-					(italic yes)
-				)
-				(justify left)
-				(hide yes)
-			)
-		)
-		(property "Datasheet" "https://www.infineon.com/dgdl/irf7403pbf.pdf?fileId=5546d462533600a4015355fa23541b9c"
-			(at 189.23 71.12 0)
-			(effects
-				(font
-					(size 1.27 1.27)
-				)
-				(justify left)
-				(hide yes)
-			)
-		)
-		(property "Description" "9.7A Id, 30V Vds, N-Channel HEXFET Power MOSFET, SO-8"
-			(at 184.15 67.31 0)
-			(effects
-				(font
-					(size 1.27 1.27)
-				)
-				(hide yes)
-			)
-		)
-		(property "MPN" "IRF7469TRPBF"
-			(at 184.15 67.31 0)
-			(effects
-				(font
-					(size 1.27 1.27)
-				)
-				(hide yes)
-			)
-		)
-		(pin "1"
-		)
-		(pin "7"
-		)
-		(pin "4"
-		)
-		(pin "3"
-		)
-		(pin "6"
-		)
-		(pin "2"
-		)
-		(pin "8"
-		)
-		(pin "5"
-		)
-		(instances
-			(project ""
-				(path "/a03941d3-2006-4bae-a82d-663063c77238/5d8fcbd7-e8f6-4322-b7f5-743508fec2cc"
-					(reference "Q5")
-					(unit 1)
-				)

Commit message: Chariots of War
Parts:
- Q3: MPN (none) -> SI7288DP-T1-GE3
Changed lines of the file:
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@@
+			)
+		)
+		(property "MPN" "SI7288DP-T1-GE3"
+			(at 184.15 91.44 0)
+			(effects
+				(font
+					(size 1.27 1.27)
+				)
+				(hide yes)
 			)
 		)
@@
 			(at 184.15 67.31 0)
 			(effects
+				(font
+					(size 1.27 1.27)
+				)
+				(hide yes)
+			)
+		)
+		(property "MPN" "SI7288DP-T1-GE3"
+			(at 184.15 67.31 0)
+			(effects

Commit message: Is There a Doctor in the House?
Parts:
- added Q4: 2N7002, Package_TO_SOT_SMD:SOT-23, symbol Transistor_FET:2N7002
Connections:
- net GND: now also Q4.2 (S)
- net at R2.2, R3.1, U6.2 (MPPSET): now also Q4.3 (D)
- new net CE: Q4.1 (G)
Changed lines of the file:
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@@
 	)
 	(junction
+		(at 63.5 85.09)
+		(diameter 0)
+		(color 0 0 0 0)
+	)
+	(junction
 		(at 186.69 78.74)
 		(diameter 0)
@@
 	(wire
 		(pts
+			(xy 49.53 88.9) (xy 49.53 85.09)
+		)
+		(stroke
+			(width 0)
+			(type default)
+		)
+	)
+	(wire
+		(pts
 			(xy 63.5 48.26) (xy 78.74 48.26)
 		)
@@
 	(wire
 		(pts
-			(xy 63.5 82.55) (xy 63.5 87.63)
+			(xy 63.5 82.55) (xy 63.5 85.09)
 		)
 		(stroke
@@
 	(wire
 		(pts
+			(xy 36.83 93.98) (xy 41.91 93.98)
+		)
+		(stroke
+			(width 0)
+			(type default)
+		)
+	)
+	(wire
+		(pts
 			(xy 129.54 82.55) (xy 205.74 82.55)
 		)
@@
 	(wire
 		(pts
+			(xy 49.53 85.09) (xy 63.5 85.09)
+		)
+		(stroke
+			(width 0)
+			(type default)
+		)
+	)
+	(wire
+		(pts
 			(xy 105.41 60.96) (xy 116.84 60.96)
 		)
@@
 	(wire
 		(pts
+			(xy 63.5 85.09) (xy 63.5 87.63)
+		)
+		(stroke
+			(width 0)
+			(type default)
+		)
+	)
+	(wire
+		(pts
 			(xy 172.72 69.85) (xy 172.72 78.74)
 		)
@@
 	(wire
 		(pts
+			(xy 49.53 99.06) (xy 49.53 107.95)
+		)
+		(stroke
+			(width 0)
+			(type default)
+		)
+	)
+	(wire
+		(pts
 			(xy 129.54 87.63) (xy 133.35 87.63)
 		)
@@
 		)
 	)
+	(hierarchical_label "CE"
+		(shape input)
+		(at 36.83 93.98 180)
+		(effects
+			(font
+				(size 1.27 1.27)
+			)
+			(justify right)
+		)
+	)
 	(hierarchical_label "BAT+"
 		(shape output)
@@
 	(symbol
 		(lib_id "power:GND")
+		(at 49.53 107.95 0)
+		(unit 1)
+		(exclude_from_sim no)
+		(in_bom yes)
+		(on_board yes)
+		(dnp no)
+		(fields_autoplaced yes)
+		(property "Reference" "#PWR053"
+			(at 49.53 114.3 0)
+			(effects
+				(font
+					(size 1.27 1.27)
+				)
+				(hide yes)
+			)
+		)
+		(property "Value" "GND"
+			(at 49.53 113.03 0)
+			(effects
+				(font
+					(size 1.27 1.27)
+				)
+			)
+		)
+		(property "Footprint" ""
+			(at 49.53 107.95 0)
+			(effects
+				(font
+					(size 1.27 1.27)
+				)
+				(hide yes)
+			)
+		)
+		(property "Datasheet" ""
+			(at 49.53 107.95 0)
+			(effects
+				(font
+					(size 1.27 1.27)
+				)
+				(hide yes)
+			)
+		)
+		(property "Description" "Power symbol creates a global label with name \"GND\" , ground"
+			(at 49.53 107.95 0)
+			(effects
+				(font
+					(size 1.27 1.27)
+				)
+				(hide yes)
+			)
+		)
+		(pin "1"
+		)
+		(instances
+			(project "Ryujin"
+				(path "/a03941d3-2006-4bae-a82d-663063c77238/5d8fcbd7-e8f6-4322-b7f5-743508fec2cc"
+					(reference "#PWR053")
+					(unit 1)
+				)
+			)
+		)
+	)
+	(symbol
+		(lib_id "power:GND")
 		(at 170.18 87.63 90)
 		(unit 1)
@@
 					(unit 1)
 				)
+			)
+		)
+	)
+	(symbol
+		(lib_id "Transistor_FET:2N7002")
+		(at 46.99 93.98 0)
+		(unit 1)
+		(exclude_from_sim no)
+		(in_bom yes)
+		(on_board no)
+		(dnp no)
+		(fields_autoplaced yes)
+		(property "Reference" "Q4"
+			(at 53.34 92.7099 0)
+			(effects
+				(font
+					(size 1.27 1.27)
+				)
+				(justify left)
+			)
+		)
+		(property "Value" "2N7002"
+			(at 53.34 95.2499 0)
+			(effects
+				(font
+					(size 1.27 1.27)
+				)
+				(justify left)
+				(hide yes)
+			)
+		)
+		(property "Footprint" "Package_TO_SOT_SMD:SOT-23"
+			(at 52.07 95.885 0)
+			(effects
+				(font
+					(size 1.27 1.27)
+					(italic yes)
+				)
+				(justify left)
+				(hide yes)
+			)
+		)
+		(property "Datasheet" "https://www.onsemi.com/pub/Collateral/NDS7002A-D.PDF"
+			(at 52.07 97.79 0)
+			(effects
+				(font
+					(size 1.27 1.27)
+				)
+				(justify left)
+				(hide yes)
+			)
+		)
+		(property "Description" "0.115A Id, 60V Vds, N-Channel MOSFET, SOT-23"
+			(at 46.99 93.98 0)
+			(effects
+				(font
+					(size 1.27 1.27)
+				)
+				(hide yes)
+			)
+		)
+		(pin "3"
+		)
+		(pin "2"
+		)
+		(pin "1"
+		)
+		(instances
+			(project ""
+				(path "/a03941d3-2006-4bae-a82d-663063c77238/5d8fcbd7-e8f6-4322-b7f5-743508fec2cc"
+					(reference "Q4")
+					(unit 1)
+				)

Commit message: Orphan of War
Connections:
- no-connect marks 3 -> 2
Changed lines of the file:
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@@
 	)
 	(no_connect
-		(at 115.57 88.9)
-	)
-	(no_connect
 		(at 129.54 100.33)
 	)
@@
 			)
 		)
-		(property "Datasheet" "~"
+		(property "Datasheet" "../../docs/PDS1040.pdf"
 			(at 83.82 48.26 0)
 			(effects
@@
 		(exclude_from_sim no)
 		(in_bom yes)
-		(on_board no)
+		(on_board yes)
 		(dnp no)
 		(fields_autoplaced yes)

Commit message: The Convert
Parts:
- R15: MPN 100k 0402 -> 97.6k 0402
- R16: MPN 499k 0402 -> 536k 0402
Changed lines of the file:
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@@
 			)
 		)
-		(property "MPN" "100k 0402"
+		(property "MPN" "97.6k 0402"
 			(at 248.92 104.14 0)
 			(effects
@@
 			)
 		)
-		(property "MPN" "499k 0402"
+		(property "MPN" "536k 0402"
 			(at 248.92 91.44 0)
 			(effects

Commit message: Sacrifice, Part 1
Parts:
- C11, C13: MPN 0.1uF 35V 0805 -> C0805C104K6RACTU
- R1: footprint Resistor_SMD:R_0805_2012Metric -> Resistor_SMD:R_2512_6332Metric; MPN 2 0805 1W -> 2 5% 1W
Changed lines of the file:
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@@
 			)
 		)
-		(property "MPN" "0.1uF 35V 0805"
+		(property "MPN" "C0805C104K6RACTU"
 			(at 148.59 74.93 90)
 			(effects
@@
 			)
 		)
-		(property "Footprint" "Resistor_SMD:R_0805_2012Metric"
+		(property "Footprint" "Resistor_SMD:R_2512_6332Metric"
 			(at 45.212 58.42 90)
 			(effects
@@
 			)
 		)
-		(property "MPN" "2 0805 1W"
+		(property "MPN" "2 5% 1W"
 			(at 46.99 58.42 0)
 			(effects
@@
 			)
 		)
-		(property "MPN" "0.1uF 35V 0805"
+		(property "MPN" "C0805C104K6RACTU"
 			(at 205.74 88.9 90)
 			(effects
