File: kicad/Ryujin/volt_supp.kicad_sch (KiCad schematic)
At the start: 10 parts, among them SW1 AS11CH, U7 R-78E5.0-1.0, U8 LM66100DCK, U9 74LVC1G17

Commit message: Soul Possession
Parts:
- added D1: LED, LED_SMD:LED_0805_2012Metric, symbol Device:LED
- added R12: 330, Resistor_SMD:R_0603_1608Metric, symbol Device:R
Connections:
- net GND: now also D1.1 (K)
- net at R11.2, SW1.3 (B), U8.3 (~{CE})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: now also R12.1
- new net: D1.2 (A), R12.2

Commit message: A Friend in Need, Part 1
Parts:
- D1: footprint LED_SMD:LED_0805_2012Metric -> LED_SMD:LED_0603_1608Metric; MPN (none) -> LTST-C193KRKT-5A
- R12: value 330 -> 540; MPN 330 0603 -> 540 0603
Changed lines of the file:
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@@
 			)
 		)
-		(property "Footprint" "LED_SMD:LED_0805_2012Metric"
+		(property "Footprint" "LED_SMD:LED_0603_1608Metric"
 			(at 128.27 92.71 0)
 			(effects
@@
 		)
 		(property "Sim.Pins" "1=K 2=A"
+			(at 128.27 92.71 0)
+			(effects
+				(font
+					(size 1.27 1.27)
+				)
+				(hide yes)
+			)
+		)
+		(property "MPN" "LTST-C193KRKT-5A"
 			(at 128.27 92.71 0)
 			(effects
@@
 			)
 		)
-		(property "Value" "330"
+		(property "Value" "540"
 			(at 140.716 92.71 90)
 			(effects
@@
 			)
 		)
-		(property "MPN" "330 0603"
+		(property "MPN" "540 0603"
 			(at 138.43 92.71 0)
 			(effects

Commit message: A Friend in Need, Part 2
Parts:
- R12: value 540 -> 536; MPN 540 0603 -> 536 0603
Changed lines of the file:
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@@
 			)
 		)
-		(property "Value" "540"
+		(property "Value" "536"
 			(at 140.716 92.71 90)
 			(effects
@@
 			)
 		)
-		(property "MPN" "540 0603"
+		(property "MPN" "536 0603"
 			(at 138.43 92.71 0)
 			(effects

Commit message: A Family Affair
Connections:
- net VCC renamed VREF

Commit message: Give Me Liberté
Parts:
- R12: value 536 -> 590; MPN 536 0603 -> 590 0603
Changed lines of the file:
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@@
 			)
 		)
-		(property "Value" "536"
+		(property "Value" "590"
 			(at 140.716 92.71 90)
 			(effects
@@
 			)
 		)
-		(property "MPN" "536 0603"
+		(property "MPN" "590 0603"
 			(at 138.43 92.71 0)
 			(effects
