File: kicad/A2SDI12/A2SDI12.kicad_pcb (KiCad board)
At the start: 2 copper layers, 111.2 x 82 mm, 20 parts, among them J1 Conn_02x03_Odd_Even, J10 Conn_02x03_Odd_Even, J11 Conn_02x03_Odd_Even, J12 Conn_02x03_Odd_Even, J14 Screw_Terminal_01x04, J15 Screw_Terminal_01x04, J16 Screw_Terminal_01x04, J2 Conn_02x03_Odd_Even, J3 Screw_Terminal_01x04, J4 Screw_Terminal_01x04, J5 Conn_02x03_Odd_Even, J6 Screw_Terminal_01x04, J7 Conn_02x03_Odd_Even, J8 Screw_Terminal_01x03, J9 Screw_Terminal_01x03

Commit message: The Vanishing Dead
Parts:
- removed J7: Conn_02x03_Odd_Even, Connector_PinHeader_2.54mm:PinHeader_2x03_P2.54mm_Vertical
- moved J8 54.2 mm to (50.0, 53.0)
- moved A1 52.1 mm to (112.0, 49.0)
- moved H1 52.0 mm to (35.5, 20.5)
- moved H2 52.0 mm to (140.5, 20.5)
- moved H3 52.0 mm to (35.5, 95.5)
- moved H4 52.0 mm to (140.5, 95.5)
- moved J1 52.0 mm to (96.5, 40.0)
- moved J10 52.0 mm to (76.2, 73.5)
- moved J11 52.0 mm to (96.5, 73.5)
- moved J12 52.0 mm to (116.8, 73.5)
- moved J15 52.0 mm to (81.5, 87.5)
- moved J16 52.0 mm to (101.8, 87.5)
- moved J2 52.0 mm to (116.8, 40.0)
- moved J3 52.0 mm to (96.5, 28.5)
- moved J4 52.0 mm to (116.8, 28.5)
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Connections:
- J6 pad 1: Net-(J6-Pin_1) -> /A5
Routing:
- net /D7: track 58.6 -> 0.00 mm, vias 1 -> 0
- net /D5: track 57.6 -> 0.00 mm, vias 1 -> 0
- net Net-(J6-Pin_1): track 37.4 -> 0.00 mm, vias 1 -> 0
- net /GND: track 202.2 -> 219.6 mm, vias 2 -> 0
- net /3V3: track 140.1 -> 124.6 mm, vias 0 -> 2
- net /5V: track 148.7 -> 133.7 mm, vias 1 -> 2
- net Net-(J5-Pin_2): track 23.5 -> 29.2 mm
- net /D13: track 77.6 -> 82.6 mm
- net /A2: track 39.9 -> 35.8 mm
- net /A5: track 30.8 -> 26.7 mm
- net Net-(J2-Pin_2): track 28.7 -> 25.3 mm, vias 1 -> 0
- net /VIN: track 163.9 -> 166.4 mm
- net /A0: track 29.3 -> 30.9 mm
- net /A4: track 34.6 -> 33.5 mm
- net /A3: track 44.2 -> 43.6 mm
Other:
- board text removed: "ANL"
- board text removed: "INT"
- board text removed: "SIG"

Commit message: Unchained Heart
Parts:
- moved J9 0.50 mm to (125.5, 63.0)
Routing:
- net /3V3: track 124.6 -> 129.6 mm
- net /A2: track 35.8 -> 40.1 mm
- net /5V: track 133.7 -> 137.9 mm, vias 2 -> 1
- net /GND: track 219.6 -> 222.8 mm, vias 0 -> 1
- net Net-(J2-Pin_2): track 25.3 -> 23.5 mm
- net /A0: track 30.9 -> 29.3 mm
- net /VIN: track 166.4 -> 165.6 mm, vias 1 -> 0
- net /A3: track 43.6 -> 44.2 mm
Other:
- board size 111.2 x 82 mm -> 111.2 x 81 mm
