File: kicad/A2SDI12/A2SDI12.kicad_pcb (KiCad board)
At the start: 2 copper layers, 111.2 x 81 mm, 19 parts, among them J1 Conn_02x03_Odd_Even, J10 Conn_02x03_Odd_Even, J11 Conn_02x03_Odd_Even, J12 Conn_02x03_Odd_Even, J14 Screw_Terminal_01x04, J15 Screw_Terminal_01x04, J16 Screw_Terminal_01x04, J2 Conn_02x03_Odd_Even, J3 Screw_Terminal_01x04, J4 Screw_Terminal_01x04, J5 Conn_02x03_Odd_Even, J6 Screw_Terminal_01x04, J8 Screw_Terminal_01x03, J9 Screw_Terminal_01x03

Commit message: Cast a Giant Shadow
Connections:
- J14 pad 1: /A10 -> /A11
- J14 pad 2: /A11 -> /A10
- J15 pad 1: /A6 -> /A7
- J15 pad 2: /A7 -> /A6
- J16 pad 1: /A8 -> /A9
- J16 pad 2: /A9 -> /A8
Routing:
- net /A7: track 24.5 -> 31.7 mm
- net /A8: track 23.5 -> 29.2 mm
- net /A10: track 63.1 -> 57.8 mm
- net /A11: track 62.4 -> 67.5 mm
- net /A6: track 24.5 -> 22.4 mm
- net /A9: track 24.5 -> 22.4 mm

Commit message: Highway to Hades
Parts:
- added SW1: SW_Push, Button_Switch_THT:SW_PUSH_6mm, F.Cu at (53.0, 40.0)
Connections:
- A1 pad D0: unconnected-(A1-D0/RX-PadD0) -> /D0
Routing:
- net /D0: track 0.00 -> 34.1 mm
- net /GND: track 222.8 -> 211.6 mm
- net /5V: track 137.9 -> 139.3 mm, vias 1 -> 2
- net /VIN: track 165.6 -> 164.6 mm
- net /3V3: vias 2 -> 1

Commit message: The Sword of Veracity
Parts:
- SW1: footprint Button_Switch_THT:SW_PUSH_6mm -> Button_Switch_THT:SW_TH_Tactile_Omron_B3F-10xx
- moved J1 5.59 mm to (91.5, 42.5), turned to 90 degrees
- moved J2 5.59 mm to (111.8, 42.5), turned to 90 degrees
- moved J5 5.59 mm to (71.2, 42.5), turned to 90 degrees
Connections:
- A1 pad D0: /D0 -> unconnected-(A1-D0/RX-PadD0)
- A1 pad D5: /D5 -> unconnected-(A1-PadD5)
- SW1 pad 2: /D0 -> /D7
Routing:
- net /D7: track 0.00 -> 61.8 mm, vias 0 -> 1
- net /D0: track 34.1 -> 0.00 mm
- net /VIN: track 164.6 -> 176.1 mm
- net Net-(J5-Pin_2): track 29.2 -> 20.8 mm
- net /GND: track 211.6 -> 216.9 mm, vias 1 -> 0
- net /3V3: track 129.6 -> 124.9 mm, vias 1 -> 3
- net /5V: track 139.3 -> 143.3 mm, vias 2 -> 0
- net /A2: track 40.2 -> 36.8 mm
- net Net-(J1-Pin_2): track 23.5 -> 20.8 mm
- net Net-(J2-Pin_2): track 23.5 -> 20.8 mm
- net /A0: track 29.3 -> 31.7 mm
- net /A3: track 44.2 -> 42.2 mm
Other:
- board text added: "BUS"
- board text added: "RST"
- board text added: "SDI12"
- board text added: "V+"
- board text added: "V-"

Commit message: The Enforcer
Parts:
- removed SW1: SW_Push, Button_Switch_THT:SW_TH_Tactile_Omron_B3F-10xx
- added J7: Conn_02x02_Odd_Even, Connector_PinHeader_2.54mm:PinHeader_2x02_P2.54mm_Vertical, F.Cu at (48.5, 40.0)
Connections:
- A1 pad D0: unconnected-(A1-D0/RX-PadD0) -> /D0
- A1 pad D1: unconnected-(A1-D1/TX-PadD1) -> /D1
- A1 pad D7: /D7 -> unconnected-(A1-D7_INT4-PadD7)
Routing:
- net /D7: track 61.8 -> 0.00 mm, vias 1 -> 0
- net /D1: track 0.00 -> 50.4 mm, vias 0 -> 1
- net /D0: track 0.00 -> 44.6 mm, vias 0 -> 1
- net /5V: track 143.3 -> 165.2 mm, vias 0 -> 2
- net /VIN: track 176.1 -> 159.4 mm
- net /GND: track 216.9 -> 208.4 mm, vias 0 -> 1
- net /3V3: track 124.9 -> 120.6 mm, vias 3 -> 1
- net /A0: track 31.7 -> 29.3 mm
- net /A2: track 36.8 -> 39.2 mm
- net /A3: track 42.2 -> 43.9 mm
Other:
- board text added: "CHG"
- board text removed: "RST"

Commit message: Add files via upload
Parts:
- removed J7: Conn_02x02_Odd_Even, Connector_PinHeader_2.54mm:PinHeader_2x02_P2.54mm_Vertical
Routing:
- net /D1: track 50.4 -> 0.00 mm, vias 1 -> 0
- net /D0: track 44.6 -> 0.00 mm, vias 1 -> 0
- net /5V: track 165.2 -> 138.9 mm
- net /GND: track 208.4 -> 216.8 mm, vias 1 -> 0
- net /VIN: track 159.4 -> 162.5 mm
- net /3V3: track 120.6 -> 123.3 mm
Other:
- board text removed: "CHG"
