File: kicad/Ryujin/rev1/Ryujin.kicad_pcb (KiCad board)
At the start: 2 copper layers, 56 x 77 mm, 27 parts, among them J1 BAT, J2 SDI12, J3 Conn_01x14_Socket, J4 Conn_01x14_Socket, Q1 IRLML6244, U1 TXS0101DBV, U2 R-78E5.0-0.5, U3 W25Q32JVSS, U4 SHTC3

Commit message: Outcast
Other:
- board text removed: "2024-12-15"
- board text removed: "Ryujin"
Changed lines of the file:
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@@
-		)
-	)
-	(gr_text "Ryujin"
-		(at 187 190.5 0)
-		(layer "Cmts.User")
-		(effects
-			(font
-				(size 1.5 1.5)
-				(thickness 0.3)
-				(bold yes)
-			)
-			(justify left bottom)
-		)
-	)
-	(gr_text "2024-12-15"
-		(at 206.5 194 0)
-		(layer "Cmts.User")
-		(effects
-			(font
-				(size 1.5 1.5)
-				(thickness 0.3)
-				(bold yes)
-			)
-			(justify left bottom)
 		)
 	)
