File: kicad/AoQin/AoQin.kicad_sch (KiCad schematic)
At the start: 15 parts, among them J1 Conn_02x03_Odd_Even, J10 Conn_02x03_Odd_Even, J11 Conn_02x03_Odd_Even, J12 Conn_02x03_Odd_Even, J14 Screw_Terminal_01x04, J15 Screw_Terminal_01x04, J16 Screw_Terminal_01x04, J2 Conn_02x03_Odd_Even, J3 Screw_Terminal_01x04, J4 Screw_Terminal_01x04, J5 Conn_02x03_Odd_Even, J6 Screw_Terminal_01x04, J8 Screw_Terminal_01x03, J9 Screw_Terminal_01x03

Commit message: The Cave of Echoes
Parts:
- removed J14, J15, J16, J3, J4, J6: Screw_Terminal_01x04, TerminalBlock_Phoenix:TerminalBlock_Phoenix_MKDS-1,5-4-5.08_1x04_P5.08mm_Horizontal, symbol Connector:Screw_Terminal_01x04
- added J3, J7: Screw_Terminal_01x12, footprints:1869318, symbol Connector:Screw_Terminal_01x12
Connections:
- net A0: now also J7.2 (Pin_2)
- net A1: now also J7.1 (Pin_1)
- net A10: now also J3.10 (Pin_10)
- net A11: now also J3.9 (Pin_9)
- net A2: now also J7.6 (Pin_6)
- net A3: now also J7.5 (Pin_5)
- net A4: now also J7.10 (Pin_10)
- net A5: now also J7.9 (Pin_9)
- net A6: now also J3.2 (Pin_2)
- net A7: now also J3.1 (Pin_1)
- net A8: now also J3.6 (Pin_6)
- net A9: now also J3.5 (Pin_5)
- net GND: now also J3.11 (Pin_11), J3.3 (Pin_3), J3.7 (Pin_7), J7.11 (Pin_11), J7.3 (Pin_3), J7.7 (Pin_7)
- net at J11.2 (Pin_2), J11.4 (Pin_4), J11.6 (Pin_6): now also J3.4 (Pin_4)
- net at J10.2 (Pin_2), J10.4 (Pin_4), J10.6 (Pin_6): now also J3.12 (Pin_12)
- net at J2.2 (Pin_2), J2.4 (Pin_4), J2.6 (Pin_6): now also J7.8 (Pin_8)
- net at J5.2 (Pin_2), J5.4 (Pin_4), J5.6 (Pin_6): now also J7.12 (Pin_12)
- net at J12.2 (Pin_2), J12.4 (Pin_4), J12.6 (Pin_6): now also J3.8 (Pin_8)
- net at J1.2 (Pin_2), J1.4 (Pin_4), J1.6 (Pin_6): now also J7.4 (Pin_4)
Other:
- moved on the sheet: J1, J10, J11, J12, J2, J5

Commit message: The Sword of Veracity
Parts:
- removed J10, J11, J12, J5: Conn_02x03_Odd_Even, Connector_PinHeader_2.54mm:PinHeader_2x03_P2.54mm_Vertical, symbol Connector_Generic:Conn_02x03_Odd_Even
- J3, J7: MPN (none) -> MKDSN 1.5/12
Connections:
- net A0: now also J7.1 (Pin_1); no longer J7.2 (Pin_2)
- net A1: now also J7.2 (Pin_2); no longer J7.1 (Pin_1)
- net A10: now also J3.9 (Pin_9); no longer J3.10 (Pin_10)
- net A11: now also J3.10 (Pin_10); no longer J3.9 (Pin_9)
- net A2: now also J7.5 (Pin_5); no longer J7.6 (Pin_6)
- net A3: now also J7.6 (Pin_6); no longer J7.5 (Pin_5)
- net A4: now also J7.9 (Pin_9); no longer J7.10 (Pin_10)
- net A5: now also J7.10 (Pin_10); no longer J7.9 (Pin_9)
- net A6: now also J3.1 (Pin_1); no longer J3.2 (Pin_2)
- net A7: now also J3.2 (Pin_2); no longer J3.1 (Pin_1)
- net A8: now also J3.5 (Pin_5); no longer J3.6 (Pin_6)
- net A9: now also J3.6 (Pin_6); no longer J3.5 (Pin_5)
- net VIN2: now reaches J3.4 (Pin_4)
- net VIN2: now also J2.2 (Pin_2), J2.4 (Pin_4), J2.6 (Pin_6), J3.12 (Pin_12), J3.8 (Pin_8)
- net VIN1: now reaches J7.12 (Pin_12)
- net VIN1: now also J1.2 (Pin_2), J1.4 (Pin_4), J1.6 (Pin_6), J7.4 (Pin_4), J7.8 (Pin_8)
- net VIN renamed +12V
Other:
- moved on the sheet: J3, J7

Commit message: When a Man Loves a Woman
Parts:
- removed J1, J2: Conn_02x03_Odd_Even, Connector_PinHeader_2.54mm:PinHeader_2x03_P2.54mm_Vertical, symbol Connector_Generic:Conn_02x03_Odd_Even
- removed J3, J7: Screw_Terminal_01x12, footprints:1869318, symbol Connector:Screw_Terminal_01x12
- added J1, J2, J3, J4, J5, J6: 1869253, footprints:SMKDSN_15_6_508, symbol PheonixContact:1869253
- added J15, J16, J7: Conn_02x03_Odd_Even, Connector_PinHeader_2.54mm:PinHeader_2x03_P2.54mm_Vertical, symbol Connector_Generic:Conn_02x03_Odd_Even
Connections:
- net +12V: now also J15.1 (Pin_1), J16.1 (Pin_1)
- net 3V3: now also J15.5 (Pin_5), J16.5 (Pin_5)
- net 5V: now also J15.3 (Pin_3), J16.3 (Pin_3)
- net A0: now also J1.3
- net A1: now also J1.4
- net A10: now also J6.3
- net A11: now also J6.4
- net A2: now also J2.3
- net A3: now also J2.4
- net A4: now also J3.3
- net A5: now also J3.4
- net A6: now also J4.3
- net A7: now also J4.4
- net A8: now also J5.3
- net A9: now also J5.4
- net GND: now also J1.1, J1.6, J2.1, J2.6, J3.1, J3.6, J4.1, J4.6, J5.1, J5.6, J6.1, J6.6
- net VIN1: now also J1.2, J15.2 (Pin_2), J15.4 (Pin_4), J15.6 (Pin_6), J2.2, J3.2, J4.2, J5.2, J6.2
- net VIN2: now also J1.5, J16.2 (Pin_2), J16.4 (Pin_4), J16.6 (Pin_6), J2.5, J3.5, J4.5, J5.5, J6.5

Commit message: Regrets… I've Had a Few
Parts:
- removed J1, J2, J3, J4, J5, J6: 1869253, footprints:SMKDSN_15_6_508, symbol PheonixContact:1869253
- removed J15, J16, J7: Conn_02x03_Odd_Even, Connector_PinHeader_2.54mm:PinHeader_2x03_P2.54mm_Vertical, symbol Connector_Generic:Conn_02x03_Odd_Even
- added J1, J2: Conn_02x03_Odd_Even, Connector_PinHeader_2.54mm:PinHeader_2x03_P2.54mm_Vertical, symbol Connector_Generic:Conn_02x03_Odd_Even
- added J3, J7: Screw_Terminal_01x12, footprints:1869318, symbol Connector:Screw_Terminal_01x12
Connections:
- net +12V: now also J1.1 (Pin_1), J2.1 (Pin_1)
- net 3V3: now also J1.5 (Pin_5), J2.5 (Pin_5)
- net 5V: now also J1.3 (Pin_3), J2.3 (Pin_3)
- net A0: now also J7.1 (Pin_1)
- net A1: now also J7.2 (Pin_2)
- net A10: now also J3.9 (Pin_9)
- net A11: now also J3.10 (Pin_10)
- net A2: now also J7.5 (Pin_5)
- net A3: now also J7.6 (Pin_6)
- net A4: now also J7.9 (Pin_9)
- net A5: now also J7.10 (Pin_10)
- net A6: now also J3.1 (Pin_1)
- net A7: now also J3.2 (Pin_2)
- net A8: now also J3.5 (Pin_5)
- net A9: now also J3.6 (Pin_6)
- net GND: now also J3.11 (Pin_11), J3.3 (Pin_3), J3.7 (Pin_7), J7.11 (Pin_11), J7.3 (Pin_3), J7.7 (Pin_7)
- net VIN1: now also J1.2 (Pin_2), J1.4 (Pin_4), J1.6 (Pin_6), J7.12 (Pin_12), J7.4 (Pin_4), J7.8 (Pin_8)
- net VIN2: now also J2.2 (Pin_2), J2.4 (Pin_4), J2.6 (Pin_6), J3.12 (Pin_12), J3.4 (Pin_4), J3.8 (Pin_8)

Commit message: Web of Desire
Parts:
- removed J3, J7: Screw_Terminal_01x12, footprints:1869318, symbol Connector:Screw_Terminal_01x12
- added J10, J3, J4, J5, J6, J7: 1869237, footprints:SMKDSN_15_4_508, symbol PheonixContact:1869237
Connections:
- net A0: now also J3.1
- net A1: now also J4.1
- net A10: now also J7.2
- net A11: now also J10.2
- net A2: now also J5.1
- net A3: now also J6.1
- net A4: now also J7.1
- net A5: now also J10.1
- net A6: now also J3.2
- net A7: now also J4.2
- net A8: now also J5.2
- net A9: now also J6.2
- net GND: now also J10.3, J3.3, J4.3, J5.3, J6.3, J7.3
- net VIN1: now also J3.4, J4.4, J5.4
- net VIN2: now also J10.4, J6.4, J7.4

Commit message: Prodigal Sister
Parts:
- J10, J3, J4, J5, J6, J7: MPN (none) -> 1869237
Connections:
- net A0: now also J10.2; no longer J3.1
- net A1: now also J10.1; no longer J4.1
- net A10: now also J3.2; no longer J7.2
- net A11: now also J3.1; no longer J10.2
- net A2: now also J7.2; no longer J5.1
- net A3: now also J7.1; no longer J6.1
- net A4: now also J6.2; no longer J7.1
- net A5: now also J6.1; no longer J10.1
- net A6: now also J5.2; no longer J3.2
- net A7: now also J5.1; no longer J4.2
- net A8: now also J4.2; no longer J5.2
- net A9: now also J4.1; no longer J6.2

Commit message: ...and Fancy Free
Parts:
- removed J2: Conn_02x03_Odd_Even, Connector_PinHeader_2.54mm:PinHeader_2x03_P2.54mm_Vertical, symbol Connector_Generic:Conn_02x03_Odd_Even
- added R1: 226k, Resistor_THT:R_Axial_DIN0207_L6.3mm_D2.5mm_P7.62mm_Horizontal, symbol Device:R
- added S1: 2454982-4, footprints:24549824, symbol 2454982-4:2454982-4
Connections:
- net A0: now also S1.B6
- net A10: now also S1.B1
- net A2: now also S1.B5
- net A4: now also S1.B4
- net A6: now also S1.B3
- net A8: now also S1.B2
- net GND: now also R1.1
- net VIN1: no longer J1.2 (Pin_2), J1.4 (Pin_4), J1.6 (Pin_6), J3.4, J4.4
- net VIN2 renamed VIN
- net VIN: now also J1.2 (Pin_2), J1.4 (Pin_4), J1.6 (Pin_6), J3.4, J4.4
- new net: R1.2, S1.A1, S1.A2, S1.A3, S1.A4, S1.A5, S1.A6

Commit message: If I Had a Hammer
Parts:
- removed R1: 226k, Resistor_THT:R_Axial_DIN0207_L6.3mm_D2.5mm_P7.62mm_Horizontal, symbol Device:R
- removed S1: 2454982-4, footprints:24549824, symbol 2454982-4:2454982-4
- added RN1, RN2: 5.1k, Resistor_THT:R_Array_SIP7, symbol Device:R_Network06
Connections:
- net 5V: now also RN1.1 (common), RN2.1 (common)
- net A0: now also RN2.7 (R6)
- net A1: now also RN2.6 (R5)
- net A10: now also RN1.6 (R5)
- net A11: now also RN1.7 (R6)
- net A2: now also RN2.5 (R4)
- net A3: now also RN2.4 (R3)
- net A4: now also RN2.3 (R2)
- net A5: now also RN2.2 (R1)
- net A6: now also RN1.2 (R1)
- net A7: now also RN1.3 (R2)
- net A8: now also RN1.4 (R3)
- net A9: now also RN1.5 (R4)
Other:
- moved on the sheet: J10, J3, J4, J5, J6, J7
