File: kicad/AoQin/AoQin.kicad_sch (KiCad schematic)
At the start: 8 parts, among them J1 Conn_02x03_Odd_Even, J2 Conn_02x03_Odd_Even, J3 1869237, J8 Screw_Terminal_01x03, J9 Screw_Terminal_01x03

Commit message: Armageddon Now: Part 1
Parts:
- removed J2: Conn_02x03_Odd_Even, Connector_PinHeader_2.54mm:PinHeader_2x03_P2.54mm_Vertical, symbol Connector_Generic:Conn_02x03_Odd_Even
- removed J3: 1869237, footprints:SMKDSN_15_4_508, symbol PheonixContact:1869237
- removed S2: 2454982-4, footprints:24549824, symbol TEConnectivity:2454982-4
- added J10, J5, J6, J7, J8, J9: 1985218, footprints:PTSA_15_4_35_Z, symbol PheonixContact:1985218
- added S1: 2454982-4, footprints:24549824, symbol TEConnectivity:2454982-4
- R13: value 10k -> 100k; MPN 10k -> 100k
- renumbered J9 to J1, J8 to J2, J1 to J3
Connections:
- net +12V: no longer J3.1 (Pin_1)
- net A0: now also J8.3
- net A1: now also J8.4
- net A10: now also J7.3
- net A11: now also J7.4
- net A2: now also J9.3
- net A3: now also J9.4
- net A4: now also J10.3
- net A5: now also J10.4
- net A6: now also J5.3
- net A7: now also J5.4
- net A8: now also J6.3
- net A9: now also J6.4
- net GND: now also J10.2, J5.2, J6.2, J7.2, J8.2, J9.2
- net VIN1: now also J10.1, J5.1, J6.1, J7.1, J8.1, J9.1; no longer J3.2 (Pin_2), J3.4 (Pin_4), J3.6 (Pin_6)
- new net VIN: J3.2 (Pin_2), J3.4 (Pin_4), J3.6 (Pin_6)

Commit message: Armageddon Now: Part 2
Parts:
- added R1, R2: 100k, Resistor_THT:R_Axial_DIN0204_L3.6mm_D1.6mm_P7.62mm_Horizontal, symbol Device:R
- added U1: PCF8574AP, Package_DIP:DIP-20_W7.62mm, symbol Interface_Expansion:PCF8574AP
Connections:
- net 5V: now also S1.B1, S1.B2, S1.B3, S1.B4, S1.B5, S1.B6, R1.2, R2.2, U1.1 (A0), U1.16 (VDD)
- net GND: now also U1.2 (A1), U1.3 (A2), U1.8 (GND)
- net at S1.A1: now also U1.4 (P0)
- net at S1.A2: now also U1.5 (P1)
- net at S1.A3: now also U1.6 (P2)
- net at S1.A4: now also U1.7 (P3)
- net at S1.A5: now also U1.9 (P4)
- net at S1.A6: now also U1.10 (P5)
- net SDA: now reaches A1.D2 (D2/SDA)
- net SDA: now also R2.1, U1.15 (SDA)
- net SCL: now reaches A1.D3 (D3/SCL)
- net SCL: now also R1.1, U1.14 (SCL)
Other:
- moved on the sheet: S1

Commit message: Hero's Heart
Parts:
- removed R1, R2: 100k, Resistor_THT:R_Axial_DIN0204_L3.6mm_D1.6mm_P7.62mm_Horizontal, symbol Device:R
- removed S1: 2454982-4, footprints:24549824, symbol TEConnectivity:2454982-4
- removed U1: PCF8574AP, Package_DIP:DIP-20_W7.62mm, symbol Interface_Expansion:PCF8574AP
- added J4: Conn_02x03_Odd_Even, Connector_PinHeader_2.54mm:PinHeader_2x03_P2.54mm_Vertical, symbol Connector_Generic:Conn_02x03_Odd_Even
- added S2: NDS-06-V, footprints:NDS06V, symbol Apem:NDS-06-V
Connections:
- net VIN is gone; now on net VIN1: J3.2 (Pin_2), J3.4 (Pin_4), J3.6 (Pin_6)
- net +12V: now also J3.1 (Pin_1), J4.1 (Pin_1)
- net 3V3: now also J4.5 (Pin_5)
- net 5V: now also J4.3 (Pin_3)
- net GND: now also S2.10 (NO_4), S2.11 (NO_5), S2.12 (NO_6), S2.7 (NO_1), S2.8 (NO_2), S2.9 (NO_3)
- net VIN1: no longer J10.1, J8.1, J9.1
- net D0: now reaches A1.D0 (D0/RX)
- net D0: now also S2.1 (COM_1)
- net D1: now reaches A1.D1 (D1/TX)
- net D1: now also S2.2 (COM_2)
- net D5: now reaches A1.D5
- net D5: now also S2.5 (COM_5)
- net D7: now reaches A1.D7 (D7_INT4)
- net D7: now also S2.6 (COM_6)
- net SCL renamed D3
- net D3: now also S2.4 (COM_4)
- net SDA renamed D2
- net D2: now also S2.3 (COM_3)
- new net VIN2: J10.1, J4.2 (Pin_2), J4.4 (Pin_4), J4.6 (Pin_6), J8.1, J9.1

Commit message: Dreamworker
Parts:
- removed J1, J2: Screw_Terminal_01x03, TerminalBlock_Phoenix:TerminalBlock_Phoenix_MKDS-1,5-3-5.08_1x03_P5.08mm_Horizontal, symbol Connector:Screw_Terminal_01x03
- added J1, J2: Screw_Terminal_01x04, TerminalBlock_Phoenix:TerminalBlock_Phoenix_MKDS-1,5-4-5.08_1x04_P5.08mm_Horizontal, symbol Connector:Screw_Terminal_01x04
- added J11: Conn_02x02_Odd_Even, Connector_PinHeader_2.54mm:PinHeader_2x02_P2.54mm_Vertical, symbol Connector_Generic:Conn_02x02_Odd_Even
Connections:
- net +12V: now also J1.2 (Pin_2), J11.3 (Pin_3), J2.2 (Pin_2); no longer A1.VIN
- net D13: now also J1.4 (Pin_4), J2.4 (Pin_4)
- net GND: now also J1.3 (Pin_3), J2.3 (Pin_3)
- new net +12VCC: J1.1 (Pin_1), J11.1 (Pin_1), J2.1 (Pin_1)
- new net VCC: A1.VIN, J11.2 (Pin_2), J11.4 (Pin_4)

Commit message: Stranger and Stranger
Connections:
- net A4: now also J5.3; no longer J10.3
- net A5: now also J5.4; no longer J10.4
- net D2: now also J10.2; no longer S2.3 (COM_3)
- net D3: now also J10.4; no longer S2.4 (COM_4)
- net D5: now also S2.4 (COM_4); no longer S2.5 (COM_5)
- net GND: now also J10.1, J10.3; no longer J10.2
- net VIN2: no longer J10.1
- net A6 renamed D4
- net D4: now also S2.3 (COM_3); no longer J5.3
- net A7 renamed D6
- net D6: now also S2.5 (COM_5); no longer J5.4
Changed lines of the file:
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@@
-		)
-	)
-	(label "GND"
-		(at 228.6 132.08 0)
-		(effects
-			(font
-				(size 1.27 1.27)
-			)
-			(justify left bottom)
 		)
 	)
@@
 		)
 	)
+	(label "D4"
+		(at 130.81 127 0)
+		(effects
+			(font
+				(size 1.27 1.27)
+			)
+			(justify left bottom)
+		)
+	)
 	(label "A5"
 		(at 121.92 64.77 0)
@@
 		)
 	)
-	(label "D5"
+	(label "D6"
 		(at 130.81 132.08 0)
 		(effects
@@
 			)
 			(justify left bottom)
+		)
+	)
+	(label "GND"
+		(at 266.7 132.08 180)
+		(effects
+			(font
+				(size 1.27 1.27)
+			)
+			(justify right bottom)
 		)
 	)
@@
 		)
 	)
-	(label "A4"
-		(at 266.7 134.62 180)
-		(effects
-			(font
-				(size 1.27 1.27)
-			)
-			(justify right bottom)
-		)
-	)
 	(label "VCC"
 		(at 121.92 85.09 0)
@@
 		)
 	)
+	(label "D5"
+		(at 130.81 129.54 0)
+		(effects
+			(font
+				(size 1.27 1.27)
+			)
+			(justify left bottom)
+		)
+	)
 	(label "VIN1"
 		(at 82.55 124.46 180)
@@
 		)
 	)
-	(label "A5"
-		(at 228.6 134.62 0)
-		(effects
-			(font
-				(size 1.27 1.27)
-			)
-			(justify left bottom)
-		)
-	)
 	(label "GND"
 		(at 44.45 124.46 0)
@@
 	)
 	(label "GND"
+		(at 266.7 134.62 180)
+		(effects
+			(font
+				(size 1.27 1.27)
+			)
+			(justify right bottom)
+		)
+	)
+	(label "GND"
 		(at 44.45 157.48 0)
+		(effects
+			(font
+				(size 1.27 1.27)
+			)
+			(justify left bottom)
+		)
+	)
+	(label "D2"
+		(at 228.6 132.08 0)
 		(effects
 			(font
@@
 		)
 	)
-	(label "A7"
+	(label "A5"
 		(at 44.45 127 0)
 		(effects
@@
 		)
 	)
-	(label "VIN2"
-		(at 266.7 132.08 180)
-		(effects
-			(font
-				(size 1.27 1.27)
-			)
-			(justify right bottom)
-		)
-	)
 	(label "5V"
 		(at 234.95 76.2 0)
@@
 		)
 	)
-	(label "D2"
-		(at 130.81 127 0)
-		(effects
-			(font
-				(size 1.27 1.27)
-			)
-			(justify left bottom)
-		)
-	)
 	(label "3V3"
 		(at 50.8 111.76 0)
@@
 	)
 	(label "D3"
-		(at 130.81 129.54 0)
-		(effects
-			(font
-				(size 1.27 1.27)
-			)
-			(justify left bottom)
-		)
-	)
-	(label "A6"
+		(at 228.6 134.62 0)
+		(effects
+			(font
+				(size 1.27 1.27)
+			)
+			(justify left bottom)
+		)
+	)
+	(label "D4"
 		(at 190.5 49.53 180)
 		(effects
@@
 		)
 	)
-	(label "A7"
+	(label "D6"
 		(at 190.5 54.61 180)
 		(effects
@@
 		)
 	)
-	(label "A6"
+	(label "A4"
 		(at 82.55 127 180)
 		(effects

Commit message: A Necessary Evil
Parts:
- removed J10, J7: 1985218, footprints:PTSA_15_4_35_Z, symbol PheonixContact:1985218
- added J10, J7: 1985195, footprints:1985195, symbol PheonixContact:1985195
- added J12: 1985218, footprints:PTSA_15_4_35_Z, symbol PheonixContact:1985218
Connections:
- net A10: now also J12.3
- net A11: now also J12.4
- net D0: now also J7.1; no longer S2.1 (COM_1)
- net D1: now also J10.1; no longer S2.2 (COM_2)
- net D13: no longer J1.4 (Pin_4), R13.1
- net D4: no longer S2.3 (COM_3)
- net D5: no longer S2.4 (COM_4)
- net D6: no longer S2.5 (COM_5)
- net D7: no longer S2.6 (COM_6)
- net GND: now also J10.2, J12.2, J7.2
- net VIN1: now also J12.1
- net D11: now reaches A1.D11
- net A8 renamed A6
- net A6: no longer A1.D8
- net A9 renamed A7
- net A7: no longer A1.D9
- net D2 renamed SDA
- net D3 renamed SCL
- new net D8: A1.D8
- new net D9: A1.D9, J1.4 (Pin_4), R13.1
