File: kicad/AoQin/AoQin.kicad_sch (KiCad schematic)
At the start: 15 parts, among them J1 Screw_Terminal_01x04, J10 1985195, J11 Conn_02x02_Odd_Even, J12 1985218, J2 Screw_Terminal_01x04, J3 Conn_02x03_Odd_Even, J4 Conn_02x03_Odd_Even, J5 1985218, J6 1985218, J7 1985195, J8 1985218, J9 1985218

Commit message: Gabrielle's Hope
Parts:
- removed J1, J2: Screw_Terminal_01x04, TerminalBlock_Phoenix:TerminalBlock_Phoenix_MKDS-1,5-4-5.08_1x04_P5.08mm_Horizontal, symbol Connector:Screw_Terminal_01x04
- removed J10, J7: 1985195, footprints:1985195, symbol PheonixContact:1985195
- removed J11: Conn_02x02_Odd_Even, Connector_PinHeader_2.54mm:PinHeader_2x02_P2.54mm_Vertical, symbol Connector_Generic:Conn_02x02_Odd_Even
- added J1, J2: Conn_01x03_Socket, Connector_Wire:SolderWire-0.5sqmm_1x03_P4.6mm_D0.9mm_OD2.1mm, symbol Connector:Conn_01x03_Socket
- added J10: 1985218, footprints:PTSA_15_4_35_Z, symbol PheonixContact:1985218
Connections:
- net D4 is gone; now on net A6: A1.D4
- net D6 is gone; now on net A7: A1.D6
- net SCL is gone; now on net D3: A1.D3 (D3/SCL)
- net SDA is gone; now on net D2: A1.D2 (D2/SDA)
- net +12V: now also J1.1 (Pin_1), J2.1 (Pin_1)
- net A4: now also J10.3; no longer J5.3
- net A5: now also J10.4; no longer J5.4
- net A6: now also J5.3; no longer J6.3
- net A7: now also J5.4; no longer J6.4
- net D0: now also S2.6 (COM_6)
- net D1: now also S2.5 (COM_5)
- net D11: now also R13.1, J1.3 (Pin_3), J2.3 (Pin_3)
- net D5: now also S2.2 (COM_2)
- net D7: now also S2.1 (COM_1)
- net GND: now also J1.2 (Pin_2), J10.2, J2.2 (Pin_2)
- net VIN2: now also J10.1
- net D3: now reaches S2.3 (COM_3)
- net D2: now reaches S2.4 (COM_4)
- net D13: no longer names the net of A1.D13
- net D8 renamed A8
- net A8: now also J6.3
- net D9 renamed A9
- net A9: now also J6.4; no longer R13.1
- no-connect marks 1 -> 9

Commit message: The King of Assassins
Connections:
- net D11: now also S2.1 (COM_1); no longer J1.3 (Pin_3), J2.3 (Pin_3), R13.1
- net D7: now also J1.3 (Pin_3), J2.3 (Pin_3), R13.1; no longer S2.1 (COM_1)
Changed lines of the file:
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@@
 		)
 	)
-	(label "D11"
+	(label "D7"
 		(at 24.13 25.4 0)
 		(effects
@@
 		)
 	)
-	(label "D11"
+	(label "D7"
 		(at 20.32 44.45 0)
 		(effects
@@
 		)
 	)
-	(label "D7"
+	(label "D11"
 		(at 130.81 121.92 0)
 		(effects

Commit message: Cradle of Hope
Parts:
- added H1, H2, H3, H4: MountingHole_Pad, MountingHole:MountingHole_3.5mm_Pad, symbol Mechanical:MountingHole_Pad
Connections:
- net GND: now also H1.1, H2.1, H3.1, H4.1

Commit message: The Reckoning
Parts:
- removed H4: MountingHole_Pad, MountingHole:MountingHole_3.5mm_Pad, symbol Mechanical:MountingHole_Pad
- removed J4: Conn_02x03_Odd_Even, Connector_PinHeader_2.54mm:PinHeader_2x03_P2.54mm_Vertical, symbol Connector_Generic:Conn_02x03_Odd_Even
Connections:
- net VIN2 is gone; now on net VIN: J10.1, J8.1, J9.1
- net A0: now also J5.3; no longer J8.3
- net A1: now also J5.4; no longer J8.4
- net A10: now also J10.3; no longer J12.3
- net A11: now also J10.4; no longer J12.4
- net A2: now also J6.3; no longer J9.3
- net A3: now also J6.4; no longer J9.4
- net A4: now also J8.3; no longer J10.3
- net A5: now also J8.4; no longer J10.4
- net A6: now also J9.3; no longer J5.3
- net A7: now also J9.4; no longer J5.4
- net A8: now also J12.3; no longer J6.3
- net A9: now also J12.4; no longer J6.4
- net VIN1 renamed VIN
Other:
- moved on the sheet: J10, J12, J5, J6, J8, J9

Commit message: Prometheus
Connections:
- net VCC is gone; now on net +12V: A1.VIN
Changed lines of the file:
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@@
-		)
-	)
-	(label "VCC"
-		(at 121.92 85.09 0)
-		(effects
-			(font
-				(size 1.27 1.27)
-			)
-			(justify left bottom)
 		)
 	)
@@
 			)
 			(justify right bottom)
-		)
-	)
-	(label "GND"
-		(at 121.92 92.71 0)
-		(effects
-			(font
-				(size 1.27 1.27)
-			)
-			(justify left bottom)
 		)
 	)
@@
 	)
 	(symbol
+		(lib_id "power:GND")
+		(at 121.92 92.71 270)
+		(unit 1)
+		(exclude_from_sim no)
+		(in_bom yes)
+		(on_board yes)
+		(dnp no)
+		(fields_autoplaced yes)
+		(property "Reference" "#PWR09"
+			(at 115.57 92.71 0)
+			(effects
+				(font
+					(size 1.27 1.27)
+				)
+				(hide yes)
+			)
+		)
+		(property "Value" "GND"
+			(at 118.11 92.7099 90)
+			(effects
+				(font
+					(size 1.27 1.27)
+				)
+				(justify right)
+			)
+		)
+		(property "Footprint" ""
+			(at 121.92 92.71 0)
+			(effects
+				(font
+					(size 1.27 1.27)
+				)
+				(hide yes)
+			)
+		)
+		(property "Datasheet" ""
+			(at 121.92 92.71 0)
+			(effects
+				(font
+					(size 1.27 1.27)
+				)
+				(hide yes)
+			)
+		)
+		(property "Description" "Power symbol creates a global label with name \"GND\" , ground"
+			(at 121.92 92.71 0)
+			(effects
+				(font
+					(size 1.27 1.27)
+				)
+				(hide yes)
+			)
+		)
+		(pin "1"
+		)
+		(instances
+			(project "AoQin"
+				(path "/91dda452-9985-4be5-905c-71f5be143fcf"
+					(reference "#PWR09")
+					(unit 1)
+				)
+			)
+		)
+	)
+	(symbol
 		(lib_id "PheonixContact:1985218")
 		(at 85.09 147.32 0)
@@
 					(unit 1)
 				)
+			)
+		)
+	)
+	(symbol
+		(lib_id "power:+12V")
+		(at 121.92 85.09 90)
+		(unit 1)
+		(exclude_from_sim no)
+		(in_bom yes)
+		(on_board yes)
+		(dnp no)
+		(property "Reference" "#PWR08"
+			(at 125.73 85.09 0)
+			(effects
+				(font
+					(size 1.27 1.27)
+				)
+				(hide yes)
+			)
+		)
+		(property "Value" "+12V"
+			(at 118.11 85.0899 90)
+			(effects
+				(font
+					(size 1.27 1.27)
+				)
+				(justify left)
+			)
+		)
+		(property "Footprint" ""
+			(at 121.92 85.09 0)
+			(effects
+				(font
+					(size 1.27 1.27)
+				)
+				(hide yes)
+			)
+		)
+		(property "Datasheet" ""
+			(at 121.92 85.09 0)
+			(effects
+				(font
+					(size 1.27 1.27)
+				)
+				(hide yes)
+			)
+		)
+		(property "Description" "Power symbol creates a global label with name \"+12V\""
+			(at 121.92 85.09 0)
+			(effects
+				(font
+					(size 1.27 1.27)
+				)
+				(hide yes)
+			)
+		)
+		(pin "1"
+		)
+		(instances
+			(project "AoQin"
+				(path "/91dda452-9985-4be5-905c-71f5be143fcf"
+					(reference "#PWR08")
+					(unit 1)
+				)

Commit message: Hooves & Harlots
Parts:
- removed J1, J2: Conn_01x03_Socket, Connector_Wire:SolderWire-0.5sqmm_1x03_P4.6mm_D0.9mm_OD2.1mm, symbol Connector:Conn_01x03_Socket
- removed J10, J12, J5, J6, J8, J9: 1985218, footprints:PTSA_15_4_35_Z, symbol PheonixContact:1985218
- added J1, J2: Conn_01x04_Socket, Connector_Wire:SolderWire-0.5sqmm_1x04_P4.6mm_D0.9mm_OD2.1mm, symbol Connector:Conn_01x04_Socket
- added J4, J5, J6, J7, J8, J9: 1861959, footprints:1861959, symbol PheonixContact:1861959
Connections:
- net +12V: now also J1.2 (Pin_2), J2.2 (Pin_2)
- net A0: now also J4.5 (3.1), J4.6 (3.2)
- net A1: now also J4.7 (4.1), J4.8 (4.2)
- net A10: now also J9.5 (3.1), J9.6 (3.2)
- net A11: now also J9.7 (4.1), J9.8 (4.2)
- net A2: now also J5.5 (3.1), J5.6 (3.2)
- net A3: now also J5.7 (4.1), J5.8 (4.2)
- net A4: now also J6.5 (3.1), J6.6 (3.2)
- net A5: now also J6.7 (4.1), J6.8 (4.2)
- net A6: now also J7.5 (3.1), J7.6 (3.2)
- net A7: now also J7.7 (4.1), J7.8 (4.2)
- net A8: now also J8.5 (3.1), J8.6 (3.2)
- net A9: now also J8.7 (4.1), J8.8 (4.2)
- net D7: now also J1.4 (Pin_4), J2.4 (Pin_4)
- net GND: now also J1.3 (Pin_3), J2.3 (Pin_3), J4.3 (2.1), J4.4 (2.2), J5.3 (2.1), J5.4 (2.2), J6.3 (2.1), J6.4 (2.2), J7.3 (2.1), J7.4 (2.2), J8.3 (2.1), J8.4 (2.2), J9.3 (2.1), J9.4 (2.2)
- net VIN: now also J4.1 (1.1), J4.2 (1.2), J5.1 (1.1), J5.2 (1.2), J6.1 (1.1), J6.2 (1.2), J7.1 (1.1), J7.2 (1.2), J8.1 (1.1), J8.2 (1.2), J9.1 (1.1), J9.2 (1.2)
- new net VDD: J1.1 (Pin_1), J2.1 (Pin_1)
Other:
- moved on the sheet: H1, H2, H3, J3, R13
