File: kicad/AoQin/AoQin.kicad_pcb (KiCad board)
At the start: 2 copper layers, 111.2 x 81 mm, 15 parts, among them J1 Conn_02x03_Odd_Even, J10 Conn_02x03_Odd_Even, J11 Conn_02x03_Odd_Even, J12 Conn_02x03_Odd_Even, J2 Conn_02x03_Odd_Even, J3 Screw_Terminal_01x12, J5 Conn_02x03_Odd_Even, J7 Screw_Terminal_01x12, J8 Screw_Terminal_01x03, J9 Screw_Terminal_01x03

Commit message: The Sword of Veracity
Parts:
- removed J10, J11, J12, J5: Conn_02x03_Odd_Even, Connector_PinHeader_2.54mm:PinHeader_2x03_P2.54mm_Vertical
- moved J2 45.2 mm to (129.0, 84.3), turned to 180 degrees
- moved J1 43.4 mm to (49.5, 31.7), turned to 0 degrees
- moved J7 9.01 mm to (117.0, 36.7)
- moved J3 8.70 mm to (61.2, 79.3)
Connections:
- net /GND renamed GND
- net /VIN renamed +12V
- J1 pad 2: Net-(J1-Pin_2) -> /VIN1
- J1 pad 4: Net-(J1-Pin_2) -> /VIN1
- J1 pad 6: Net-(J1-Pin_2) -> /VIN1
- J2 pad 2: Net-(J2-Pin_2) -> /VIN2
- J2 pad 4: Net-(J2-Pin_2) -> /VIN2
- J2 pad 6: Net-(J2-Pin_2) -> /VIN2
- J3 pad 1: /A7 -> /A6
- J3 pad 10: /A10 -> /A11
- J3 pad 12: Net-(J10-Pin_2) -> /VIN2
- J3 pad 2: /A6 -> /A7
- J3 pad 4: Net-(J11-Pin_2) -> /VIN2
- J3 pad 5: /A9 -> /A8
- J3 pad 6: /A8 -> /A9
- J3 pad 8: Net-(J12-Pin_2) -> /VIN2
- J3 pad 9: /A11 -> /A10
- J7 pad 1: /A1 -> /A0
- J7 pad 10: /A4 -> /A5
- J7 pad 12: Net-(J5-Pin_2) -> /VIN1
- J7 pad 2: /A0 -> /A1
- J7 pad 4: Net-(J1-Pin_2) -> /VIN1
- J7 pad 5: /A3 -> /A2
- J7 pad 6: /A2 -> /A3
- J7 pad 8: Net-(J2-Pin_2) -> /VIN1
- J7 pad 9: /A5 -> /A4
Routing:
- net /VIN2: track 0.00 -> 58.5 mm
- net /VIN1: track 0.00 -> 58.3 mm
- net /A11: track 67.5 -> 14.2 mm, vias 1 -> 0
- net /A10: track 57.8 -> 14.2 mm, vias 1 -> 0
- net +12V: track 162.5 -> 128.2 mm
- net GND: track 216.8 -> 183.8 mm, vias 0 -> 1
- net /A3: track 43.9 -> 14.2 mm, vias 1 -> 0
- net /A2: track 39.3 -> 14.2 mm, vias 1 -> 0
- net Net-(J1-Pin_2): track 20.8 -> 0.00 mm
- net Net-(J5-Pin_2): track 20.8 -> 0.00 mm
- net Net-(J2-Pin_2): track 20.8 -> 0.00 mm
- net Net-(J12-Pin_2): track 16.6 -> 0.00 mm
- net Net-(J10-Pin_2): track 16.6 -> 0.00 mm
- net Net-(J11-Pin_2): track 16.6 -> 0.00 mm
- net /5V: track 138.9 -> 128.7 mm
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
Commit message: Web of Desire
Parts:
- added J10: 1869237, footprints:SMKDSN_15_4_508, F.Cu at (101.8, 79.3)
- added J4: 1869237, footprints:SMKDSN_15_4_508, F.Cu at (76.7, 36.7)
- added J5: 1869237, footprints:SMKDSN_15_4_508, F.Cu at (102.2, 36.7)
- added J6: 1869237, footprints:SMKDSN_15_4_508, F.Cu at (52.2, 79.2)
- J3, J7: value Screw_Terminal_01x12 -> 1869237; footprint footprints:1869318 -> footprints:SMKDSN_15_4_508
- moved J7 58.4 mm to (76.8, 79.2), turned to 0 degrees
- moved J3 43.5 mm to (52.3, 36.7)
- moved J1 11.4 mm to (38.3, 29.2)
Connections:
- J3 pad 1: /A6 -> /A0
- J3 pad 2: /A7 -> /A6
- J3 pad 4: /VIN2 -> /VIN1
- J7 pad 1: /A0 -> /A4
- J7 pad 2: /A1 -> /A10
- J7 pad 4: /VIN1 -> /VIN2
Routing:
- net GND: track 183.8 -> 0.00 mm, vias 1 -> 0
- net /5V: track 128.7 -> 0.00 mm, vias 2 -> 0
- net +12V: track 128.2 -> 0.00 mm
- net /3V3: track 113.3 -> 0.00 mm, vias 1 -> 0
- net /D13: track 89.8 -> 0.00 mm, vias 1 -> 0
- net /VIN2: track 58.5 -> 0.00 mm
- net /VIN1: track 58.3 -> 0.00 mm
- net /A7: track 32.4 -> 0.00 mm
- net /A6: track 32.4 -> 0.00 mm
- net /A5: track 29.5 -> 0.00 mm, vias 1 -> 0
- net /A4: track 25.0 -> 0.00 mm, vias 1 -> 0
- net /A0: track 22.3 -> 0.00 mm
- net /A8: track 22.3 -> 0.00 mm
- net /A1: track 20.1 -> 0.00 mm
- net /A9: track 20.1 -> 0.00 mm
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
Commit message: Two Men and a Baby
Parts:
- moved J1 110.9 mm to (134.8, 83.9), turned to 180 degrees
- moved J2 102.3 mm to (41.1, 32.0), turned to 0 degrees
- moved J3 80.2 mm to (120.6, 78.7), turned to 180 degrees
- moved J5 53.0 mm to (69.8, 78.7), turned to 180 degrees
- moved J4 45.9 mm to (95.2, 78.7), turned to 180 degrees
- moved J10 42.2 mm to (106.1, 37.3)
- moved J7 42.2 mm to (80.7, 37.2)
- moved J6 42.1 mm to (55.3, 37.2)
- moved J9 2.66 mm to (122.8, 63.1)
- moved J8 2.24 mm to (52.2, 52.9)
- moved A1 0.20 mm to (111.8, 49.0)
Routing:
- net GND: track 0.00 -> 193.3 mm, vias 0 -> 1
- net /3V3: track 0.00 -> 134.9 mm, vias 0 -> 1
- net /5V: track 0.00 -> 132.3 mm, vias 0 -> 1
- net +12V: track 0.00 -> 131.6 mm
- net /VIN1: track 0.00 -> 86.6 mm
- net /VIN2: track 0.00 -> 86.2 mm
- net /D13: track 0.00 -> 78.6 mm, vias 0 -> 1
- net /A9: track 0.00 -> 64.8 mm, vias 0 -> 1
- net /A2: track 0.00 -> 51.4 mm, vias 0 -> 1
- net /A0: track 0.00 -> 48.8 mm, vias 0 -> 1
- net /A3: track 0.00 -> 44.3 mm
- net /A6: track 0.00 -> 40.0 mm, vias 0 -> 1
- net /A8: track 0.00 -> 38.6 mm
- net /A10: track 0.00 -> 35.7 mm
- net /A5: track 0.00 -> 30.3 mm, vias 0 -> 1
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
Commit message: Prodigal Sister
Connections:
- J10 pad 1: /A5 -> /A1
- J10 pad 2: /A11 -> /A0
- J3 pad 1: /A0 -> /A11
- J3 pad 2: /A6 -> /A10
- J4 pad 1: /A1 -> /A9
- J4 pad 2: /A7 -> /A8
- J5 pad 1: /A2 -> /A7
- J5 pad 2: /A8 -> /A6
- J6 pad 1: /A3 -> /A5
- J6 pad 2: /A9 -> /A4
- J7 pad 1: /A4 -> /A3
- J7 pad 2: /A10 -> /A2
Routing:
- net /A9: track 64.8 -> 15.2 mm, vias 1 -> 0
- net /A2: track 51.4 -> 17.0 mm, vias 1 -> 0
- net /A0: track 48.8 -> 17.6 mm, vias 1 -> 0
- net /A3: track 44.3 -> 18.8 mm
- net /A8: track 38.6 -> 16.3 mm
- net /A4: track 17.0 -> 35.4 mm
- net /A10: track 35.7 -> 18.9 mm
- net /A7: track 14.2 -> 28.5 mm
- net /A1: track 29.4 -> 16.6 mm
- net /3V3: track 134.9 -> 122.1 mm
- net /A6: track 40.0 -> 28.5 mm, vias 1 -> 0
- net /A11: track 29.7 -> 19.2 mm
- net /A5: track 30.3 -> 38.4 mm, vias 1 -> 0
- net /D13: track 78.6 -> 85.1 mm
- net /5V: track 132.3 -> 134.8 mm
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Other:
- board text removed: "BUS"
- board text removed: "SDI12"
- board text removed: "V+"
- board text removed: "V-"

Commit message: ...and Fancy Free
Parts:
- removed J2: Conn_02x03_Odd_Even, Connector_PinHeader_2.54mm:PinHeader_2x03_P2.54mm_Vertical
- added R1: 226k, Resistor_THT:R_Axial_DIN0207_L6.3mm_D2.5mm_P7.62mm_Horizontal, F.Cu at (132.3, 26.7)
- added S1: 2454982-4, footprints:24549824, F.Cu at (139.9, 44.4)
Connections:
- J1 pad 2: /VIN1 -> /VIN
- J1 pad 4: /VIN1 -> /VIN
- J1 pad 6: /VIN1 -> /VIN
- J3 pad 4: /VIN1 -> /VIN
Routing:
- net /3V3: track 122.1 -> 51.0 mm
- net /A6: track 28.5 -> 92.2 mm, vias 0 -> 1
- net /VIN1: track 87.0 -> 26.8 mm
- net /A8: track 16.3 -> 71.2 mm, vias 0 -> 1
- net /A10: track 18.9 -> 70.2 mm, vias 0 -> 1
- net /5V: track 134.8 -> 83.6 mm
- net /A4: track 35.4 -> 85.2 mm
- net /A2: track 17.0 -> 65.8 mm
- net GND: track 193.4 -> 235.1 mm, vias 0 -> 2
- net /VIN: track 0.00 -> 33.1 mm
- net /VIN2: track 86.0 -> 53.3 mm
- net /A0: track 17.6 -> 44.3 mm
- net +12V: track 130.2 -> 104.6 mm
- net Net-(R1-Pad2): track 0.00 -> 17.8 mm

Commit message: If I Had a Hammer
Parts:
- removed R1: 226k, Resistor_THT:R_Axial_DIN0207_L6.3mm_D2.5mm_P7.62mm_Horizontal
- removed S1: 2454982-4, footprints:24549824
- added RN1: 5.1k, Resistor_THT:R_Array_SIP7, F.Cu at (59.5, 65.6)
- added RN2: 5.1k, Resistor_THT:R_Array_SIP7, F.Cu at (115.5, 65.7)
- moved J1 3.34 mm to (132.8, 81.3)
- moved J8 1.90 mm to (50.3, 52.9)
- moved J9 1.90 mm to (124.7, 63.1)
Connections:
- J10 pad 4: /VIN2 -> /VIN
- J4 pad 4: /VIN1 -> /VIN
- J6 pad 4: /VIN2 -> /VIN
- J7 pad 4: /VIN2 -> /VIN
Routing:
- net /VIN: track 33.1 -> 156.1 mm
- net /A11: track 19.2 -> 74.1 mm
- net /VIN2: track 53.3 -> 0.00 mm
- net /A9: track 15.2 -> 60.3 mm
- net /A6: track 92.2 -> 47.4 mm, vias 1 -> 0
- net /A5: track 38.4 -> 71.7 mm, vias 0 -> 1
- net GND: track 235.1 -> 202.2 mm, vias 2 -> 0
- net /VIN1: track 26.8 -> 0.00 mm
- net /A7: track 28.5 -> 54.8 mm, vias 0 -> 1
- net /A3: track 18.8 -> 45.1 mm
- net /A2: track 65.8 -> 39.7 mm
- net /5V: track 83.6 -> 105.5 mm
- net /A4: track 85.2 -> 65.4 mm
- net /A1: track 16.7 -> 35.7 mm
- net Net-(R1-Pad2): track 17.8 -> 0.00 mm
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
Commit message: Judgment Day
Parts:
- removed RN1, RN2: 5.1k, Resistor_THT:R_Array_SIP7
- added J2: Conn_02x03_Odd_Even, Connector_PinHeader_2.54mm:PinHeader_2x03_P2.54mm_Vertical, F.Cu at (43.1, 37.4)
- added R1: 5.1k, Resistor_THT:R_Axial_DIN0204_L3.6mm_D1.6mm_P7.62mm_Horizontal, F.Cu at (85.2, 54.3)
- added R10: 5.1k, Resistor_THT:R_Axial_DIN0204_L3.6mm_D1.6mm_P7.62mm_Horizontal, F.Cu at (99.4, 61.9)
- added R11: 5.1k, Resistor_THT:R_Axial_DIN0204_L3.6mm_D1.6mm_P7.62mm_Horizontal, F.Cu at (102.5, 61.9)
- added R12: 5.1k, Resistor_THT:R_Axial_DIN0204_L3.6mm_D1.6mm_P7.62mm_Horizontal, F.Cu at (105.7, 61.9)
- added R2: 5.1k, Resistor_THT:R_Axial_DIN0204_L3.6mm_D1.6mm_P7.62mm_Horizontal, F.Cu at (82.0, 54.3)
- added R3: 5.1k, Resistor_THT:R_Axial_DIN0204_L3.6mm_D1.6mm_P7.62mm_Horizontal, F.Cu at (78.9, 54.3)
- added R4: 5.1k, Resistor_THT:R_Axial_DIN0204_L3.6mm_D1.6mm_P7.62mm_Horizontal, F.Cu at (75.7, 54.3)
- added R5: 5.1k, Resistor_THT:R_Axial_DIN0204_L3.6mm_D1.6mm_P7.62mm_Horizontal, F.Cu at (72.6, 54.3)
- added R6: 5.1k, Resistor_THT:R_Axial_DIN0204_L3.6mm_D1.6mm_P7.62mm_Horizontal, F.Cu at (69.4, 54.3)
- added R7: 5.1k, Resistor_THT:R_Axial_DIN0204_L3.6mm_D1.6mm_P7.62mm_Horizontal, F.Cu at (89.9, 61.9)
- added R8: 5.1k, Resistor_THT:R_Axial_DIN0204_L3.6mm_D1.6mm_P7.62mm_Horizontal, F.Cu at (93.1, 61.9)
- added R9: 5.1k, Resistor_THT:R_Axial_DIN0204_L3.6mm_D1.6mm_P7.62mm_Horizontal, F.Cu at (96.2, 61.9)
- moved J1 2.68 mm to (132.8, 78.6)
- moved J8 1.90 mm to (52.2, 52.9)
- moved J9 1.90 mm to (122.8, 63.1)
Connections:
- J1 pad 2: /VIN -> /VIN1
- J1 pad 4: /VIN -> /VIN1
- J1 pad 6: /VIN -> /VIN1
- J10 pad 4: /VIN -> /VIN2
- J3 pad 4: /VIN -> /VIN1
- J4 pad 4: /VIN -> /VIN1
- J6 pad 4: /VIN -> /VIN2
- J7 pad 4: /VIN -> /VIN2
Routing:
- net GND: track 202.2 -> 0.00 mm
- net /VIN: track 156.1 -> 0.00 mm
- net /5V: track 105.5 -> 0.00 mm, vias 1 -> 0
- net +12V: track 104.2 -> 0.00 mm
- net /D13: track 95.7 -> 0.00 mm, vias 1 -> 0
- net /A11: track 74.1 -> 0.00 mm
- net /A5: track 71.7 -> 0.00 mm, vias 1 -> 0
- net /A10: track 67.6 -> 0.00 mm
- net /A4: track 65.4 -> 0.00 mm
- net /A9: track 60.3 -> 0.00 mm
- net /A8: track 57.8 -> 0.00 mm
- net /A7: track 54.8 -> 0.00 mm, vias 1 -> 0
- net /3V3: track 47.9 -> 0.00 mm, vias 1 -> 0
- net /A6: track 47.4 -> 0.00 mm
- net /A3: track 45.1 -> 0.00 mm
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Other:
- board text added: "+12V"
- board text added: "-12V"
- board text added: "BUS"

Commit message: The Lost City
Parts:
- A1: footprint PCM_arduino-library:Arduino_Micro_Socket -> footprints:Arduino_Micro_Socket
Connections:
- A1 pad GND2: unconnected-(A1-GND-PadGND2) -> GND
Routing:
- net GND: track 0.00 -> 202.6 mm
- net /5V: track 0.00 -> 127.0 mm
- net +12V: track 0.00 -> 118.0 mm
- net /3V3: track 0.00 -> 112.6 mm, vias 0 -> 1
- net /VIN2: track 0.00 -> 102.4 mm
- net /D13: track 0.00 -> 85.1 mm, vias 0 -> 1
- net /VIN1: track 0.00 -> 84.0 mm
- net /A11: track 0.00 -> 52.0 mm
- net /A5: track 0.00 -> 47.7 mm, vias 0 -> 1
- net /A10: track 0.00 -> 46.7 mm
- net /A4: track 0.00 -> 45.4 mm, vias 0 -> 1
- net /A7: track 0.00 -> 42.0 mm, vias 0 -> 1
- net /A8: track 0.00 -> 40.0 mm
- net /A6: track 0.00 -> 38.5 mm
- net /A9: track 0.00 -> 38.3 mm
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Other:
- board text added: "GND"
- board text added: "VCC"
- board text removed: "+12V"
- board text removed: "-12V"
