File: kicad/AoQin/AoQin.kicad_pcb (KiCad board)
At the start: 2 copper layers, 111.2 x 81 mm, 17 parts, among them J1 Screw_Terminal_01x03, J10 1985218, J2 Screw_Terminal_01x03, J3 Conn_02x03_Odd_Even, J4 Conn_02x03_Odd_Even, J5 1985218, J6 1985218, J7 1985218, J8 1985218, J9 1985218

Commit message: Dreamworker
Parts:
- added J11: Conn_02x02_Odd_Even, Connector_PinHeader_2.54mm:PinHeader_2x02_P2.54mm_Vertical, F.Cu at (120.7, 43.7)
- J1, J2: value Screw_Terminal_01x03 -> Screw_Terminal_01x04; footprint TerminalBlock_Phoenix:TerminalBlock_Phoenix_MKDS-1,5-3-5.08_1x03_P5.08mm_Horizontal -> TerminalBlock_Phoenix:TerminalBlock_Phoenix_MKDS-1,5-4-5.08_1x04_P5.08mm_Horizontal
- moved J2 72.5 mm to (123.6, 65.6), turned to 90 degrees
- moved J1 71.6 mm to (52.3, 50.4), turned to -90 degrees
- moved J3 1.67 mm to (123.1, 81.6)
Connections:
- A1 pad VIN: +12V -> /VCC
- J1 pad 1: +12V -> /+12VCC
- J1 pad 2: GND -> +12V
- J1 pad 3: /D13 -> GND
- J2 pad 1: +12V -> /+12VCC
- J2 pad 2: GND -> +12V
- J2 pad 3: /D13 -> GND
Routing:
- net /+12VCC: track 0.00 -> 95.6 mm
- net /VCC: track 0.00 -> 67.6 mm, vias 0 -> 1
- net +12V: track 117.7 -> 138.7 mm
- net /D13: track 86.3 -> 77.8 mm, vias 1 -> 0
- net /3V3: track 89.5 -> 97.7 mm, vias 0 -> 1
- net /A2: track 18.3 -> 13.1 mm
- net /D3: track 33.8 -> 38.1 mm, vias 0 -> 1
- net /D2: track 35.3 -> 39.4 mm
- net /5V: track 102.0 -> 105.4 mm
- net /VIN1: track 67.0 -> 64.8 mm
- net /D7: track 44.2 -> 42.0 mm
- net /D5: track 39.5 -> 41.3 mm
- net GND: track 209.8 -> 211.3 mm, vias 0 -> 1
- net /A6: track 19.5 -> 20.3 mm, vias 0 -> 1
- net /A7: track 23.1 -> 23.7 mm
Other:
- board text added: "PERM"
- board text added: "SWCH"
- board text removed: "BUS"
- board text removed: "GND"
- board text removed: "VCC"

Commit message: Stranger and Stranger
Connections:
- A1 pad D4: /A6 -> /D4
- A1 pad D6: /A7 -> /D6
- J10 pad 1: /VIN2 -> GND
- J10 pad 2: GND -> /D2
- J10 pad 3: /A4 -> GND
- J10 pad 4: /A5 -> /D3
- J5 pad 3: /A6 -> /A4
- J5 pad 4: /A7 -> /A5
- S2 pad 3: /D2 -> /D4
- S2 pad 4: /D3 -> /D5
- S2 pad 5: /D5 -> /D6
Routing:
- net /D4: track 0.00 -> 42.9 mm, vias 0 -> 1
- net /D6: track 0.00 -> 40.6 mm
- net /A7: track 23.7 -> 0.00 mm
- net /A6: track 20.3 -> 0.00 mm, vias 1 -> 0
- net /VCC: track 67.6 -> 55.2 mm, vias 1 -> 0
- net /A4: track 27.0 -> 38.6 mm, vias 0 -> 1
- net /D3: track 38.1 -> 48.2 mm
- net /D2: track 39.4 -> 33.0 mm, vias 1 -> 0
- net /A5: track 36.3 -> 41.0 mm
- net /3V3: track 97.7 -> 93.5 mm
- net GND: track 211.3 -> 207.5 mm, vias 1 -> 0
- net /A3: track 20.0 -> 17.0 mm
- net /D13: track 77.8 -> 80.6 mm, vias 0 -> 1
- net /A2: track 13.1 -> 15.3 mm
- net +12V: track 138.7 -> 136.9 mm
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Other:
- board text added: "3 / INT (x2)"
- board text removed: "3"

Commit message: A Necessary Evil
Parts:
- added J12: 1985218, footprints:PTSA_15_4_35_Z, F.Cu at (102.5, 73.3)
- J10, J7: value 1985218 -> 1985195; footprint footprints:PTSA_15_4_35_Z -> footprints:1985195
- moved J7 46.7 mm to (67.2, 42.7), turned to 180 degrees
- moved J3 26.1 mm to (138.6, 60.6)
- moved J11 15.6 mm to (136.3, 44.0)
- moved J4 10.6 mm to (43.1, 33.4)
- moved J10 5.70 mm to (79.2, 42.7)
- moved J8 1.70 mm to (113.2, 42.7)
- moved J9 1.70 mm to (94.2, 42.7)
Connections:
- A1 pad D11: unconnected-(A1-PadD11) -> /D11
- A1 pad D2: /D2 -> /SDA
- A1 pad D3: /D3 -> /SCL
- A1 pad D8: /A8 -> /D8
- A1 pad D9: /A9 -> /D9
- J1 pad 4: /D13 -> /D9
- J10 pad 1: GND -> /D1
- J10 pad 2: /D2 -> GND
- J6 pad 3: /A8 -> /A6
- J6 pad 4: /A9 -> /A7
- J7 pad 1: /VIN1 -> /D0
- R13 pad 1: /D13 -> /D9
- S2 pad 1: /D0 -> unconnected-(S2-COM_1-Pad1)
- S2 pad 2: /D1 -> unconnected-(S2-COM_2-Pad2)
- S2 pad 3: /D4 -> unconnected-(S2-COM_3-Pad3)
- S2 pad 4: /D5 -> unconnected-(S2-COM_4-Pad4)
- S2 pad 5: /D6 -> unconnected-(S2-COM_5-Pad5)
- S2 pad 6: /D7 -> unconnected-(S2-COM_6-Pad6)
Routing:
- net GND: track 207.5 -> 0.00 mm
- net +12V: track 136.9 -> 0.00 mm
- net /5V: track 105.8 -> 0.00 mm, vias 2 -> 0
- net /+12VCC: track 94.5 -> 0.00 mm, vias 1 -> 0
- net /3V3: track 93.5 -> 0.00 mm, vias 1 -> 0
- net /D13: track 80.6 -> 0.00 mm, vias 1 -> 0
- net /VIN1: track 64.7 -> 0.00 mm
- net /VIN2: track 63.6 -> 0.00 mm
- net /VCC: track 55.2 -> 0.00 mm
- net /D3: track 48.2 -> 0.00 mm, vias 1 -> 0
- net /D4: track 42.9 -> 0.00 mm, vias 1 -> 0
- net /D5: track 42.3 -> 0.00 mm
- net /D7: track 42.1 -> 0.00 mm, vias 1 -> 0
- net /A5: track 41.0 -> 0.00 mm, vias 1 -> 0
- net /D6: track 40.6 -> 0.00 mm
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Other:
- board text added: "3"
- board text removed: "3 / INT (x2)"
- board text removed: "6"

Commit message: Gabrielle's Hope
Parts:
- removed J11: Conn_02x02_Odd_Even, Connector_PinHeader_2.54mm:PinHeader_2x02_P2.54mm_Vertical
- removed J7: 1985195, footprints:1985195
- J1, J2: value Screw_Terminal_01x04 -> Conn_01x03_Socket; footprint TerminalBlock_Phoenix:TerminalBlock_Phoenix_MKDS-1,5-4-5.08_1x04_P5.08mm_Horizontal -> Connector_Wire:SolderWire-0.5sqmm_1x03_P4.6mm_D0.9mm_OD2.1mm
- J10: value 1985195 -> 1985218; footprint footprints:1985195 -> footprints:PTSA_15_4_35_Z
- moved J2 67.8 mm to (56.9, 53.4), turned to -90 degrees
- moved J1 67.0 mm to (118.2, 62.6), turned to 90 degrees
- moved J3 24.1 mm to (124.8, 80.3)
- moved J4 8.41 mm to (51.1, 35.7)
- moved J10 5.70 mm to (73.5, 42.7)
- moved J8 1.70 mm to (111.5, 42.7)
- moved J9 1.70 mm to (92.5, 42.7)
Connections:
- A1 pad D13: /D13 -> unconnected-(A1-PadD13)
- A1 pad D2: /SDA -> /D2
- A1 pad D3: /SCL -> /D3
- A1 pad D4: /D4 -> /A6
- A1 pad D6: /D6 -> /A7
- A1 pad D8: /D8 -> /A8
- A1 pad D9: /D9 -> /A9
- J1 pad 1: /+12VCC -> +12V
- J1 pad 2: +12V -> GND
- J1 pad 3: GND -> /D11
- J10 pad 1: /D1 -> /VIN2
- J2 pad 1: /+12VCC -> +12V
- J2 pad 2: +12V -> GND
- J2 pad 3: GND -> /D11
- J5 pad 3: /A4 -> /A6
- J5 pad 4: /A5 -> /A7
- J6 pad 3: /A6 -> /A8
- J6 pad 4: /A7 -> /A9
- R13 pad 1: /D9 -> /D11
- S2 pad 1: unconnected-(S2-COM_1-Pad1) -> /D7
- S2 pad 2: unconnected-(S2-COM_2-Pad2) -> /D5
- S2 pad 3: unconnected-(S2-COM_3-Pad3) -> /D3
- S2 pad 4: unconnected-(S2-COM_4-Pad4) -> /D2
- S2 pad 5: unconnected-(S2-COM_5-Pad5) -> /D1
- S2 pad 6: unconnected-(S2-COM_6-Pad6) -> /D0
Routing:
- net GND: track 0.00 -> 203.9 mm, vias 0 -> 1
- net /5V: track 0.00 -> 109.3 mm, vias 0 -> 2
- net +12V: track 0.00 -> 108.0 mm
- net /3V3: track 0.00 -> 101.5 mm, vias 0 -> 1
- net /D11: track 0.00 -> 74.8 mm
- net /VIN2: track 0.00 -> 66.1 mm
- net /VIN1: track 0.00 -> 65.7 mm
- net /D7: track 0.00 -> 51.8 mm, vias 0 -> 1
- net /D5: track 0.00 -> 49.7 mm, vias 0 -> 1
- net /D3: track 0.00 -> 41.1 mm, vias 0 -> 1
- net /A5: track 0.00 -> 35.3 mm, vias 0 -> 1
- net /D2: track 0.00 -> 31.8 mm
- net /A7: track 0.00 -> 27.7 mm
- net /A4: track 0.00 -> 27.0 mm
- net /D1: track 0.00 -> 23.6 mm
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Other:
- board text removed: "PERM"
- board text removed: "SWCH"

Commit message: The King of Assassins
Parts:
- removed H1, H2, H3, H4: MountingHole_2.5mm, MountingHole:MountingHole_2.5mm
- added M1: MountingHole_3.5mm, MountingHole:MountingHole_3.5mm, F.Cu at (35.5, 95.5)
- added M2: MountingHole_3.5mm, MountingHole:MountingHole_3.5mm, F.Cu at (140.5, 95.5)
- added M3: MountingHole_3.5mm, MountingHole:MountingHole_3.5mm, F.Cu at (140.5, 20.5)
- added M4: MountingHole_3.5mm, MountingHole:MountingHole_3.5mm, F.Cu at (35.5, 20.5)
Connections:
- J1 pad 3: /D11 -> /D7
- J2 pad 3: /D11 -> /D7
- R13 pad 1: /D11 -> /D7
- S2 pad 1: /D7 -> /D11
Routing:
- net /D7: track 51.8 -> 78.0 mm
- net /D11: track 74.8 -> 63.4 mm, vias 0 -> 1
- net /A2: track 22.1 -> 13.1 mm
- net /3V3: track 101.5 -> 93.5 mm, vias 1 -> 0
- net GND: track 203.9 -> 209.1 mm, vias 1 -> 0
- net /D3: track 41.1 -> 36.3 mm
- net /A10: track 10.5 -> 14.1 mm
- net /A5: track 35.3 -> 32.0 mm
- net /5V: track 109.3 -> 111.3 mm
- net /A3: track 19.0 -> 17.1 mm
- net /A4: track 27.0 -> 28.5 mm
- net /D5: track 49.7 -> 50.8 mm
- net /A7: track 27.7 -> 27.3 mm, vias 0 -> 1
Other:
- board size 111.2 x 81 mm -> 113.5 x 83 mm
