File: kicad/cable-connector/cable-connector.kicad_sch (KiCad schematic)
At the start: 0 parts

Commit message: Dreamworker
Parts:
- added J1, J10, J2, J3, J4, J5, J6, J7, J8, J9: Conn_01x04_Pin, footprints:SDI_Connector, symbol Connector:Conn_01x04_Pin

Commit message: Cradle of Hope
Parts:
- added J11: Conn_01x04_Pin, footprints:GROVE-HW4-2.0, symbol Connector:Conn_01x04_Pin
Connections:
- net BLUE: now reaches J3.1 (Pin_1)
- net BLUE: now also J1.1 (Pin_1), J10.1 (Pin_1), J2.1 (Pin_1), J4.1 (Pin_1), J5.1 (Pin_1), J6.1 (Pin_1), J7.1 (Pin_1), J8.1 (Pin_1), J9.1 (Pin_1), J11.1 (Pin_1)
- net WHITE: now reaches J3.2 (Pin_2)
- net WHITE: now also J1.2 (Pin_2), J10.2 (Pin_2), J2.2 (Pin_2), J4.2 (Pin_2), J5.2 (Pin_2), J6.2 (Pin_2), J7.2 (Pin_2), J8.2 (Pin_2), J9.2 (Pin_2), J11.2 (Pin_2)
- net BROWN: now reaches J3.3 (Pin_3)
- net BROWN: now also J1.3 (Pin_3), J10.3 (Pin_3), J2.3 (Pin_3), J4.3 (Pin_3), J5.3 (Pin_3), J6.3 (Pin_3), J7.3 (Pin_3), J8.3 (Pin_3), J9.3 (Pin_3), J11.3 (Pin_3)
- net BLACK: now reaches J3.4 (Pin_4)
- net BLACK: now also J1.4 (Pin_4), J10.4 (Pin_4), J2.4 (Pin_4), J4.4 (Pin_4), J5.4 (Pin_4), J6.4 (Pin_4), J7.4 (Pin_4), J8.4 (Pin_4), J9.4 (Pin_4), J11.4 (Pin_4)

Commit message: War Wounds
Connections:
- net BLUE: now also J1.2 (Pin_2), J10.2 (Pin_2), J11.2 (Pin_2), J2.2 (Pin_2), J3.2 (Pin_2), J4.2 (Pin_2), J5.2 (Pin_2), J6.2 (Pin_2), J7.2 (Pin_2), J8.2 (Pin_2), J9.2 (Pin_2); no longer J1.1 (Pin_1), J10.1 (Pin_1), J11.1 (Pin_1), J2.1 (Pin_1), J3.1 (Pin_1), J4.1 (Pin_1), J5.1 (Pin_1), J6.1 (Pin_1), J7.1 (Pin_1), J8.1 (Pin_1), J9.1 (Pin_1)
- net WHITE: now also J1.1 (Pin_1), J10.1 (Pin_1), J11.1 (Pin_1), J2.1 (Pin_1), J3.1 (Pin_1), J4.1 (Pin_1), J5.1 (Pin_1), J6.1 (Pin_1), J7.1 (Pin_1), J8.1 (Pin_1), J9.1 (Pin_1); no longer J1.2 (Pin_2), J10.2 (Pin_2), J11.2 (Pin_2), J2.2 (Pin_2), J3.2 (Pin_2), J4.2 (Pin_2), J5.2 (Pin_2), J6.2 (Pin_2), J7.2 (Pin_2), J8.2 (Pin_2), J9.2 (Pin_2)

Commit message: The Academy
Parts:
- removed J10, J9: Conn_01x04_Pin, footprints:SDI_Connector, symbol Connector:Conn_01x04_Pin
- removed J11: Conn_01x04_Pin, footprints:GROVE-HW4-2.0, symbol Connector:Conn_01x04_Pin
- J8: footprint footprints:SDI_Connector -> footprints:GROVE-HW4-2.0
Connections:
- net BLACK renamed LINE
- net BLUE renamed +12V
- net BROWN renamed GND
- net WHITE renamed VBUS
Other:
- moved on the sheet: J2, J3, J4, J5, J6, J7, J8
