File: kicad/Ryujin_v2/Ryujin_v2.kicad_sch (KiCad schematic)
At the start: 32 parts, among them J1 Screw_Terminal_01x02, J10 Conn_01x04_Pin, J11 Conn_01x04_Pin, J12 Conn_01x04_Pin, J2 Conn_02x02_Odd_Even, J3 Conn_01x14_Socket, J4 Conn_01x14_Socket, J6 Conn_01x04_Pin, J7 Conn_01x04_Pin, J8 Conn_01x04_Pin, J9 Conn_01x04_Pin, Q1 IRLML5203, Q2 IRLML6244, U1 74LVC1G17, U2 74AHCT1G14, U3 TMUX1119DBVR, U4 SHTC3, U5 W25Q32JVSS, U7 R-78E5.0-1.0

Commit message: Once Upon a Future King
Parts:
- added D2, D3: D, Diode_SMD:D_0201_0603Metric, symbol Device:D
- added J5: Screw_Terminal_01x02, TerminalBlock_Phoenix:TerminalBlock_Phoenix_MKDS-1,5-2-5.08_1x02_P5.08mm_Horizontal, symbol Connector:Screw_Terminal_01x02
- added Q3: BC547, Package_TO_SOT_THT:TO-92_Inline, symbol Transistor_BJT:BC547
- added R11: 240, Resistor_SMD:R_0603_1608Metric, symbol Device:R
- added R12: 10k, Resistor_SMD:R_0603_1608Metric, symbol Device:R
- added R13: 0.2, Resistor_SMD:R_0603_1608Metric, symbol Device:R
- added U6: LM317_SOT-223, Package_TO_SOT_SMD:SOT-223-3_TabPin2, symbol Regulator_Linear:LM317_SOT-223
Connections:
- net +12V: now also D3.1 (K)
- net GND: now also Q3.2 (B), R12.2, R13.1
- new net: D3.2 (A), R11.1, U6.2 (VO)
- new net: Q3.1 (C), R11.2, R12.1, U6.1 (ADJ)
- new net: D2.1 (K), U6.3 (VI)
- new net: D2.2 (A), J5.2 (Pin_2)
- new net: J5.1 (Pin_1), Q3.3 (E), R13.2
Other:
- moved on the sheet: J2

Commit message: Ten Little Warlords
Parts:
- removed D2, D3: D, Diode_SMD:D_0201_0603Metric, symbol Device:D
- removed J5: Screw_Terminal_01x02, TerminalBlock_Phoenix:TerminalBlock_Phoenix_MKDS-1,5-2-5.08_1x02_P5.08mm_Horizontal, symbol Connector:Screw_Terminal_01x02
- removed Q3: BC547, Package_TO_SOT_THT:TO-92_Inline, symbol Transistor_BJT:BC547
- removed R11: 240, Resistor_SMD:R_0603_1608Metric, symbol Device:R
- removed R12: 10k, Resistor_SMD:R_0603_1608Metric, symbol Device:R
- removed R13: 0.2, Resistor_SMD:R_0603_1608Metric, symbol Device:R
- removed U6: LM317_SOT-223, Package_TO_SOT_SMD:SOT-223-3_TabPin2, symbol Regulator_Linear:LM317_SOT-223
- added U6: BQ24650, Package_DFN_QFN:Texas_RVA_VQFN-16-1EP_3.5x3.5mm_P0.5mm_EP2.14x2.14mm_ThermalVias, symbol Battery_Management:BQ24650
Connections:
- new net: U6.11 (GND), U6.17 (GND)
