File: kicad/Ryujin_v2/Ryujin_v2.kicad_pcb (KiCad board)
At the start: 2 copper layers, 172 x 71 mm, 33 parts, among them J1 Screw_Terminal_01x02, J10 Conn_01x04_Pin, J11 Conn_01x04_Pin, J12 Conn_01x04_Pin, J2 Conn_02x02_Odd_Even, J3 Conn_01x14_Socket, J4 Conn_01x14_Socket, J6 Conn_01x04_Pin, J7 Conn_01x04_Pin, J8 Conn_01x04_Pin, J9 Conn_01x04_Pin, Q1 IRLML5203, Q2 IRLML6244, U1 74LVC1G17, U2 74AHCT1G14, U3 TMUX1119DBVR, U4 SHTC3, U5 W25Q32JVSS, U7 R-78E5.0-1.0

Commit message: Once Upon a Future King
Parts:
- added D2: D, Diode_SMD:D_0201_0603Metric, F.Cu at (166.3, 56.0)
- added D3: D, Diode_SMD:D_0201_0603Metric, F.Cu at (166.3, 57.8)
- added J5: Screw_Terminal_01x02, TerminalBlock_Phoenix:TerminalBlock_Phoenix_MKDS-1,5-2-5.08_1x02_P5.08mm_Horizontal, F.Cu at (156.2, 53.9)
- added Q3: BC547, Package_TO_SOT_THT:TO-92_Inline, F.Cu at (164.5, 63.0)
- added R11: 240, Resistor_SMD:R_0603_1608Metric, F.Cu at (166.8, 48.9)
- added R12: 10k, Resistor_SMD:R_0603_1608Metric, F.Cu at (166.8, 51.4)
- added R13: 0.2, Resistor_SMD:R_0603_1608Metric, F.Cu at (166.8, 53.9)
- added U6: LM317_SOT-223, Package_TO_SOT_SMD:SOT-223-3_TabPin2, F.Cu at (157.6, 63.9)

Commit message: Ten Little Warlords
Parts:
- removed D2, D3: D, Diode_SMD:D_0201_0603Metric
- removed J5: Screw_Terminal_01x02, TerminalBlock_Phoenix:TerminalBlock_Phoenix_MKDS-1,5-2-5.08_1x02_P5.08mm_Horizontal
- removed Q3: BC547, Package_TO_SOT_THT:TO-92_Inline
- removed R11: 240, Resistor_SMD:R_0603_1608Metric
- removed R12: 10k, Resistor_SMD:R_0603_1608Metric
- removed R13: 0.2, Resistor_SMD:R_0603_1608Metric
- removed U6: LM317_SOT-223, Package_TO_SOT_SMD:SOT-223-3_TabPin2
- moved G2 92.2 mm to (105.3, 79.5)
- moved G1 71.5 mm to (128.4, 82.5)
- moved U5 49.2 mm to (23.1, 55.6), turned to -90 degrees
- moved U7 34.0 mm to (103.1, 58.1)
- moved C1 13.8 mm to (91.4, 68.7)
- moved C6 8.67 mm to (62.1, 57.0)
- moved C4 8.67 mm to (61.7, 68.8)
- moved R6 8.67 mm to (67.9, 53.6)
- moved U1 8.67 mm to (61.7, 60.5)
- moved U2 8.67 mm to (61.5, 65.1)
- moved U3 8.67 mm to (59.5, 72.3)
- moved U4 8.67 mm to (61.9, 54.0)
- moved R7 8.67 mm to (65.4, 53.6)
Routing:
- net GND: track 0.00 -> 335.0 mm, vias 0 -> 2
- net +12V: track 0.00 -> 223.9 mm
- net LINE: track 0.00 -> 166.0 mm, vias 0 -> 2
- net /D5: track 0.00 -> 160.7 mm, vias 0 -> 1
- net VBUS: track 0.00 -> 148.3 mm
- net +5V: track 0.00 -> 99.3 mm, vias 0 -> 3
- net +3.3V: track 0.00 -> 72.5 mm, vias 0 -> 2
- net /D0: track 0.00 -> 47.6 mm
- net /D7: track 0.00 -> 44.2 mm, vias 0 -> 1
- net /D1: track 0.00 -> 40.3 mm, vias 0 -> 1
- net /CIPO: track 0.00 -> 36.7 mm, vias 0 -> 1
- net /RX: track 0.00 -> 36.5 mm, vias 0 -> 1
- net /COPI: track 0.00 -> 34.7 mm
- net /SCK: track 0.00 -> 32.5 mm
- net /TX: track 0.00 -> 31.9 mm
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
Commit message: A Solstice Carol
Parts:
- removed J2: Conn_02x02_Odd_Even, Connector_PinHeader_2.54mm:PinHeader_2x02_P2.54mm_Vertical
- moved R10 82.6 mm to (161.0, 64.4), turned to 90 degrees
- moved U5 79.9 mm to (102.3, 66.5), turned to 0 degrees
- moved C2 79.8 mm to (159.9, 48.4), turned to 180 degrees
- moved R9 77.5 mm to (158.4, 64.4), turned to -90 degrees
- moved R8 73.7 mm to (156.6, 59.8), turned to 90 degrees
- moved Q2 70.6 mm to (155.0, 64.2), turned to 180 degrees
- moved Q1 66.8 mm to (153.1, 59.8), turned to 180 degrees
- moved C1 66.6 mm to (154.9, 48.4), turned to 0 degrees
- moved U7 54.0 mm to (155.1, 43.3), turned to 0 degrees
- moved C4 21.8 mm to (82.9, 63.6), turned to -90 degrees
- moved U3 20.1 mm to (79.2, 68.1), turned to 0 degrees
- moved U4 18.2 mm to (79.2, 59.6)
- moved U2 17.7 mm to (79.2, 63.6), turned to 0 degrees
- moved R6 15.9 mm to (82.6, 59.6)
- moved C6 13.4 mm to (75.3, 59.1)
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Routing:
- net GND: track 335.0 -> 0.00 mm, vias 2 -> 0
- net +12V: track 223.9 -> 0.00 mm
- net LINE: track 166.0 -> 0.00 mm, vias 2 -> 0
- net /D5: track 160.7 -> 0.00 mm, vias 1 -> 0
- net VBUS: track 148.3 -> 0.00 mm
- net +5V: track 99.3 -> 0.00 mm, vias 3 -> 0
- net +3.3V: track 72.5 -> 0.00 mm, vias 2 -> 0
- net /D0: track 47.6 -> 0.00 mm
- net /D7: track 44.2 -> 0.00 mm, vias 1 -> 0
- net /D1: track 40.3 -> 0.00 mm, vias 1 -> 0
- net /CIPO: track 36.7 -> 0.00 mm, vias 1 -> 0
- net /RX: track 36.5 -> 0.00 mm, vias 1 -> 0
- net /COPI: track 34.7 -> 0.00 mm
- net /SCK: track 32.5 -> 0.00 mm
- net /TX: track 31.9 -> 0.00 mm
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Other:
- board text removed: "-"
- board text removed: "<"
- board text removed: "∅"
