File: kicad/SonTinh/SonTinh.kicad_pcb (KiCad board)
At the start: 2 copper layers, 111.2 x 81 mm, 12 parts, among them J1 Conn_01x04_Socket, J10 1985195, J11 Conn_01x03_Socket, J13 Conn_01x03_Socket, J2 Conn_01x04_Socket, J7 1985195

Commit message: The Debt, Part 1
Parts:
- removed J1, J2: Conn_01x04_Socket, Connector_Molex:Molex_KK-254_AE-6410-04A_1x04_P2.54mm_Vertical
- added J12: 1985195, footprints:1985195, F.Cu at (71.4, 31.9)
- added J3: Conn_02x03_Odd_Even, Connector_PinHeader_2.54mm:PinHeader_2x03_P2.54mm_Vertical, F.Cu at (124.8, 80.3)
- added J4: Conn_02x03_Odd_Even, Connector_PinHeader_2.54mm:PinHeader_2x03_P2.54mm_Vertical, F.Cu at (116.6, 33.5)
- added J4: 1985218, footprints:PTSA_15_4_35_Z, F.Cu at (39.8, 47.0)
- added J5: 1985218, footprints:PTSA_15_4_35_Z, F.Cu at (39.8, 62.1)
- added J8: 1985195, footprints:1985195, F.Cu at (48.2, 31.9)
- moved J7 57.4 mm to (36.6, 31.9)
- moved J10 45.8 mm to (59.8, 31.9)
- moved J13 2.17 mm to (118.2, 62.6)
- moved J11 2.08 mm to (56.9, 53.4)
Other:
- board text added: "12V"
- board text added: "3V3"
- board text added: "5V"

Commit message: The Debt, Part 2
Parts:
- removed J3: Conn_02x03_Odd_Even, Connector_PinHeader_2.54mm:PinHeader_2x03_P2.54mm_Vertical
- removed the J4 at (116.6, 33.5)
- moved J7 59.5 mm to (95.3, 41.0), turned to 180 degrees
- moved J10 57.8 mm to (99.1, 74.3)
- moved J8 56.5 mm to (85.6, 74.3)
- moved J4 40.4 mm to (79.8, 41.0), turned to 180 degrees
- moved J12 37.1 mm to (107.3, 41.0), turned to 180 degrees
- moved J5 32.3 mm to (69.8, 74.0)
Other:
- board text removed: "12V"
- board text removed: "3V3"
- board text removed: "5V"

Commit message: The Quill Is Mightier…
Parts:
- removed H1, H2, H3, H4: MountingHole_2.5mm, MountingHole:MountingHole_2.5mm
- added M1: MountingHole_3.5mm, MountingHole:MountingHole_3.5mm, F.Cu at (35.5, 95.5)
- added M2: MountingHole_3.5mm, MountingHole:MountingHole_3.5mm, F.Cu at (140.5, 95.5)
- added M3: MountingHole_3.5mm, MountingHole:MountingHole_3.5mm, F.Cu at (140.5, 20.5)
- added M4: MountingHole_3.5mm, MountingHole:MountingHole_3.5mm, F.Cu at (35.5, 20.5)
- moved J5 40.2 mm to (91.3, 40.0), turned to 180 degrees
- moved J12 34.8 mm to (72.6, 40.0)
- moved J10 34.0 mm to (65.1, 72.5)
- moved J4 31.8 mm to (83.8, 72.5), turned to 0 degrees
- moved J8 19.1 mm to (104.6, 72.5)
- moved J7 15.3 mm to (110.6, 40.8)
- moved J11 1.41 mm to (55.9, 52.4)
- moved J13 1.41 mm to (117.2, 61.6)
Connections:
- A1 pad A2: /A2 -> unconnected-(A1-PadA2)
- A1 pad A3: /A3 -> unconnected-(A1-PadA3)
- A1 pad A4: /A4 -> unconnected-(A1-PadA4)
- A1 pad A5: /A5 -> unconnected-(A1-PadA5)
- A1 pad D10: /A10 -> unconnected-(A1-PadD10)
- A1 pad D11: /D11 -> unconnected-(A1-PadD11)
- A1 pad D12: /A11 -> unconnected-(A1-PadD12)
- A1 pad D13: /D13 -> unconnected-(A1-PadD13)
- A1 pad D9: /D9 -> unconnected-(A1-PadD9)
- J11 pad 3: /D11 -> /D7
- J13 pad 3: /D11 -> /D7
- R13 pad 1: /D11 -> /D7
Routing:
- net GND: track 0.00 -> 171.0 mm, vias 0 -> 4
- net /D7: track 0.00 -> 74.7 mm, vias 0 -> 1
- net +12V: track 0.00 -> 68.2 mm
- net /D0: track 0.00 -> 63.1 mm, vias 0 -> 1
- net /5V: track 0.00 -> 48.9 mm
- net /A0: track 0.00 -> 41.1 mm
- net /SDA: track 0.00 -> 40.9 mm, vias 0 -> 1
- net /SCL: track 0.00 -> 35.7 mm
- net /A1: track 0.00 -> 33.3 mm
- net /D1: track 0.00 -> 12.1 mm
Other:
- board size 111.2 x 81 mm -> 113.5 x 83 mm

Commit message: The Bitter Suite
Parts:
- removed J10, J12, J7, J8: 1985195, footprints:1985195
- removed J13: Conn_01x03_Socket, Connector_Wire:SolderWire-0.25sqmm_1x03_P4.5mm_D0.65mm_OD2mm
- removed J4, J5: 1985218, footprints:PTSA_15_4_35_Z
- removed M1, M2, M3, M4: MountingHole_3.5mm, MountingHole:MountingHole_3.5mm
- added J1: Screw_Terminal_01x02, TerminalBlock_Phoenix:TerminalBlock_Phoenix_MPT-0,5-2-2.54_1x02_P2.54mm_Horizontal, F.Cu at (109.8, 48.5)
- added J2: Screw_Terminal_01x02, TerminalBlock_Phoenix:TerminalBlock_Phoenix_MPT-0,5-2-2.54_1x02_P2.54mm_Horizontal, F.Cu at (111.6, 24.6)
- added J3: Screw_Terminal_01x02, TerminalBlock_Phoenix:TerminalBlock_Phoenix_MPT-0,5-2-2.54_1x02_P2.54mm_Horizontal, F.Cu at (123.3, 36.5)
- added U1: BME680, Package_LGA:Bosch_LGA-8_3x3mm_P0.8mm_ClockwisePinNumbering, F.Cu at (149.0, 34.3)
- moved R13 70.3 mm to (43.7, 38.3), turned to 90 degrees
- moved J11 29.2 mm to (38.3, 29.0)
- moved A1 26.8 mm to (97.3, 26.4)
Connections:
- A1 pad MISO: unconnected-(A1-SPI_MISO-PadMISO) -> Net-(A1-SPI_MISO)
- A1 pad MOSI: unconnected-(A1-SPI_MOSI-PadMOSI) -> Net-(A1-SPI_MOSI)
- A1 pad SCK: unconnected-(A1-SPI_SCK-PadSCK) -> Net-(A1-SPI_SCK)
- A1 pad SS: unconnected-(A1-SPI_CS-PadSS) -> Net-(A1-SPI_CS)
Routing:
- net GND: track 171.0 -> 0.00 mm, vias 4 -> 0
- net /D7: track 74.7 -> 0.00 mm, vias 1 -> 0
- net +12V: track 68.2 -> 0.00 mm
- net /D0: track 63.1 -> 0.00 mm, vias 1 -> 0
- net /5V: track 48.9 -> 0.00 mm
- net /A0: track 41.1 -> 0.00 mm
- net /SDA: track 40.9 -> 0.00 mm, vias 1 -> 0
- net /SCL: track 35.7 -> 0.00 mm
- net /A1: track 33.3 -> 0.00 mm
- net /D1: track 12.1 -> 0.00 mm
Other:
- board size 113.5 x 83 mm -> 129 x 39 mm

Commit message: The Path Not Taken
Parts:
- moved A1 26.7 mm to (106.8, 51.4)
- moved J11 26.7 mm to (47.8, 54.0)
- moved J2 26.7 mm to (121.1, 49.6)
- moved J3 26.7 mm to (132.8, 61.5)
- moved R13 26.7 mm to (53.2, 63.3)
- moved U1 26.7 mm to (158.5, 59.3)
- moved J1 26.7 mm to (119.3, 73.5)
Routing:
- added copper zone on B.Cu, net GND
- added copper zone on F.Cu, net GND
Changed lines of the file:
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@@
 		(allow_soldermask_bridges_in_footprints no)
 		(tenting front back)
-		(grid_origin 31.3379 16.491)
+		(grid_origin 40.8379 41.491)
 		(pcbplotparams
 			(layerselection 0x00000000_00000000_55555555_5755f5ff)
@@
 	(footprint "Resistor_THT:R_Axial_DIN0204_L3.6mm_D1.6mm_P7.62mm_Horizontal"
 		(layer "F.Cu")
-		(at 43.6779 38.251 90)
+		(at 53.1779 63.251 90)
 		(descr "Resistor, Axial_DIN0204 series, Axial, Horizontal, pin pitch=7.62mm, 0.167W, length*diameter=3.6*1.6mm^2, http://cdn-reichelt.de/documents/datenblatt/B400/1_4W%23YAG.pdf")
 		(tags "Resistor Axial_DIN0204 series Axial Horizontal pin pitch 7.62mm 0.167W length 3.6mm diameter 1.6mm")
@@
 	(footprint "footprints:Arduino_Micro_Socket"
 		(layer "F.Cu")
-		(at 97.3379 26.371 180)
+		(at 106.8379 51.371 180)
 		(descr "https://docs.arduino.cc/hardware/micro")
 		(property "Reference" "A1"
@@
 	(footprint "TerminalBlock_Phoenix:TerminalBlock_Phoenix_MPT-0,5-2-2.54_1x02_P2.54mm_Horizontal"
 		(layer "F.Cu")
-		(at 109.7979 48.451)
+		(at 119.2979 73.451)
 		(descr "Terminal Block Phoenix MPT-0,5-2-2.54, 2 pins, pitch 2.54mm, size 5.54x6.2mm, drill diameter 1.1mm, pad diameter 2.2mm, http://www.mouser.com/ds/2/324/ItemDetail_1725656-920552.pdf, script-generated using https://gitlab.com/kicad/libraries/kicad-footprint-generator/-/tree/master/scripts/TerminalBlock_Phoenix")
 		(tags "THT Terminal Block Phoenix MPT-0,5-2-2.54 pitch 2.54mm size 5.54x6.2mm drill 1.1mm pad 2.2mm")
@@
 	(footprint "Package_LGA:Bosch_LGA-8_3x3mm_P0.8mm_ClockwisePinNumbering"
 		(layer "F.Cu")
-		(at 149.0254 34.291 90)
+		(at 158.5254 59.291 90)
 		(descr "Bosch  LGA, 8 Pin (https://ae-bst.resource.bosch.com/media/_tech/media/datasheets/BST-BME680-DS001-00.pdf#page=44), generated with kicad-footprint-generator ipc_noLead_generator.py")
 		(tags "Bosch LGA NoLead")
@@
 	(footprint "TerminalBlock_Phoenix:TerminalBlock_Phoenix_MPT-0,5-2-2.54_1x02_P2.54mm_Horizontal"
 		(layer "F.Cu")
-		(at 111.6079 24.6235 180)
+		(at 121.1079 49.6235 180)
 		(descr "Terminal Block Phoenix MPT-0,5-2-2.54, 2 pins, pitch 2.54mm, size 5.54x6.2mm, drill diameter 1.1mm, pad diameter 2.2mm, http://www.mouser.com/ds/2/324/ItemDetail_1725656-920552.pdf, script-generated using https://gitlab.com/kicad/libraries/kicad-footprint-generator/-/tree/master/scripts/TerminalBlock_Phoenix")
 		(tags "THT Terminal Block Phoenix MPT-0,5-2-2.54 pitch 2.54mm size 5.54x6.2mm drill 1.1mm pad 2.2mm")
@@
 	(footprint "TerminalBlock_Phoenix:TerminalBlock_Phoenix_MPT-0,5-2-2.54_1x02_P2.54mm_Horizontal"
 		(layer "F.Cu")
-		(at 123.2979 36.491 90)
+		(at 132.7979 61.491 90)
 		(descr "Terminal Block Phoenix MPT-0,5-2-2.54, 2 pins, pitch 2.54mm, size 5.54x6.2mm, drill diameter 1.1mm, pad diameter 2.2mm, http://www.mouser.com/ds/2/324/ItemDetail_1725656-920552.pdf, script-generated using https://gitlab.com/kicad/libraries/kicad-footprint-generator/-/tree/master/scripts/TerminalBlock_Phoenix")
 		(tags "THT Terminal Block Phoenix MPT-0,5-2-2.54 pitch 2.54mm size 5.54x6.2mm drill 1.1mm pad 2.2mm")
@@
 	(footprint "Connector_Wire:SolderWire-0.25sqmm_1x03_P4.5mm_D0.65mm_OD2mm"
 		(layer "F.Cu")
-		(at 38.3379 28.991 -90)
+		(at 47.8379 53.991 -90)
 		(descr "Soldered wire connection, for 3 times 0.25 mm² wires, reinforced insulation, conductor diameter 0.65mm, outer diameter 2mm, size source Multi-Contact FLEXI-2V 0.25 (https://ec.staubli.com/AcroFiles/Catalogues/TM_Cab-Main-11014119_(en)_hi.pdf), bend radius 3 times outer diameter, generated with kicad-footprint-generator")
 		(tags "connector wire 0.25sqmm")
@@
 	)
 	(gr_rect
-		(start 31.3379 16.491)
-		(end 160.3379 55.491)
+		(start 40.8379 41.491)
+		(end 169.8379 80.491)
 		(stroke
 			(width 0.05)
@@
 		(layer "Edge.Cuts")
 	)
+	(zone
+		(net 12)
+		(net_name "GND")
+		(layers "F.Cu" "B.Cu")
+		(hatch edge 0.5)
+		(connect_pads
+			(clearance 0.5)
+		)
+		(min_thickness 0.25)
+		(filled_areas_thickness no)
+		(fill yes
+			(thermal_gap 0.5)
+			(thermal_bridge_width 0.5)
+		)
+		(polygon
+			(pts
+				(xy 175.8379 34.991) (xy 175.8379 85.991) (xy 174.8379 86.991) (xy 36.8379 86.991) (xy 36.8379 34.991)
+			)
+		)
+	)
 	(embedded_fonts no)

Commit message: Fins, Femmes and Gems
Parts:
- moved J1 47.7 mm to (158.3, 46.0)
- moved J2 30.4 mm to (151.3, 46.0)
- moved J11 26.6 mm to (71.8, 65.5), turned to 90 degrees
- moved R13 25.9 mm to (78.3, 57.2), turned to -90 degrees
- moved A1 25.3 mm to (89.3, 69.6), turned to 0 degrees
- moved J3 16.3 mm to (139.3, 46.5)
- moved U1 2.61 mm to (160.8, 60.5)
Other:
- board size 129 x 39 mm -> 128 x 38 mm

Commit message: The Reckoning
Parts:
- removed J11: Conn_01x03_Socket, Connector_Wire:SolderWire-0.25sqmm_1x03_P4.5mm_D0.65mm_OD2mm
- added J4: Screw_Terminal_01x03, TerminalBlock_Phoenix:TerminalBlock_Phoenix_MPT-0,5-3-2.54_1x03_P2.54mm_Horizontal, F.Cu at (61.3, 58.0)
- moved J1 97.1 mm to (61.3, 50.4), turned to -90 degrees
- moved J2 92.7 mm to (61.3, 68.1), turned to -90 degrees
- moved J3 15.3 mm to (140.8, 61.8)
- moved R13 11.1 mm to (69.0, 63.0), turned to 0 degrees
- moved A1 8.26 mm to (81.0, 69.5)
- moved U1 0.08 mm to (160.8, 60.4)
Connections:
- net /5V renamed +5V
- net Net-(A1-SPI_CS) renamed /SS
- net Net-(A1-SPI_MISO) renamed /MISO
- net Net-(A1-SPI_MOSI) renamed /MOSI
- net Net-(A1-SPI_SCK) renamed /SCK
- A1 pad 3V3: /3V3 -> unconnected-(A1-3.3V-Pad3V3)
- A1 pad A1: /A1 -> unconnected-(A1-PadA1)
- A1 pad D0: /D0 -> unconnected-(A1-D0/RX-PadD0)
- A1 pad D1: /D1 -> unconnected-(A1-D1/TX-PadD1)
- A1 pad D2: /SDA -> /D2
- A1 pad D3: /SCL -> /D3
- A1 pad D4: /D4 -> unconnected-(A1-PadD4)
- A1 pad D5: /D5 -> unconnected-(A1-PadD5)
- A1 pad D6: /D6 -> unconnected-(A1-PadD6)
- A1 pad D8: /D8 -> unconnected-(A1-PadD8)
- J1 pad 2: /D1 -> /D3
- J3 pad 2: /D0 -> /D2
Routing:
- net +12V: track 0.00 -> 67.3 mm, vias 0 -> 1
- net +5V: track 0.00 -> 54.3 mm
- net /D3: track 0.00 -> 47.7 mm
- net /MISO: track 0.00 -> 45.8 mm
- net /D7: track 0.00 -> 45.3 mm, vias 0 -> 1
- net /SCK: track 0.00 -> 42.4 mm, vias 0 -> 1
- net /SS: track 0.00 -> 40.1 mm
- net /MOSI: track 0.00 -> 37.0 mm
- net /D2: track 0.00 -> 33.7 mm
- net /A0: track 0.00 -> 32.5 mm

Commit message: Tsunami
Routing:
- net /SS: track 40.1 -> 45.9 mm, vias 0 -> 1
- net +12V: track 67.3 -> 65.1 mm
- net /MOSI: track 37.0 -> 38.6 mm
- net /SCK: track 42.4 -> 43.4 mm
- net GND: track 0.00 -> 0.76 mm, vias 0 -> 1
- net /D7: track 45.3 -> 45.9 mm
- net /MISO: track 45.8 -> 45.4 mm, vias 0 -> 1
