File: kicad/SonTinh/SonTinh.kicad_pcb (KiCad board)
At the start: 2 copper layers, 128 x 38 mm, 7 parts, among them J1 Screw_Terminal_01x02, J2 Screw_Terminal_01x02, J3 Screw_Terminal_01x02, J4 Screw_Terminal_01x03, U1 BME680

Commit message: The Titans
Parts:
- removed J1, J2: Screw_Terminal_01x02, TerminalBlock_Phoenix:TerminalBlock_Phoenix_MPT-0,5-2-2.54_1x02_P2.54mm_Horizontal
- removed J4: Screw_Terminal_01x03, TerminalBlock_Phoenix:TerminalBlock_Phoenix_MPT-0,5-3-2.54_1x03_P2.54mm_Horizontal
- added J5: Screw_Terminal_01x07, TerminalBlock_WAGO:TerminalBlock_WAGO_233-507_2x07_P2.54mm, F.Cu at (86.3, 54.4)
- added R14: 10k, Resistor_THT:R_Axial_DIN0204_L3.6mm_D1.6mm_P7.62mm_Horizontal, F.Cu at (66.4, 56.0)
- added R15: 10k, Resistor_THT:R_Axial_DIN0204_L3.6mm_D1.6mm_P7.62mm_Horizontal, F.Cu at (66.4, 59.1)
- added R16: 10k, Resistor_THT:R_Axial_DIN0204_L3.6mm_D1.6mm_P7.62mm_Horizontal, F.Cu at (66.4, 62.3)
- added R17: 10k, Resistor_THT:R_Axial_DIN0204_L3.6mm_D1.6mm_P7.62mm_Horizontal, F.Cu at (66.4, 65.4)
- added U2: TCA9517ADGK, Package_SO:VSSOP-8_3x3mm_P0.65mm, F.Cu at (58.3, 60.6)
- J3: value Screw_Terminal_01x02 -> Conn_01x02_Socket; footprint TerminalBlock_Phoenix:TerminalBlock_Phoenix_MPT-0,5-2-2.54_1x02_P2.54mm_Horizontal -> Connector_Wire:SolderWire-0.5sqmm_1x02_P4.8mm_D0.9mm_OD2.3mm
- moved U1 109.0 mm to (51.8, 60.6), turned to 180 degrees
- moved R13 23.4 mm to (92.3, 64.3), turned to 90 degrees
- moved A1 16.8 mm to (97.8, 70.1)
- moved J3 13.5 mm to (154.3, 62.3)
Connections:
- A1 pad 3V3: unconnected-(A1-3.3V-Pad3V3) -> +3V3
- A1 pad D2: /D2 -> Net-(A1-D2/SDA)
- A1 pad D3: /D3 -> Net-(A1-D3/SCL)
- U1 pad 2: /SS -> +3V3
- U1 pad 3: /MOSI -> Net-(U1-SDI)
- U1 pad 4: /SCK -> Net-(U1-SCK)
- U1 pad 5: /MISO -> GND
- U1 pad 6: +5V -> +3V3
- U1 pad 8: +5V -> +3V3
Routing:
- net Net-(A1-D3/SCL): track 0.00 -> 79.5 mm
- net +3V3: track 0.00 -> 73.8 mm, vias 0 -> 2
- net Net-(A1-D2/SDA): track 0.00 -> 73.2 mm
- net /SS: track 45.9 -> 0.00 mm, vias 1 -> 0
- net /MISO: track 45.4 -> 0.00 mm, vias 1 -> 0
- net /SCK: track 43.4 -> 0.00 mm, vias 1 -> 0
- net /D3: track 47.6 -> 5.00 mm
- net /MOSI: track 38.6 -> 0.00 mm
- net /D2: track 33.7 -> 0.00 mm
- net +5V: track 54.3 -> 82.4 mm
- net Net-(U1-SDI): track 0.00 -> 24.9 mm
- net Net-(U1-SCK): track 0.00 -> 18.6 mm
- net /A0: track 32.5 -> 28.8 mm
- net +12V: track 65.1 -> 68.0 mm
- net /D7: track 45.9 -> 44.2 mm
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
Commit message: Beware Greeks Bearing Gifts
Parts:
- removed J3: Conn_01x02_Socket, Connector_Wire:SolderWire-0.5sqmm_1x02_P4.8mm_D0.9mm_OD2.3mm
- removed J5: Screw_Terminal_01x07, TerminalBlock_WAGO:TerminalBlock_WAGO_233-507_2x07_P2.54mm
- added J1: 1823353, footprints:1823353, F.Cu at (78.3, 51.2)
- added J2: 1823638, footprints:1823638, F.Cu at (160.3, 63.5)
- R13, R14, R15, R16, R17: footprint Resistor_THT:R_Axial_DIN0204_L3.6mm_D1.6mm_P7.62mm_Horizontal -> Resistor_SMD:R_0805_2012Metric
- turned R13 to -90 degrees
- turned U1 to -90 degrees
Routing:
- net +5V: track 82.4 -> 0.00 mm
- net Net-(A1-D3/SCL): track 79.5 -> 0.00 mm
- net +3V3: track 73.8 -> 0.00 mm, vias 2 -> 0
- net Net-(A1-D2/SDA): track 73.2 -> 0.00 mm
- net +12V: track 68.0 -> 0.00 mm, vias 1 -> 0
- net /D7: track 44.2 -> 0.00 mm, vias 1 -> 0
- net /A0: track 28.8 -> 0.00 mm
- net Net-(U1-SDI): track 24.9 -> 0.00 mm
- net Net-(U1-SCK): track 18.6 -> 0.00 mm
- net /D3: track 5.00 -> 0.00 mm

Commit message: Athens City Academy of the Performing Bards
Parts:
- moved R13 9.19 mm to (84.8, 59.0)
- moved J1 7.26 mm to (71.8, 47.9)
- moved J2 6.88 mm to (154.3, 60.1)
- moved A1 6.18 mm to (91.8, 68.6)
- moved U1 5.22 mm to (46.8, 59.1)
- moved R14 4.92 mm to (61.8, 54.3)
- moved R15 4.92 mm to (61.8, 57.4)
- moved R17 4.92 mm to (61.8, 63.7)
- moved R16 4.92 mm to (61.8, 60.6), turned to 180 degrees
- moved U2 2.18 mm to (56.8, 59.0)
Connections:
- J1 pad 12: unconnected-(J1-6.2-Pad12) -> GND
Routing:
- net +5V: track 0.00 -> 79.2 mm, vias 0 -> 1
- net +12V: track 0.00 -> 75.0 mm, vias 0 -> 1
- net Net-(A1-D2/SDA): track 0.00 -> 70.0 mm
- net Net-(A1-D3/SCL): track 0.00 -> 69.4 mm, vias 0 -> 1
- net +3V3: track 0.00 -> 62.5 mm
- net /D7: track 0.00 -> 40.8 mm
- net /A0: track 0.00 -> 33.2 mm
- net Net-(U1-SDI): track 0.00 -> 27.0 mm
- net Net-(U1-SCK): track 0.00 -> 15.5 mm
- net /D2: track 0.00 -> 7.00 mm
- net /D3: track 0.00 -> 5.50 mm
- net GND: track 0.00 -> 0.94 mm, vias 0 -> 1
Other:
- board size 128 x 38 mm -> 120 x 35 mm
- board text added: "+12V"
- board text added: "-12V"
- board text added: "A0"
- board text added: "BUS"
- board text added: "GND"
- board text added: "INT"

Commit message: A Fistful of Dinars
Parts:
- added J3: Conn_01x02_Pin, Connector_Wire:SolderWire-0.75sqmm_1x02_P4.8mm_D1.25mm_OD2.3mm, F.Cu at (75.8, 64.9)
- added J4: Conn_01x02_Pin, Connector_Wire:SolderWire-0.75sqmm_1x02_P4.8mm_D1.25mm_OD2.3mm, F.Cu at (75.8, 74.4)
- J1: value 1823353 -> Conn_01x02_Pin; footprint footprints:1823353 -> Connector_Wire:SolderWire-0.75sqmm_1x02_P4.8mm_D1.25mm_OD2.3mm
- J2: value 1823638 -> Conn_01x03_Pin; footprint footprints:1823638 -> Connector_Wire:SolderWire-0.75sqmm_1x03_P4.8mm_D1.25mm_OD2.3mm
- moved J2 78.6 mm to (75.8, 56.0)
- moved J1 77.6 mm to (148.3, 61.0), turned to 90 degrees
Connections:
- J1 pad 1: +12V -> GND
- J1 pad 2: +12V -> /D2
- J2 pad 1: GND -> /D7
- J2 pad 3: /D2 -> +12V
Routing:
- net +5V: track 79.2 -> 0.00 mm, vias 1 -> 0
- net +12V: track 75.0 -> 0.00 mm, vias 1 -> 0
- net Net-(A1-D2/SDA): track 70.0 -> 0.00 mm
- net Net-(A1-D3/SCL): track 69.4 -> 0.00 mm, vias 1 -> 0
- net +3V3: track 62.5 -> 0.00 mm
- net /D7: track 40.8 -> 0.00 mm
- net /A0: track 33.2 -> 0.00 mm
- net Net-(U1-SDI): track 27.0 -> 0.00 mm
- net Net-(U1-SCK): track 15.5 -> 0.00 mm
- net /D2: track 7.00 -> 0.00 mm
- net /D3: track 5.50 -> 0.00 mm
- net GND: track 0.94 -> 0.00 mm, vias 1 -> 0

Commit message: Warrior... Princess
Parts:
- J1: value Conn_01x02_Pin -> Conn_01x02_Socket; footprint Connector_Wire:SolderWire-0.75sqmm_1x02_P4.8mm_D1.25mm_OD2.3mm -> Connector_JST:JST_EH_S2B-EH_1x02_P2.50mm_Horizontal
- J2: value Conn_01x03_Pin -> Conn_01x02_Socket; footprint Connector_Wire:SolderWire-0.75sqmm_1x03_P4.8mm_D1.25mm_OD2.3mm -> Connector_JST:JST_EH_B2B-EH-A_1x02_P2.50mm_Vertical
- J3: value Conn_01x02_Pin -> Conn_01x02_Socket; footprint Connector_Wire:SolderWire-0.75sqmm_1x02_P4.8mm_D1.25mm_OD2.3mm -> Connector_JST:JST_EH_B2B-EH-A_1x02_P2.50mm_Vertical
- J4: value Conn_01x02_Pin -> Conn_01x03_Socket; footprint Connector_Wire:SolderWire-0.75sqmm_1x02_P4.8mm_D1.25mm_OD2.3mm -> Connector_JST:JST_EH_B3B-EH-A_1x03_P2.50mm_Vertical
- moved J2 23.4 mm to (97.1, 46.3), turned to 180 degrees
- moved J3 19.9 mm to (94.6, 71.7), turned to 0 degrees
- moved J4 13.5 mm to (71.8, 61.5)
- moved J1 6.39 mm to (142.8, 57.7), turned to -90 degrees
- moved A1 4.80 mm to (87.0, 68.0)
- moved R13 4.72 mm to (80.8, 56.5), turned to 0 degrees
Connections:
- A1 pad D0: unconnected-(A1-D0/RX-PadD0) -> /D0
- A1 pad D1: unconnected-(A1-D1/TX-PadD1) -> /D1
- J1 pad 1: GND -> /D0
- J1 pad 2: /D2 -> GND
- J2 pad 1: /D7 -> /D1
- J3 pad 2: /D3 -> /A0
- J4 pad 1: /A0 -> +12V
Routing:
- net +5V: track 0.00 -> 78.0 mm
- net Net-(A1-D2/SDA): track 0.00 -> 64.2 mm
- net Net-(A1-D3/SCL): track 0.00 -> 62.1 mm
- net +3V3: track 0.00 -> 60.2 mm
- net +12V: track 0.00 -> 56.8 mm
- net /D7: track 0.00 -> 34.1 mm
- net /D1: track 0.00 -> 31.5 mm
- net /D0: track 0.00 -> 21.7 mm
- net Net-(U1-SCK): track 0.00 -> 15.6 mm
- net Net-(U1-SDI): track 0.00 -> 14.5 mm
- net /A0: track 0.00 -> 5.66 mm
- net GND: track 0.00 -> 0.89 mm, vias 0 -> 2
Other:
- board size 120 x 35 mm -> 110 x 35 mm
- board text removed: "+12V"
- board text removed: "-12V"
- board text removed: "A0"
- board text removed: "BUS"
- board text removed: "GND"
- board text removed: "INT"

Commit message: Here She Comes... Miss Amphipolis
Parts:
- removed J1: Conn_01x02_Socket, Connector_JST:JST_EH_S2B-EH_1x02_P2.50mm_Horizontal
- removed J2, J3: Conn_01x02_Socket, Connector_JST:JST_EH_B2B-EH-A_1x02_P2.50mm_Vertical
- removed J4: Conn_01x03_Socket, Connector_JST:JST_EH_B3B-EH-A_1x03_P2.50mm_Vertical
- added J8: 791077010, footprints:CONN22_791077010_MOL, F.Cu at (73.8, 68.5)
- moved R13 14.6 mm to (68.6, 64.5), turned to 180 degrees
Connections:
- net Net-(A1-D2/SDA) renamed /SDA_5V
- net Net-(A1-D3/SCL) renamed /SCL_5V
- net Net-(U1-SCK) renamed /SCL_3V3
- net Net-(U1-SDI) renamed /SDA_3V3
- A1 pad A1: unconnected-(A1-PadA1) -> /A1
Routing:
- net /SDA_3V3: track 14.5 -> 56.7 mm, vias 0 -> 1
- net /A1: track 0.00 -> 41.4 mm, vias 0 -> 1
- net /D0: track 21.7 -> 59.2 mm, vias 0 -> 1
- net /A0: track 5.66 -> 36.0 mm, vias 0 -> 1
- net /D1: track 31.5 -> 56.6 mm
- net /SCL_3V3: track 15.6 -> 31.5 mm
- net /D7: track 34.1 -> 46.8 mm, vias 0 -> 2
- net +5V: track 78.0 -> 85.6 mm, vias 0 -> 2
- net /SDA_5V: track 64.2 -> 71.7 mm, vias 0 -> 1
- net +3V3: track 60.2 -> 56.8 mm
- net +12V: track 56.8 -> 54.3 mm
- net /SCL_5V: track 62.1 -> 64.2 mm
- net GND: track 0.89 -> 2.30 mm

Commit message: Destiny
Connections:
- A1 pad VIN: +12V -> Net-(D1-K)
Routing:
- net +5V: track 85.6 -> 0.00 mm, vias 2 -> 0
- net /SDA_5V: track 71.7 -> 0.00 mm, vias 1 -> 0
- net /SCL_5V: track 64.2 -> 0.00 mm
- net /D0: track 59.2 -> 0.00 mm, vias 1 -> 0
- net +3V3: track 56.8 -> 0.00 mm
- net /SDA_3V3: track 56.7 -> 0.00 mm, vias 1 -> 0
- net /D1: track 56.6 -> 0.00 mm
- net +12V: track 54.3 -> 0.00 mm
- net /D7: track 46.8 -> 0.00 mm, vias 2 -> 0
- net /A1: track 41.4 -> 0.00 mm, vias 1 -> 0
- net /A0: track 36.0 -> 0.00 mm, vias 1 -> 0
- net /SCL_3V3: track 31.5 -> 0.00 mm
- net GND: track 2.30 -> 0.00 mm, vias 2 -> 0

Commit message: A Day in the Life
Parts:
- removed J8: 791077010, footprints:CONN22_791077010_MOL
- added J1: 1823450, footprints:1823450, F.Cu at (93.1, 46.7)
- added J2: 1823450, footprints:1823450, F.Cu at (82.3, 46.7)
- added J3: 1823450, footprints:1823450, F.Cu at (71.6, 46.7)
- added J4: 1823450, footprints:1823450, F.Cu at (60.8, 46.7)
- R13, R14, R15, R16, R17, U2: moved to B.Cu
- moved A1 65.7 mm to (149.9, 49.1), turned to 180 degrees
- moved U2 56.0 mm to (112.8, 58.1), turned to -90 degrees
- moved R13 52.1 mm to (120.3, 58.0)
- moved R17 45.6 mm to (106.3, 53.6)
- moved R14 45.4 mm to (106.3, 63.0)
- moved R16 44.7 mm to (106.3, 56.7)
- moved R15 44.6 mm to (106.3, 59.9)
- moved U1 2.21 mm to (45.5, 57.3)
Connections:
- A1 pad VIN: Net-(D1-K) -> +12V
