File: kicad/SonTinh/SonTinh.kicad_pcb (KiCad board)
At the start: 2 copper layers, 110 x 35 mm, 12 parts, among them J1 1823450, J2 1823450, J3 1823450, J4 1823450, U1 BME680, U2 TCA9517ADGK

Commit message: For Him the Bell Tolls
Parts:
- added J5: 1752117, footprints:1752117, F.Cu at (95.3, 71.0)
- added J6: 1752117, footprints:1752117, F.Cu at (53.8, 63.5)
- added J7: 1752117, footprints:1752117, F.Cu at (67.3, 70.5)
- J1, J2, J3, J4: value 1823450 -> 1752117; footprint footprints:1823450 -> footprints:1752117
- moved A1 49.0 mm to (104.3, 66.9), turned to 0 degrees
- moved J4 31.4 mm to (80.8, 71.0), turned to 90 degrees
- moved J1 26.6 mm to (67.3, 53.5), turned to 90 degrees
- moved J3 24.2 mm to (94.6, 54.1), turned to 90 degrees
- moved J2 7.89 mm to (80.8, 54.5), turned to 90 degrees
- moved U1 1.80 mm to (44.5, 58.8)
Connections:
- J1 pad 1: GND -> unconnected-(J1-Pad1)
- J1 pad 2: GND -> unconnected-(J1-Pad2)
- J1 pad 3: +3V3 -> unconnected-(J1-Pad3)
- J2 pad 1: GND -> unconnected-(J2-Pad1)
- J2 pad 2: GND -> unconnected-(J2-Pad2)
- J2 pad 3: +3V3 -> unconnected-(J2-Pad3)
- J3 pad 1: GND -> unconnected-(J3-Pad1)
- J3 pad 2: GND -> unconnected-(J3-Pad2)
- J3 pad 3: +3V3 -> unconnected-(J3-Pad3)
- J4 pad 1: GND -> unconnected-(J4-Pad1)
- J4 pad 2: GND -> unconnected-(J4-Pad2)
- J4 pad 3: +3V3 -> unconnected-(J4-Pad3)

Commit message: Blind Faith
Parts:
- removed J5, J6, J7: 1752117, footprints:1752117
- added H1: MountingHole_Pad, MountingHole:MountingHole_3.5mm_Pad, F.Cu at (70.8, 70.0)
- added H2: MountingHole_Pad, MountingHole:MountingHole_3.5mm_Pad, F.Cu at (50.8, 48.0)
- J1, J2: value 1752117 -> Screw_Terminal_01x02; footprint footprints:1752117 -> footprints:MKDSFW_15_2_35
- J3: value 1752117 -> Screw_Terminal_01x02; footprint footprints:1752117 -> footprints:MKDS_15_2_35
- J4: value 1752117 -> Screw_Terminal_01x03; footprint footprints:1752117 -> footprints:MKDS_15_3_35
- moved J3 50.2 mm to (144.4, 60.7)
- moved R14 25.5 mm to (131.8, 63.6)
- moved R15 25.5 mm to (131.8, 60.5)
- moved R16 25.5 mm to (131.8, 57.3)
- moved R17 25.5 mm to (131.8, 54.2)
- moved J1 15.9 mm to (78.8, 64.4), turned to 0 degrees
- moved A1 15.0 mm to (89.3, 68.0)
- moved J4 13.1 mm to (70.8, 62.5)
- moved U2 11.1 mm to (123.8, 59.3), turned to 0 degrees
- moved R13 7.21 mm to (113.3, 59.7), turned to 90 degrees
- moved U1 6.32 mm to (50.8, 59.1), turned to 0 degrees
- moved J2 1.78 mm to (82.3, 53.5), turned to 180 degrees
Connections:
- J1 pad 1: unconnected-(J1-Pad1) -> /D0
- J1 pad 2: unconnected-(J1-Pad2) -> GND
- J2 pad 1: unconnected-(J2-Pad1) -> /A0
- J2 pad 2: unconnected-(J2-Pad2) -> GND
- J3 pad 1: unconnected-(J3-Pad1) -> /D1
- J3 pad 2: unconnected-(J3-Pad2) -> GND
- J4 pad 1: unconnected-(J4-Pad1) -> +12V
- J4 pad 2: unconnected-(J4-Pad2) -> /D7
- J4 pad 3: unconnected-(J4-Pad3) -> GND
- R13 pad 1: /D7 -> GND
- R13 pad 2: GND -> /D7
Routing:
- net +3V3: track 0.00 -> 98.0 mm
- net /SCL_3V3: track 0.00 -> 83.4 mm, vias 0 -> 1
- net /SDA_3V3: track 0.00 -> 83.3 mm, vias 0 -> 1
- net /D0: track 0.00 -> 60.4 mm, vias 0 -> 1
- net +12V: track 0.00 -> 59.7 mm
- net /D7: track 0.00 -> 50.7 mm
- net /SDA_5V: track 0.00 -> 30.2 mm
- net /A0: track 0.00 -> 24.1 mm
- net /SCL_5V: track 0.00 -> 20.5 mm, vias 0 -> 1
- net +5V: track 0.00 -> 20.4 mm
- net /D1: track 0.00 -> 19.7 mm
- net GND: track 0.00 -> 11.3 mm, vias 0 -> 2

Commit message: Been There, Done That
Parts:
- removed U1: BME680, Package_LGA:Bosch_LGA-8_3x3mm_P0.8mm_ClockwisePinNumbering
- added C1: C, Capacitor_SMD:C_0805_2012Metric, F.Cu at (56.8, 67.0)
- added IC1: SHT35-DIS-F2.5kS, footprints:SON50P250X250X100-9N-D, F.Cu at (61.5, 50.7)
- added IC2: STC31-C-R3, footprints:QFN80P300X350X110-13N-D, F.Cu at (51.5, 59.8)
- added IC3: BMP384, footprints:BMP384, F.Cu at (56.7, 59.4)
Routing:
- net +3V3: track 98.0 -> 0.00 mm
- net /SCL_3V3: track 83.4 -> 0.00 mm, vias 1 -> 0
- net /SDA_3V3: track 83.3 -> 0.00 mm, vias 1 -> 0
- net /D0: track 60.4 -> 0.00 mm, vias 1 -> 0
- net +12V: track 59.7 -> 0.00 mm
- net /D7: track 50.7 -> 0.00 mm
- net /SDA_5V: track 30.2 -> 0.00 mm
- net /A0: track 24.1 -> 0.00 mm
- net /SCL_5V: track 20.5 -> 0.00 mm, vias 1 -> 0
- net +5V: track 20.4 -> 0.00 mm
- net /D1: track 19.7 -> 0.00 mm
- net GND: track 11.3 -> 0.00 mm, vias 2 -> 0

Commit message: Little Problems
Parts:
- J1, J2: footprint footprints:MKDSFW_15_2_35 -> TerminalBlock_Phoenix:TerminalBlock_Phoenix_PT-1,5-2-3.5-H_1x02_P3.50mm_Horizontal
- J3: footprint footprints:MKDS_15_2_35 -> TerminalBlock_Phoenix:TerminalBlock_Phoenix_PT-1,5-2-3.5-H_1x02_P3.50mm_Horizontal
- J4: footprint footprints:MKDS_15_3_35 -> TerminalBlock_Phoenix:TerminalBlock_Phoenix_PT-1,5-3-3.5-H_1x03_P3.50mm_Horizontal
- R13, R14, R15, R16, R17, U2: moved to F.Cu
- moved U2 52.2 mm to (72.3, 50.6), turned to -90 degrees
- moved R14 50.2 mm to (83.3, 50.8)
- moved R13 49.5 mm to (64.3, 53.0), turned to -90 degrees
- moved R15 48.9 mm to (83.3, 54.0)
- moved R17 48.9 mm to (83.3, 60.3)
- moved R16 48.5 mm to (83.3, 57.1)
- moved J1 39.2 mm to (117.8, 68.5)
- moved J2 30.4 mm to (108.8, 68.5), turned to 0 degrees
- moved J4 26.2 mm to (96.3, 68.5), turned to 0 degrees
- moved J3 19.2 mm to (126.8, 68.5), turned to 0 degrees
- moved IC1 14.9 mm to (47.5, 55.7)
- moved IC2 11.2 mm to (47.5, 70.2)
- moved IC3 6.87 mm to (63.6, 59.5)
- moved A1 5.40 mm to (89.2, 62.6)
- moved H1 5.00 mm to (75.8, 70.0)

Commit message: Gabrielle's Hope
Parts:
- added C2: C, Capacitor_SMD:C_0805_2012Metric, F.Cu at (62.3, 59.0)
- R13: moved to B.Cu
- moved R13 42.7 mm to (106.8, 48.0), turned to 180 degrees
- moved IC2 30.0 mm to (75.3, 59.0), turned to 180 degrees
- moved C1 26.0 mm to (68.8, 44.0)
- moved R17 16.0 mm to (82.3, 44.3), turned to 180 degrees
- moved IC3 12.6 mm to (68.8, 48.0)
- moved R16 9.70 mm to (82.3, 47.5), turned to 0 degrees
- moved H1 5.00 mm to (80.8, 70.0)
- moved U2 4.00 mm to (75.3, 48.0)
- moved IC1 3.66 mm to (49.1, 59.0), turned to 180 degrees
- moved R15 3.50 mm to (82.3, 50.6), turned to 180 degrees
- moved R14 3.11 mm to (82.3, 53.8), turned to 180 degrees
- moved J1 2.00 mm to (117.8, 66.5)
- moved J2 2.00 mm to (108.8, 66.5)
- moved J3 2.00 mm to (126.8, 66.5)
- moved J4 2.00 mm to (96.3, 66.5)
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Connections:
- IC1 pad 1: unconnected-(IC1-SDA-Pad1) -> /SDA_5V
- IC1 pad 2: unconnected-(IC1-ADDR-Pad2) -> GND
- IC1 pad 4: unconnected-(IC1-SCL-Pad4) -> /SCL_5V
- IC1 pad 5: unconnected-(IC1-VDD-Pad5) -> +5V
- IC1 pad 7: unconnected-(IC1-R-Pad7) -> GND
- IC1 pad 8: unconnected-(IC1-VSS-Pad8) -> GND
- IC1 pad 9: unconnected-(IC1-EP-Pad9) -> GND
- IC2 pad 1: unconnected-(IC2-VSS_1-Pad1) -> GND
- IC2 pad 11: unconnected-(IC2-VSS_4-Pad11) -> GND
- IC2 pad 13: unconnected-(IC2-EP-Pad13) -> GND
- IC2 pad 3: unconnected-(IC2-ADDR-Pad3) -> GND
- IC2 pad 4: unconnected-(IC2-SCL-Pad4) -> /SCL_5V
- IC2 pad 5: unconnected-(IC2-VSS_2-Pad5) -> GND
- IC2 pad 6: unconnected-(IC2-VDD-Pad6) -> +5V
- IC2 pad 7: unconnected-(IC2-SDA-Pad7) -> /SDA_5V
- IC2 pad 9: unconnected-(IC2-VSS_3-Pad9) -> GND
- IC3 pad 5: /A2 -> GND
- IC3 pad 6: unconnected-(IC3-CSB-Pad6) -> +3V3
Routing:
- net +5V: track 0.00 -> 93.1 mm, vias 0 -> 3
- net /SCL_5V: track 0.00 -> 87.9 mm, vias 0 -> 3
- net /SDA_5V: track 0.00 -> 84.0 mm, vias 0 -> 2
- net +3V3: track 0.00 -> 53.7 mm, vias 0 -> 3
- net +12V: track 0.00 -> 35.0 mm
- net /SDA_3V3: track 0.00 -> 29.9 mm
- net /D0: track 0.00 -> 24.9 mm
- net /D7: track 0.00 -> 24.3 mm
- net /D1: track 0.00 -> 22.3 mm
- net /SCL_3V3: track 0.00 -> 18.5 mm
- net GND: track 0.00 -> 11.8 mm, vias 0 -> 2
- net /A0: track 0.00 -> 10.9 mm
Other:
- board text added: "+12V"
- board text added: "A0"
- board text added: "BUS"
- board text added: "GND"
- board text added: "INT0"
- board text added: "INT1"

Commit message: Old Ares had a Farm
Parts:
- added C3: 10uF, Capacitor_SMD:C_1206_3216Metric, F.Cu at (147.6, 71.4)
- added C4: 10uF, Capacitor_SMD:C_0805_2012Metric, F.Cu at (147.4, 66.3)
- added U7: R-78E5.0-1.0, Converter_DCDC:Converter_DCDC_RECOM_R-78E-0.5_THT, F.Cu at (142.8, 71.5)
- R13: moved to F.Cu
- turned IC2 to -90 degrees
- turned IC3 to -90 degrees
Connections:
- A1 pad VIN: +12V -> unconnected-(A1-PadVIN)
Routing:
- net +5V: track 93.1 -> 135.1 mm, vias 3 -> 2
- net +12V: track 35.0 -> 54.5 mm
- net /SDA_3V3: track 29.9 -> 23.0 mm
- net +3V3: track 53.7 -> 50.7 mm, vias 3 -> 1
- net /D7: track 24.3 -> 27.2 mm
- net /SCL_3V3: track 18.5 -> 16.9 mm
- net /SCL_5V: track 87.9 -> 86.4 mm
- net /SDA_5V: track 84.0 -> 84.9 mm, vias 2 -> 3
- net GND: track 11.8 -> 11.1 mm, vias 2 -> 3

Commit message: Dangerous Prey
Connections:
- R16 pad 1: +3V3 -> /SDA_3V3
- R16 pad 2: /SDA_3V3 -> +3V3
Changed lines of the file:
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@@
 			(layers "F.Cu" "F.Mask" "F.Paste")
 			(roundrect_rratio 0.243902)
-			(net 30 "+3V3")
+			(net 33 "/SDA_3V3")
 			(pintype "passive")
 		)
@@
 			(layers "F.Cu" "F.Mask" "F.Paste")
 			(roundrect_rratio 0.243902)
-			(net 33 "/SDA_3V3")
+			(net 30 "+3V3")
 			(pintype "passive")
 		)
@@
 			)
 		)
-		(property "MPN" "1751251"
+		(property "MPN" "1984620"
 			(at 0 0 0)
 			(unlocked yes)
@@
 			)
 		)
-		(property "MPN" "1868128"
+		(property "MPN" "1984617"
 			(at 0 0 0)
 			(unlocked yes)
@@
 			)
 		)
+		(property "MPN" "1984617"
+			(at 0 0 0)
+			(unlocked yes)
+			(layer "F.Fab")
+			(hide yes)
+			(effects
+				(font
+					(size 1 1)
+					(thickness 0.15)
+				)
+			)
+		)
 		(property ki_fp_filters "TerminalBlock*:*")
 		(sheetname "/")
@@
 			)
 		)
-		(property "MPN" "1868128"
+		(property "MPN" "1984617"
 			(at 0 0 0)
 			(unlocked yes)

Commit message: Path of Vengeance
Parts:
- added C5: C, Capacitor_SMD:C_0805_2012Metric, F.Cu at (68.8, 52.0)
- added C6: C, Capacitor_SMD:C_0805_2012Metric, F.Cu at (49.1, 55.7)
- moved A1 50.9 mm to (136.8, 43.4), turned to 180 degrees
- moved J3 31.6 mm to (95.2, 66.4)
- moved J4 28.4 mm to (124.8, 66.4)
- moved R13 15.4 mm to (119.2, 57.0), turned to 0 degrees
- moved J1 12.8 mm to (105.1, 66.4)
- moved R17 8.95 mm to (73.4, 45.1), turned to -90 degrees
- moved R14 8.74 mm to (82.9, 45.1), turned to -90 degrees
- moved R16 6.26 mm to (76.6, 45.1), turned to 90 degrees
- moved R15 6.16 mm to (79.7, 45.1), turned to -90 degrees
- moved J2 6.08 mm to (114.9, 66.4)
- moved U2 5.00 mm to (78.3, 52.0), turned to 0 degrees
Routing:
- net +3V3: track 50.7 -> 89.0 mm
- net +12V: track 54.5 -> 25.5 mm
- net /D0: track 24.9 -> 8.56 mm
- net /D1: track 22.3 -> 7.22 mm
- net /A0: track 10.9 -> 25.9 mm
- net +5V: track 135.1 -> 149.6 mm, vias 2 -> 3
- net /D7: track 27.2 -> 13.9 mm
- net GND: track 11.1 -> 22.7 mm
- net /SCL_3V3: track 16.9 -> 25.3 mm, vias 0 -> 2
- net /SDA_3V3: track 23.0 -> 16.9 mm
- net /SCL_5V: track 86.4 -> 88.1 mm, vias 3 -> 2
- net /SDA_5V: track 84.9 -> 85.7 mm
