File: kicad/SonTinh/SonTinh.kicad_sch (KiCad schematic)
At the start: 12 parts, among them J1 Conn_01x02_Pin, J2 Conn_01x03_Pin, J3 Conn_01x02_Pin, J4 Conn_01x02_Pin, U1 BME680, U2 TCA9517ADGK

Commit message: Warrior... Princess
Parts:
- removed J1, J3, J4: Conn_01x02_Pin, Connector_Wire:SolderWire-0.75sqmm_1x02_P4.8mm_D1.25mm_OD2.3mm, symbol Connector:Conn_01x02_Pin
- removed J2: Conn_01x03_Pin, Connector_Wire:SolderWire-0.75sqmm_1x03_P4.8mm_D1.25mm_OD2.3mm, symbol Connector:Conn_01x03_Pin
- added J1: Conn_01x02_Socket, Connector_JST:JST_EH_S2B-EH_1x02_P2.50mm_Horizontal, symbol Connector:Conn_01x02_Socket
- added J2, J3: Conn_01x02_Socket, Connector_JST:JST_EH_B2B-EH-A_1x02_P2.50mm_Vertical, symbol Connector:Conn_01x02_Socket
- added J4: Conn_01x03_Socket, Connector_JST:JST_EH_B3B-EH-A_1x03_P2.50mm_Vertical, symbol Connector:Conn_01x03_Socket
Connections:
- net +12V: now also J4.1 (Pin_1)
- net A0: now also J3.2 (Pin_2)
- net D7: now also J4.3 (Pin_3)
- net GND: now also J1.2 (Pin_2), J2.2 (Pin_2), J3.1 (Pin_1), J4.2 (Pin_2)
- net D0: now reaches A1.D0 (D0/RX)
- net D0: now also J1.1 (Pin_1)
- net D1: now reaches A1.D1 (D1/TX)
- net D1: now also J2.1 (Pin_1)
- no-connect marks 21 -> 19

Commit message: Here She Comes... Miss Amphipolis
Parts:
- removed J1: Conn_01x02_Socket, Connector_JST:JST_EH_S2B-EH_1x02_P2.50mm_Horizontal, symbol Connector:Conn_01x02_Socket
- removed J2, J3: Conn_01x02_Socket, Connector_JST:JST_EH_B2B-EH-A_1x02_P2.50mm_Vertical, symbol Connector:Conn_01x02_Socket
- removed J4: Conn_01x03_Socket, Connector_JST:JST_EH_B3B-EH-A_1x03_P2.50mm_Vertical, symbol Connector:Conn_01x03_Socket
- added J8: 791077010, footprints:CONN22_791077010_MOL, symbol Molex:791077010
Connections:
- net +12V: now also J8.A1
- net +3V3: now also J8.B3
- net +5V: now also J8.B7
- net A0: now also J8.A8
- net D0: now also J8.A4
- net D1: now also J8.A6
- net D7: now also J8.A3
- net GND: now also J8.A11, J8.A2, J8.A5, J8.A7, J8.A9, J8.B4, J8.B8
- net SCL_3V3: now reaches R17.1, U1.4 (SCK), U2.2 (SCLA)
- net SCL_3V3: now also J8.B2
- net SDA_3V3: now reaches R16.2, U1.3 (SDI), U2.3 (SDAA)
- net SDA_3V3: now also J8.B1
- net SDA_5V: now reaches A1.D2 (D2/SDA), R15.1, U2.6 (SDAB)
- net SDA_5V: now also J8.B5
- net SCL_5V: now reaches A1.D3 (D3/SCL), R14.1, U2.7 (SCLB)
- net SCL_5V: now also J8.B6
- net A1: now reaches A1.A1
- net A1: now also J8.A10
- no-connect marks 19 -> 21

Commit message: Destiny
Changed lines of the file:
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@@
+	(wire
+		(pts
+			(xy 204.47 102.87) (xy 204.47 105.41)
+		)
+		(stroke
+			(width 0)
+			(type default)
+		)
+	)
 	(wire
 		(pts
@@
 	(wire
 		(pts
-			(xy 193.04 105.41) (xy 204.47 105.41)
+			(xy 177.8 102.87) (xy 204.47 102.87)
 		)
 		(stroke
@@
 	)
 	(symbol
+		(lib_id "power:+12V")
+		(at 177.8 102.87 90)
+		(unit 1)
+		(exclude_from_sim no)
+		(in_bom yes)
+		(on_board yes)
+		(dnp no)
+		(property "Reference" "#PWR05"
+			(at 181.61 102.87 0)
+			(effects
+				(font
+					(size 1.27 1.27)
+				)
+				(hide yes)
+			)
+		)
+		(property "Value" "+12V"
+			(at 173.99 102.8699 90)
+			(effects
+				(font
+					(size 1.27 1.27)
+				)
+				(justify left)
+			)
+		)
+		(property "Footprint" ""
+			(at 177.8 102.87 0)
+			(effects
+				(font
+					(size 1.27 1.27)
+				)
+				(hide yes)
+			)
+		)
+		(property "Datasheet" ""
+			(at 177.8 102.87 0)
+			(effects
+				(font
+					(size 1.27 1.27)
+				)
+				(hide yes)
+			)
+		)
+		(property "Description" "Power symbol creates a global label with name \"+12V\""
+			(at 177.8 102.87 0)
+			(effects
+				(font
+					(size 1.27 1.27)
+				)
+				(hide yes)
+			)
+		)
+		(pin "1"
+		)
+		(instances
+			(project "SonTinh"
+				(path "/91dda452-9985-4be5-905c-71f5be143fcf"
+					(reference "#PWR05")
+					(unit 1)
+				)
+			)
+		)
+	)
+	(symbol
 		(lib_id "power:GND")
 		(at 85.09 90.17 0)
@@
 	(symbol
 		(lib_id "power:+3V3")
-		(at 182.88 110.49 0)
+		(at 182.88 110.49 90)
 		(unit 1)
 		(exclude_from_sim no)
@@
 		(fields_autoplaced yes)
 		(property "Reference" "#PWR011"
-			(at 182.88 114.3 0)
+			(at 186.69 110.49 0)
 			(effects
 				(font
@@
 		)
 		(property "Value" "+3V3"
-			(at 182.88 105.41 0)
+			(at 181.61 107.95 90)
 			(effects
 				(font
@@
 	(symbol
 		(lib_id "power:+5V")
-		(at 187.96 107.95 0)
+		(at 187.96 107.95 90)
 		(unit 1)
 		(exclude_from_sim no)
@@
 		(fields_autoplaced yes)
 		(property "Reference" "#PWR01"
-			(at 187.96 111.76 0)
+			(at 191.77 107.95 0)
 			(effects
 				(font
@@
 		)
 		(property "Value" "+5V"
-			(at 187.96 102.87 0)
+			(at 186.69 105.41 90)
 			(effects
 				(font
@@
 					(unit 1)
 				)
-			)
-		)
-	)
-	(symbol
-		(lib_id "power:+12V")
-		(at 193.04 105.41 0)
-		(unit 1)
-		(exclude_from_sim no)
-		(in_bom yes)
-		(on_board yes)
-		(dnp no)
-		(property "Reference" "#PWR05"
-			(at 193.04 109.22 0)
-			(effects
-				(font
-					(size 1.27 1.27)
-				)
-				(hide yes)
-			)
-		)
-		(property "Value" "+12V"
-			(at 193.0401 101.6 90)
-			(effects
-				(font
-					(size 1.27 1.27)
-				)
-				(justify left)
-			)
-		)
-		(property "Footprint" ""
-			(at 193.04 105.41 0)
-			(effects
-				(font
-					(size 1.27 1.27)
-				)
-				(hide yes)
-			)
-		)
-		(property "Datasheet" ""
-			(at 193.04 105.41 0)
-			(effects
-				(font
-					(size 1.27 1.27)
-				)
-				(hide yes)
-			)
-		)
-		(property "Description" "Power symbol creates a global label with name \"+12V\""
-			(at 193.04 105.41 0)
-			(effects
-				(font
-					(size 1.27 1.27)
-				)
-				(hide yes)
-			)
-		)
-		(pin "1"
-		)
-		(instances
-			(project "SonTinh"
-				(path "/91dda452-9985-4be5-905c-71f5be143fcf"
-					(reference "#PWR05")
-					(unit 1)
-				)

Commit message: A Day in the Life
Parts:
- removed J8: 791077010, footprints:CONN22_791077010_MOL, symbol Molex:791077010
- added J1, J2, J3, J4: 1823450, footprints:1823450, symbol PheonicContact:1823450
Connections:
- net +3V3: now also J1.3 (2.1), J1.4 (2.2), J2.3 (2.1), J2.4 (2.2), J3.3 (2.1), J3.4 (2.2), J4.3 (2.1), J4.4 (2.2)
- net +5V: now also J1.5 (3.1), J1.6 (3.2), J2.5 (3.1), J2.6 (3.2), J3.5 (3.1), J3.6 (3.2), J4.5 (3.1), J4.6 (3.2)
- net GND: now also J1.1 (1.1), J1.2 (1.2), J2.1 (1.1), J2.2 (1.2), J3.1 (1.1), J3.2 (1.2), J4.1 (1.1), J4.2 (1.2)
- no-connect marks 21 -> 18
Other:
- moved on the sheet: R13

Commit message: For Him the Bell Tolls
Parts:
- removed J1, J2, J3, J4: 1823450, footprints:1823450, symbol PheonicContact:1823450
- added J1: 1752117, footprints:1752117, symbol PhoenicContact:1752117

Commit message: Blind Faith
Parts:
- removed J1: 1752117, footprints:1752117, symbol PhoenicContact:1752117
- added H1, H2: MountingHole_Pad, MountingHole:MountingHole_3.5mm_Pad, symbol Mechanical:MountingHole_Pad
- added J1, J2: Screw_Terminal_01x02, footprints:MKDSFW_15_2_35, symbol Connector:Screw_Terminal_01x02
- added J3: Screw_Terminal_01x02, footprints:MKDS_15_2_35, symbol Connector:Screw_Terminal_01x02
- added J4: Screw_Terminal_01x03, footprints:MKDS_15_3_35, symbol Connector:Screw_Terminal_01x03
Connections:
- net +12V: now also J4.1 (Pin_1)
- net A0: now also J2.1 (Pin_1)
- net D0: now also J1.1 (Pin_1)
- net D1: now also J3.1 (Pin_1)
- net D7: now also R13.2, J4.2 (Pin_2); no longer R13.1
- net GND: now also R13.1, H1.1, H2.1, J1.2 (Pin_2), J2.2 (Pin_2), J3.2 (Pin_2), J4.3 (Pin_3); no longer R13.2
Other:
- moved on the sheet: R13

Commit message: The Furies
Other:
- added sheet IRC-AT (irc_at.kicad_sch)
Changed lines of the file:
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@@
+		)
+	)
+	(sheet
+		(at 27.94 57.15)
+		(size 17.78 16.51)
+		(exclude_from_sim no)
+		(in_bom yes)
+		(on_board yes)
+		(dnp no)
+		(fields_autoplaced yes)
+		(stroke
+			(width 0.1524)
+			(type solid)
+		)
+		(fill
+			(color 0 0 0 0.0000)
+		)
+		(property "Sheetname" "IRC-AT"
+			(at 27.94 56.4384 0)
+			(effects
+				(font
+					(size 1.27 1.27)
+				)
+				(justify left bottom)
+			)
+		)
+		(property "Sheetfile" "irc_at.kicad_sch"
+			(at 27.94 74.2446 0)
+			(effects
+				(font
+					(size 1.27 1.27)
+				)
+				(justify left top)
+			)
+		)
+		(property "Datasheet" "../../docs/irc_at.pdf"
+			(at 27.94 57.15 0)
+			(effects
+				(font
+					(size 1.27 1.27)
+				)
+				(hide yes)
+			)
+		)
+		(instances
+			(project "SonTinh"
+				(path "/91dda452-9985-4be5-905c-71f5be143fcf"
+					(page "2")
+				)
+			)
 		)
 	)

Commit message: Been There, Done That
Parts:
- removed U1: BME680, Package_LGA:Bosch_LGA-8_3x3mm_P0.8mm_ClockwisePinNumbering, symbol Sensor:BME680
- added C1: C, Capacitor_SMD:C_0805_2012Metric, symbol Device:C
- added C2: C, symbol Device:C
- added IC1: SHT35-DIS-F2.5kS, footprints:SON50P250X250X100-9N-D, symbol Sensiron:SHT35-DIS-F2.5kS
- added IC2: STC31-C-R3, footprints:QFN80P300X350X110-13N-D, symbol Sensiron:STC31-C-R3
- added IC3: BMP384, footprints:BMP384, symbol Bosch:BMP384
Connections:
- net +3V3: now also C1.1, C2.1, IC3.1 (VDDIO), IC3.10 (VDD)
- net GND: now also C1.2, C2.2, IC3.3 (VSS_1), IC3.8 (VSS_2), IC3.9 (VSS_3)
- net SCL_3V3: now also IC3.2 (SCK)
- net SDA_3V3: now also IC3.4 (SDI)
- new net A2: IC3.5 (SDO)
Other:
- removed sheet IRC-AT
